File: main_unit/hardware/main_unit.kicad_sch (KiCad schematic)
At the start: 0 parts

Commit message: main_unit/hardware: Add STM32H753ZIT6 MCU to schematic
Parts:
- added U1: STM32H753ZIT6, Package_QFP:LQFP-100_14x14mm_P0.5mm, symbol MCU_ST_STM32H7:STM32H753ZITx
Connections:
- new net: U1.107 (VSS), U1.120 (VSS), U1.130 (VSS), U1.16 (VSS), U1.38 (VSS), U1.51 (VSS), U1.61 (VSS), U1.83 (VSS), U1.94 (VSS)

Commit message: main_unit/hardware: Add reset switch & capacitor
Parts:
- added C17, C18: 2u2, Capacitor_SMD:C_0603_1608Metric, symbol Device:C_Small
- added C19, C20: 1u, Capacitor_SMD:C_0603_1608Metric, symbol Device:C_Small
- added C21: 100n, Capacitor_SMD:C_0402_1005Metric, symbol Device:C_Small
- added SW1: SW_SPST, Connector_PinHeader_2.54mm:PinHeader_1x02_P2.54mm_Vertical, symbol Switch:SW_SPST
Connections:
- net at U1.106 (VCAP): now also C18.1
- net GND: now reaches U1.107 (VSS), U1.120 (VSS), U1.130 (VSS), U1.16 (VSS), U1.38 (VSS), U1.51 (VSS), U1.61 (VSS), U1.83 (VSS), U1.94 (VSS)
- net GND: now also U1.31 (VSSA), C17.2, C18.2, C19.2, C20.2, C21.1, SW1.2 (B)
- net +3V3: now reaches U1.108 (VDD)
- net +3V3: now also U1.121 (VDD), U1.131 (VDD), U1.144 (VDD), U1.17 (VDD), U1.30 (VDD), U1.33 (VDDA), U1.39 (VDD), U1.52 (VDD), U1.6 (VBAT), U1.62 (VDD), U1.72 (VDD), U1.84 (VDD), U1.95 (VDD33_USB), C19.1, C20.1
- net at U1.25 (NRST): now also C21.2, SW1.1 (A)
- net at U1.71 (VCAP): now also C17.1
- no-connect marks 0 -> 1
Other:
- added sheet Power (power.kicad_sch)
- note added: "1x bulk cap for VDD 1x bulk cap for VDDA"

Commit message: main_unit/hardware: Connect pull down resistor to BOOT0
Parts:
- added R1: 10k, symbol Device:R_Small
Connections:
- net GND: now also R1.2
- net at U1.138 (BOOT0): now also R1.1
- no-connect marks 1 -> 2
Changed lines of the file:
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@@
+	)
+	(no_connect
+		(at 77.47 125.73)
 	)
 	(no_connect
@@
 	(wire
 		(pts
+			(xy 67.31 133.35) (xy 67.31 135.89)
+		)
+		(stroke
+			(width 0)
+			(type default)
+		)
+	)
+	(wire
+		(pts
 			(xy 229.87 134.62) (xy 219.71 134.62)
 		)
@@
 		(pts
 			(xy 49.53 85.09) (xy 49.53 87.63)
+		)
+		(stroke
+			(width 0)
+			(type default)
+		)
+	)
+	(wire
+		(pts
+			(xy 67.31 125.73) (xy 67.31 128.27)
 		)
 		(stroke
@@
 	)
 	(symbol
+		(lib_id "Device:R_Small")
+		(at 67.31 130.81 0)
+		(unit 1)
+		(exclude_from_sim no)
+		(in_bom yes)
+		(on_board yes)
+		(dnp no)
+		(fields_autoplaced yes)
+		(property "Reference" "R1"
+			(at 69.85 129.5399 0)
+			(effects
+				(font
+					(size 1.016 1.016)
+				)
+				(justify left)
+			)
+		)
+		(property "Value" "10k"
+			(at 69.85 132.0799 0)
+			(effects
+				(font
+					(size 1.27 1.27)
+				)
+				(justify left)
+			)
+		)
+		(property "Footprint" ""
+			(at 67.31 130.81 0)
+			(effects
+				(font
+					(size 1.27 1.27)
+				)
+				(hide yes)
+			)
+		)
+		(property "Datasheet" "~"
+			(at 67.31 130.81 0)
+			(effects
+				(font
+					(size 1.27 1.27)
+				)
+				(hide yes)
+			)
+		)
+		(property "Description" "Resistor, small symbol"
+			(at 67.31 130.81 0)
+			(effects
+				(font
+					(size 1.27 1.27)
+				)
+				(hide yes)
+			)
+		)
+		(pin "1"
+		)
+		(pin "2"
+		)
+		(instances
+			(project ""
+				(path "/c1e2a568-b99f-4357-b0bb-65969671b711"
+					(reference "R1")
+					(unit 1)
+				)
+			)
+		)
+	)
+	(symbol
 		(lib_id "Device:C_Small")
 		(at 57.15 132.08 90)
@@
 					(unit 1)
 				)
+			)
+		)
+	)
+	(symbol
+		(lib_id "power:GND")
+		(at 67.31 135.89 0)
+		(unit 1)
+		(exclude_from_sim no)
+		(in_bom yes)
+		(on_board yes)
+		(dnp no)
+		(fields_autoplaced yes)
+		(property "Reference" "#PWR018"
+			(at 67.31 142.24 0)
+			(effects
+				(font
+					(size 1.27 1.27)
+				)
+				(hide yes)
+			)
+		)
+		(property "Value" "GND"
+			(at 67.31 140.97 0)
+			(effects
+				(font
+					(size 1.27 1.27)
+				)
+			)
+		)
+		(property "Footprint" ""
+			(at 67.31 135.89 0)
+			(effects
+				(font
+					(size 1.27 1.27)
+				)
+				(hide yes)
+			)
+		)
+		(property "Datasheet" ""
+			(at 67.31 135.89 0)
+			(effects
+				(font
+					(size 1.27 1.27)
+				)
+				(hide yes)
+			)
+		)
+		(property "Description" "Power symbol creates a global label with name \"GND\" , ground"
+			(at 67.31 135.89 0)
+			(effects
+				(font
+					(size 1.27 1.27)
+				)
+				(hide yes)
+			)
+		)
+		(pin "1"
+		)
+		(instances
+			(project "main_unit"
+				(path "/c1e2a568-b99f-4357-b0bb-65969671b711"
+					(reference "#PWR018")
+					(unit 1)
+				)

Commit message: main_unit/hardware: Add in 25MHz crystal oscillator and capacitors
Parts:
- added C22, C23: 18p, Capacitor_SMD:C_0201_0603Metric, symbol Device:C_Small
- added Y1: ABM8G-25.000MHZ-18-D2Y-T, Crystal:Crystal_SMD_Abracon_ABM8G-4Pin_3.2x2.5mm, symbol Device:Crystal_GND24
- R1: footprint (none) -> Resistor_SMD:R_0402_1005Metric
Connections:
- net GND: now also C22.2, C23.2, Y1.2, Y1.4
- net at U1.23 (PH0): now also C22.1, Y1.1
- net at U1.24 (PH1): now also C23.1, Y1.3

Commit message: main_unit/hardware: Add in 32.768kHz crystal
Parts:
- added C24, C25: 7p, Capacitor_SMD:C_0201_0603Metric, symbol Device:C_Small
- added Y2: SC32S-7PF20PPM, Crystal:Crystal_SMD_3215-2Pin_3.2x1.5mm, symbol Device:Crystal_Small
Connections:
- net GND: now also C24.1, C25.1
- net at U1.8 (PC14): now also C24.2, Y2.1
- net at U1.9 (PC15): now also C25.2, Y2.2

Commit message: main_unit/hardware: Fix STM32 to use LQFP-144 package instead of LQFP-100
Parts:
- U1: footprint Package_QFP:LQFP-100_14x14mm_P0.5mm -> Package_QFP:LQFP-144_20x20mm_P0.5mm
Changed lines of the file:
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@@
 			)
 		)
-		(property "Footprint" "Package_QFP:LQFP-100_14x14mm_P0.5mm"
+		(property "Footprint" "Package_QFP:LQFP-144_20x20mm_P0.5mm"
 			(at 234.95 120.65 0)
 			(effects

Commit message: main_unit/hardware: Assign all pins for STM32
Connections:
- net SDRAM_A0: now reaches U1.10 (PF0)
- net LCD_B3: now reaches U1.100 (PA8)
- net LCD_B4: now reaches U1.102 (PA10)
- net CAN_RX: now reaches U1.103 (PA11)
- net CAN_TX: now reaches U1.104 (PA12)
- net DBG_JTMS_SWDIO: now reaches U1.105 (PA13)
- net DBG_JTMS_SWCLK: now reaches U1.109 (PA14)
- net SDRAM_A1: now reaches U1.11 (PF1)
- net DBG_JTMS_JTDI: now reaches U1.110 (PA15)
- net SDMMC_D2: now reaches U1.111 (PC10)
- net SDMMC_D3: now reaches U1.112 (PC11)
- net SDMMC_CLK: now reaches U1.113 (PC12)
- net SDRAM_D2: now reaches U1.114 (PD0)
- net SDRAM_D3: now reaches U1.115 (PD1)
- net SDMMC_CMD: now reaches U1.116 (PD2)
- net LCD_G7: now reaches U1.117 (PD3)
- net SDRAM_A2: now reaches U1.12 (PF2)
- net LCD_B2: now reaches U1.122 (PD6)
- net LCDSPI_MOSI: now reaches U1.123 (PD7)
- net LCDSPI_MISO: now reaches U1.124 (PG9)
- net LCD_G3: now reaches U1.125 (PG10)
- net LCDSPI_SCK: now reaches U1.126 (PG11)
- net SDRAM_A3: now reaches U1.13 (PF3)
- net SDRAM_SDNCAS: now reaches U1.132 (PG15)
- net DBG_JTDO_SWO: now reaches U1.133 (PB3)
- net LCD_B6: now reaches U1.139 (PB8)
- net SDRAM_A4: now reaches U1.14 (PF4)
- net LCD_B7: now reaches U1.140 (PB9)
- net SDRAM_A5: now reaches U1.15 (PF5)
- net LCD_DE: now reaches U1.22 (PF10)
- net LCD_R5: now reaches U1.26 (PC0)
- net SDRAM_SDNE0: now reaches U1.28 (PC2_C)
- net SDRAM_SDCKE0: now reaches U1.29 (PC3_C)
- net LCD_R2: now reaches U1.35 (PA1)
- net LCD_R1: now reaches U1.36 (PA2)
- net LCD_B5: now reaches U1.37 (PA3)
- net LCD_VSYNC: now reaches U1.40 (PA4)
- net LCD_R4: now reaches U1.41 (PA5)
- net LCD_G2: now reaches U1.42 (PA6)
- net SDRAM_SDNWE: now reaches U1.43 (PA7)
- net LCD_R3: now reaches U1.46 (PB0)
- net LCD_R6: now reaches U1.47 (PB1)
- net SDRAM_SDNRAS: now reaches U1.49 (PF11)
- net SDRAM_A6: now reaches U1.50 (PF12)
- net SDRAM_A7: now reaches U1.53 (PF13)
- net SDRAM_A8: now reaches U1.54 (PF14)
- net SDRAM_A9: now reaches U1.55 (PF15)
- net SDRAM_A10: now reaches U1.56 (PG0)
- net SDRAM_A11: now reaches U1.57 (PG1)
- net SDRAM_D4: now reaches U1.58 (PE7)
- net SDRAM_D5: now reaches U1.59 (PE8)
- net SDRAM_D6: now reaches U1.60 (PE9)
- net SDRAM_D7: now reaches U1.63 (PE10)
- net SDRAM_D8: now reaches U1.64 (PE11)
- net SDRAM_D9: now reaches U1.65 (PE12)
- net SDRAM_D10: now reaches U1.66 (PE13)
- net SDRAM_D11: now reaches U1.67 (PE14)
- net SDRAM_D12: now reaches U1.68 (PE15)
- net LCD_G4: now reaches U1.69 (PB10)
- net LCD_G5: now reaches U1.70 (PB11)
- net UART_RX: now reaches U1.73 (PB12)
- net UART_TX: now reaches U1.74 (PB13)
- net SDRAM_D13: now reaches U1.77 (PD8)
- net SDRAM_D14: now reaches U1.78 (PD9)
- net SDRAM_D15: now reaches U1.79 (PD10)
- net SDRAM_D0: now reaches U1.85 (PD14)
- net SDRAM_D1: now reaches U1.86 (PD15)
- net SDRAM_BA0: now reaches U1.89 (PG4)
- net SDRAM_BA1: now reaches U1.90 (PG5)
- net LCD_R7: now reaches U1.91 (PG6)
- net LCD_CLK: now reaches U1.92 (PG7)
- net SDRAM_SDCLK: now reaches U1.93 (PG8)
- net LCD_HSYNC: now reaches U1.96 (PC6)
- net LCD_G6: now reaches U1.97 (PC7)
- net SDMMC_D0: now reaches U1.98 (PC8)
- net SDMMC_D1: now reaches U1.99 (PC9)
Other:
- moved on the sheet: C22, C23, C24, C25, Y1, Y2

Commit message: main_unit/hardware: Add in empty sheets for display, SDRAM, and debug
Other:
- added sheet Debug (untitled.kicad_sch)
- added sheet Display (display.kicad_sch)
- added sheet SDRAM (sdram.kicad_sch)
Changed lines of the file:
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@@
 	)
 	(sheet
-		(at 41.91 143.51)
+		(at 15.24 184.15)
+		(size 21.59 8.89)
+		(exclude_from_sim no)
+		(in_bom yes)
+		(on_board yes)
+		(dnp no)
+		(fields_autoplaced yes)
+		(stroke
+			(width 0.1524)
+			(type solid)
+		)
+		(fill
+			(color 0 0 0 0.0000)
+		)
+		(property "Sheetname" "Debug"
+			(at 15.24 183.4384 0)
+			(effects
+				(font
+					(size 1.27 1.27)
+				)
+				(justify left bottom)
+			)
+		)
+		(property "Sheetfile" "untitled.kicad_sch"
+			(at 15.24 193.6246 0)
+			(effects
+				(font
+					(size 1.27 1.27)
+				)
+				(justify left top)
+			)
+		)
+		(instances
+			(project "main_unit"
+				(path "/c1e2a568-b99f-4357-b0bb-65969671b711"
+					(page "5")
+				)
+			)
+		)
+	)
+	(sheet
+		(at 15.24 167.64)
+		(size 21.59 10.16)
+		(exclude_from_sim no)
+		(in_bom yes)
+		(on_board yes)
+		(dnp no)
+		(fields_autoplaced yes)
+		(stroke
+			(width 0.1524)
+			(type solid)
+		)
+		(fill
+			(color 0 0 0 0.0000)
+		)
+		(property "Sheetname" "SDRAM"
+			(at 15.24 166.9284 0)
+			(effects
+				(font
+					(size 1.27 1.27)
+				)
+				(justify left bottom)
+			)
+		)
+		(property "Sheetfile" "sdram.kicad_sch"
+			(at 15.24 178.3846 0)
+			(effects
+				(font
+					(size 1.27 1.27)
+				)
+				(justify left top)
+			)
+		)
+		(instances
+			(project "main_unit"
+				(path "/c1e2a568-b99f-4357-b0bb-65969671b711"
+					(page "4")
+				)
+			)
+		)
+	)
+	(sheet
+		(at 15.24 134.62)
 		(size 21.59 10.16)
 		(exclude_from_sim no)
@@
 		)
 		(property "Sheetname" "Power"
-			(at 41.91 142.7984 0)
+			(at 15.24 133.9084 0)
 			(effects
 				(font
@@
 		)
 		(property "Sheetfile" "power.kicad_sch"
-			(at 41.91 154.2546 0)
+			(at 15.24 145.3646 0)
 			(effects
 				(font
@@
 				)
 			)
+		)
+	)
+	(sheet
+		(at 15.24 151.13)
+		(size 21.59 10.16)
+		(exclude_from_sim no)
+		(in_bom yes)
+		(on_board yes)
+		(dnp no)
+		(fields_autoplaced yes)
+		(stroke
+			(width 0.1524)
+			(type solid)
+		)
+		(fill
+			(color 0 0 0 0.0000)
+		)
+		(property "Sheetname" "Display"
+			(at 15.24 150.4184 0)
+			(effects
+				(font
+					(size 1.27 1.27)
+				)
+				(justify left bottom)
+			)
+		)
+		(property "Sheetfile" "display.kicad_sch"
+			(at 15.24 161.8746 0)
+			(effects
+				(font
+					(size 1.27 1.27)
+				)
+				(justify left top)
+			)
+		)
+		(property "Field2" ""
+			(at 15.24 151.13 0)
+			(effects
+				(font
+					(size 1.27 1.27)
+				)
+			)
+		)
+		(instances
+			(project "main_unit"
+				(path "/c1e2a568-b99f-4357-b0bb-65969671b711"
+					(page "3")
+				)
+			)
