File: main_unit/hardware/main_unit.kicad_sch (KiCad schematic)
At the start: 14 parts, among them SW1 SW_SPST, U1 STM32H753ZIT6, Y1 ABM8G-25.000MHZ-18-D2Y-T, Y2 SC32S-7PF20PPM

Commit message: main_unit/hardware: Add in display connector, expand LTDC to RGB888 (fixes pin error)
Connections:
- net LCD_B1: now reaches U1.127 (PG12)
- net LCD_R0: now reaches U1.128 (PG13)
- net LCD_RST: now reaches U1.129 (PG14)
- net LCD_B0: now reaches U1.3 (PE4)
- net LCD_G0: now reaches U1.4 (PE5)
- net LCD_G1: now reaches U1.5 (PE6)
- net LCDSPI_MISO renamed LCD_CS
- net LCDSPI_MOSI renamed LCDSPI_SDA

Commit message: main_unit/hardware: Change reset button type
Parts:
- SW1: value SW_SPST -> PTS636SM43SMTR LFS; footprint Connector_PinHeader_2.54mm:PinHeader_1x02_P2.54mm_Vertical -> Button_Switch_SMD:SW_Tactile_SPST_NO_Straight_CK_PTS636Sx25SMTRLFS
Changed lines of the file:
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@@
 		(dnp no)
 		(property "Reference" "SW1"
-			(at 54.61 125.222 0)
+			(at 54.102 123.952 0)
 			(effects
 				(font
@@
 			)
 		)
-		(property "Value" "SW_SPST"
-			(at 54.61 124.46 0)
+		(property "Value" "PTS636SM43SMTR LFS"
+			(at 53.848 125.73 0)
 			(effects
 				(font
-					(size 1.27 1.27)
+					(size 0.762 0.762)
 				)
-				(hide yes)
 			)
 		)
-		(property "Footprint" "Connector_PinHeader_2.54mm:PinHeader_1x02_P2.54mm_Vertical"
+		(property "Footprint" "Button_Switch_SMD:SW_Tactile_SPST_NO_Straight_CK_PTS636Sx25SMTRLFS"
 			(at 54.61 128.27 0)
 			(effects

Commit message: main_unit/hardware: Connect LCD controller FAULT and PWM pin to STM32
Connections:
- net LEDCTRL_DIM_PWM: now reaches U1.136 (PB6)
- net LEDCTRL_FAULT: now reaches U1.137 (PB7)
Changed lines of the file:
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@@
+	(wire
+		(pts
+			(xy 123.19 57.15) (xy 123.19 59.69)
+		)
+		(stroke
+			(width 0)
+			(type default)
+		)
+	)
 	(wire
 		(pts
@@
 		(pts
 			(xy 49.53 74.93) (xy 49.53 77.47)
+		)
+		(stroke
+			(width 0)
+			(type default)
+		)
+	)
+	(wire
+		(pts
+			(xy 120.65 57.15) (xy 120.65 59.69)
 		)
 		(stroke
@@
 		)
 	)
+	(global_label "LEDCTRL_DIM_PWM"
+		(shape output)
+		(at 120.65 57.15 90)
+		(fields_autoplaced yes)
+		(effects
+			(font
+				(size 1.27 1.27)
+			)
+			(justify left)
+		)
+		(property "Intersheetrefs" "${INTERSHEET_REFS}"
+			(at 120.65 36.7478 90)
+			(effects
+				(font
+					(size 1.27 1.27)
+				)
+				(justify left)
+				(hide yes)
+			)
+		)
+	)
 	(global_label "SDRAM_BA1"
 		(shape output)
@@
 				(hide yes)
 			)
+		)
+	)
+	(global_label "LEDCTRL_FAULT"
+		(shape input)
+		(at 123.19 57.15 90)
+		(fields_autoplaced yes)
+		(effects
+			(font
+				(size 1.27 1.27)
+			)
+			(justify left)
+		)
+		(property "Intersheetrefs" "${INTERSHEET_REFS}"
+			(at 123.19 39.711 90)
+			(effects
+				(font
+					(size 1.27 1.27)
+				)
+				(justify left)
+				(hide yes)
+			)

Commit message: main_unit/hardware: Add in input power filtering and ST-Link connector
Connections:
- net NRST: now reaches C21.2, SW1.1 (A), U1.25 (NRST)
Changed lines of the file:
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@@
+	)
+	(junction
+		(at 62.23 132.08)
+		(diameter 0)
+		(color 0 0 0 0)
 	)
 	(junction
@@
 		(pts
 			(xy 196.85 125.73) (xy 196.85 128.27)
+		)
+		(stroke
+			(width 0)
+			(type default)
+		)
+	)
+	(wire
+		(pts
+			(xy 62.23 132.08) (xy 62.23 134.62)
 		)
 		(stroke
@@
 			(effects
 				(font
+					(size 1.27 1.27)
+				)
+				(justify right)
+				(hide yes)
+			)
+		)
+	)
+	(global_label "NRST"
+		(shape input)
+		(at 62.23 134.62 270)
+		(fields_autoplaced yes)
+		(effects
+			(font
+				(size 1.27 1.27)
+			)
+			(justify right)
+		)
+		(property "Intersheetrefs" "${INTERSHEET_REFS}"
+			(at 62.23 142.3828 90)
+			(effects
+				(font

Commit message: main_unit/hardware: Rearrange more components, add CAN transceiver
Connections:
- net CAN_STANDBY: now reaches U1.101 (PA9)
Other:
- added sheet CANBus (canbus.kicad_sch)
Changed lines of the file:
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@@
 	(wire
 		(pts
+			(xy 85.09 57.15) (xy 85.09 59.69)
+		)
+		(stroke
+			(width 0)
+			(type default)
+		)
+	)
+	(wire
+		(pts
 			(xy 168.91 57.15) (xy 168.91 59.69)
 		)
@@
 		)
 	)
+	(global_label "CAN_STANDBY"
+		(shape output)
+		(at 85.09 57.15 90)
+		(fields_autoplaced yes)
+		(effects
+			(font
+				(size 1.27 1.27)
+			)
+			(justify left)
+		)
+		(property "Intersheetrefs" "${INTERSHEET_REFS}"
+			(at 85.09 41.2833 90)
+			(effects
+				(font
+					(size 1.27 1.27)
+				)
+				(justify left)
+				(hide yes)
+			)
+		)
+	)
 	(global_label "SDRAM_D0"
 		(shape bidirectional)
@@
 	)
 	(sheet
-		(at 15.24 184.15)
-		(size 21.59 8.89)
+		(at 38.1 151.13)
+		(size 21.59 10.16)
 		(exclude_from_sim no)
 		(in_bom yes)
@@
 		)
 		(property "Sheetname" "Debug"
-			(at 15.24 183.4384 0)
+			(at 38.1 150.4184 0)
 			(effects
 				(font
@@
 		)
 		(property "Sheetfile" "untitled.kicad_sch"
-			(at 15.24 193.6246 0)
+			(at 38.1 161.8746 0)
 			(effects
 				(font
@@
 	)
 	(sheet
-		(at 15.24 167.64)
+		(at 38.1 167.64)
+		(size 21.59 10.16)
+		(exclude_from_sim no)
+		(in_bom yes)
+		(on_board yes)
+		(dnp no)
+		(fields_autoplaced yes)
+		(stroke
+			(width 0.1524)
+			(type solid)
+		)
+		(fill
+			(color 0 0 0 0.0000)
+		)
+		(property "Sheetname" "CANBus"
+			(at 38.1 166.9284 0)
+			(effects
+				(font
+					(size 1.27 1.27)
+				)
+				(justify left bottom)
+			)
+		)
+		(property "Sheetfile" "canbus.kicad_sch"
+			(at 38.1 178.3846 0)
+			(effects
+				(font
+					(size 1.27 1.27)
+				)
+				(justify left top)
+			)
+		)
+		(instances
+			(project "main_unit"
+				(path "/c1e2a568-b99f-4357-b0bb-65969671b711"
+					(page "6")
+				)
+			)
+		)
+	)
+	(sheet
+		(at 13.97 184.15)
 		(size 21.59 10.16)
 		(exclude_from_sim no)
@@
 		)
 		(property "Sheetname" "SDRAM"
-			(at 15.24 166.9284 0)
+			(at 13.97 183.4384 0)
 			(effects
 				(font
@@
 		)
 		(property "Sheetfile" "sdram.kicad_sch"
-			(at 15.24 178.3846 0)
+			(at 13.97 194.8946 0)
 			(effects
 				(font
@@
 	)
 	(sheet
-		(at 15.24 134.62)
+		(at 13.97 151.13)
 		(size 21.59 10.16)
 		(exclude_from_sim no)
@@
 		)
 		(property "Sheetname" "Power"
-			(at 15.24 133.9084 0)
+			(at 13.97 150.4184 0)
 			(effects
 				(font
@@
 		)
 		(property "Sheetfile" "power.kicad_sch"
-			(at 15.24 145.3646 0)
+			(at 13.97 161.8746 0)
 			(effects
 				(font
@@
 	)
 	(sheet
-		(at 15.24 151.13)
+		(at 13.97 167.64)
 		(size 21.59 10.16)
 		(exclude_from_sim no)
@@
 		)
 		(property "Sheetname" "Display"
-			(at 15.24 150.4184 0)
+			(at 13.97 166.9284 0)
 			(effects
 				(font
@@
 		)
 		(property "Sheetfile" "display.kicad_sch"
-			(at 15.24 161.8746 0)
+			(at 13.97 178.3846 0)
 			(effects
 				(font
@@
 		)
 		(property "Field2" ""
-			(at 15.24 151.13 0)
+			(at 13.97 167.64 0)
 			(effects
 				(font
