File: main_unit/hardware/sdram.kicad_sch (KiCad schematic)
At the start: 0 parts

Commit message: main_unit/hardware: Add SDRAM chip in with connections
Parts:
- added U3: W9864G6KH-6, W9864G6KH-6:SOP80P1176X120-54N, symbol W9864G6KH-6:W9864G6KH-6
Connections:
- new net +3V3: U3.1 (VDD), U3.14 (VDD__1), U3.27 (VDD__2), U3.3 (VDDQ), U3.43 (VDDQ__2), U3.49 (VDDQ__3), U3.9 (VDDQ__1)
- new net GND: U3.12 (VSSQ__1), U3.28 (VSS), U3.41 (VSS__1), U3.46 (VSSQ__2), U3.52 (VSSQ__3), U3.54 (VSS__2), U3.6 (VSSQ)
- new net SDRAM_A0: U3.23 (A0)
- new net SDRAM_A1: U3.24 (A1)
- new net SDRAM_A10: U3.22 (A10/AP)
- new net SDRAM_A11: U3.35 (A11)
- new net SDRAM_A2: U3.25 (A2)
- new net SDRAM_A3: U3.26 (A3)
- new net SDRAM_A4: U3.29 (A4)
- new net SDRAM_A5: U3.30 (A5)
- new net SDRAM_A6: U3.31 (A6)
- new net SDRAM_A7: U3.32 (A7)
- new net SDRAM_A8: U3.33 (A8)
- new net SDRAM_A9: U3.34 (A9)
- new net SDRAM_BA0: U3.20 (BS0)
- new net SDRAM_BA1: U3.21 (BS1)
- new net SDRAM_D0: U3.2 (DQ0)
- new net SDRAM_D1: U3.4 (DQ1)
- new net SDRAM_D10: U3.45 (DQ10)
- new net SDRAM_D11: U3.47 (DQ11)
- new net SDRAM_D12: U3.48 (DQ12)
- new net SDRAM_D13: U3.50 (DQ13)
- new net SDRAM_D14: U3.51 (DQ14)
- new net SDRAM_D15: U3.53 (DQ15)
- new net SDRAM_D2: U3.5 (DQ2)
- new net SDRAM_D3: U3.7 (DQ3)
- new net SDRAM_D4: U3.8 (DQ4)
- new net SDRAM_D5: U3.10 (DQ5)
- new net SDRAM_D6: U3.11 (DQ6)
- new net SDRAM_D7: U3.13 (DQ7)
- new net SDRAM_D8: U3.42 (DQ8)
- new net SDRAM_D9: U3.44 (DQ9)
- new net SDRAM_SDCKE0: U3.37 (CKE)
- new net SDRAM_SDCLK: U3.38 (CLK)
- new net SDRAM_SDNCAS: U3.17 (~{CAS})
- new net SDRAM_SDNE0: U3.19 (~{CS})
- new net SDRAM_SDNRAS: U3.18 (~{RAS})
- new net SDRAM_SDNWE: U3.16 (~{WE})
