File: main_unit/hardware/main_unit.kicad_pcb (KiCad board)
At the start: 2 copper layers, 4 parts, among them U1 STM32H753ZIT6, U2 LD39200PU33R

Commit message: main_unit/hardware: Add PCB to project with STM32 decoupling & bulk capacitors in rough positions
Parts:
- added C10: 100n, Capacitor_SMD:C_0402_1005Metric, F.Cu at (130.2, 37.9)
- added C11: 100n, Capacitor_SMD:C_0402_1005Metric, F.Cu at (126.3, 28.3)
- added C12: 100n, Capacitor_SMD:C_0402_1005Metric, F.Cu at (122.4, 24.4)
- added C13: 100n, Capacitor_SMD:C_0402_1005Metric, F.Cu at (117.9, 19.8)
- added C14: 100n, Capacitor_SMD:C_0402_1005Metric, F.Cu at (107.9, 24.0)
- added C15: 100n, Capacitor_SMD:C_0402_1005Metric, F.Cu at (104.4, 27.6)
- added C16: 100n, Capacitor_SMD:C_0402_1005Metric, F.Cu at (99.8, 32.1)
- added C17: 2u2, Capacitor_SMD:C_0603_1608Metric, F.Cu at (132.8, 65.9)
- added C18: 2u2, Capacitor_SMD:C_0603_1608Metric, F.Cu at (132.8, 68.4)
- added C19: 1u, Capacitor_SMD:C_0603_1608Metric, F.Cu at (111.6, 50.5)
- added C20: 1u, Capacitor_SMD:C_0603_1608Metric, F.Cu at (115.0, 51.2)
- added C21: 100n, Capacitor_SMD:C_0402_1005Metric, F.Cu at (107.5, 71.0)
- added C22: 18p, Capacitor_SMD:C_0201_0603Metric, F.Cu at (123.7, 81.0)
- added C23: 18p, Capacitor_SMD:C_0201_0603Metric, F.Cu at (124.7, 86.0)
- added C24: 7p, Capacitor_SMD:C_0201_0603Metric, F.Cu at (124.2, 73.5)
- added C25: 7p, Capacitor_SMD:C_0201_0603Metric, F.Cu at (124.2, 78.5)
- added C3: 100n, Capacitor_SMD:C_0402_1005Metric, F.Cu at (101.5, 39.6)
- added C4: 100n, Capacitor_SMD:C_0402_1005Metric, F.Cu at (105.4, 43.5)
- added C5: 100n, Capacitor_SMD:C_0402_1005Metric, F.Cu at (110.0, 48.1)
- added C6: 100n, Capacitor_SMD:C_0402_1005Metric, F.Cu at (111.1, 49.2)
- added C7: 100n, Capacitor_SMD:C_0402_1005Metric, F.Cu at (118.6, 49.5)
- added C8: 100n, Capacitor_SMD:C_0402_1005Metric, F.Cu at (123.2, 44.9)
- added C9: 100n, Capacitor_SMD:C_0402_1005Metric, F.Cu at (126.7, 41.4)
- added R1: 10k, Resistor_SMD:R_0402_1005Metric, F.Cu at (100.5, 73.6)
- added SW1: SW_SPST, Connector_PinHeader_2.54mm:PinHeader_1x02_P2.54mm_Vertical, F.Cu at (101.3, 67.8)
- added Y1: ABM8G-25.000MHZ-18-D2Y-T, Crystal:Crystal_SMD_Abracon_ABM8G-4Pin_3.2x2.5mm, F.Cu at (124.2, 83.5)
- added Y2: SC32S-7PF20PPM, Crystal:Crystal_SMD_3215-2Pin_3.2x1.5mm, F.Cu at (124.5, 76.0)
- U1: footprint Package_QFP:LQFP-100_14x14mm_P0.5mm -> Package_QFP:LQFP-144_20x20mm_P0.5mm
- moved U1 18.6 mm to (115.0, 35.0), turned to 45 degrees
Connections:
- U1 pad 23: unconnected-(U1-PH0-Pad23) -> Net-(U1-PH0)
- U1 pad 24: unconnected-(U1-PH1-Pad24) -> Net-(U1-PH1)
- U1 pad 25: unconnected-(U1-NRST-Pad25) -> Net-(SW1-A)
- U1 pad 71: unconnected-(U1-VCAP-Pad71) -> Net-(C17-Pad1)
- U1 pad 8: unconnected-(U1-PC14-Pad8) -> Net-(U1-PC14)
- U1 pad 9: unconnected-(U1-PC15-Pad9) -> Net-(U1-PC15)

Commit message: main_unit/hardware: Get rough positioning of crystals
Parts:
- moved C24 41.4 mm to (98.5, 41.0), turned to 45 degrees
- moved Y2 41.2 mm to (100.2, 42.8), turned to 135 degrees
- moved C23 40.9 mm to (107.2, 49.0), turned to 45 degrees
- moved C25 40.6 mm to (102.0, 44.5), turned to 45 degrees
- moved Y1 40.4 mm to (105.5, 47.6), turned to -135 degrees
- moved C22 40.0 mm to (103.8, 46.2), turned to -135 degrees
- moved C20 0.50 mm to (115.0, 51.8)

Commit message: main_unit/hardware: Position VCAP capacitors
Parts:
- moved C18 50.0 mm to (119.2, 20.3), turned to 45 degrees
- moved C17 26.9 mm to (129.7, 39.1), turned to -45 degrees
Changed lines of the file:
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@@
 	(footprint "Capacitor_SMD:C_0603_1608Metric"
 		(layer "F.Cu")
-		(at 132.84 65.86)
+		(at 129.723339 39.143013 -45)
 		(descr "Capacitor SMD 0603 (1608 Metric), square (rectangular) end terminal, IPC-7351 nominal, (Body size source: IPC-SM-782 page 76, https://www.pcb-3d.com/wordpress/wp-content/uploads/ipc-sm-782a_amendment_1_and_2.pdf), generated with kicad-footprint-generator")
 		(tags "capacitor")
 		(property "Reference" "C17"
-			(at 0 -1.43 0)
+			(at 0 -1.43 135)
 			(layer "F.SilkS")
+			(hide yes)
 			(effects
 				(font
@@
 		)
 		(property "Value" "2u2"
-			(at 0 1.43 0)
+			(at 0 1.43 135)
 			(layer "F.Fab")
 			(effects
@@
 		)
 		(property "Datasheet" "~"
-			(at 0 0 0)
+			(at 0 0 135)
 			(layer "F.Fab")
 			(hide yes)
@@
 		)
 		(property "Description" "Unpolarized capacitor, small symbol"
-			(at 0 0 0)
+			(at 0 0 135)
 			(layer "F.Fab")
 			(hide yes)
@@
 		(attr smd)
 		(fp_line
-			(start -0.14058 -0.51)
-			(end 0.14058 -0.51)
+			(start -0.140581 0.51)
+			(end 0.140581 0.51)
 			(stroke
 				(width 0.12)
@@
 		)
 		(fp_line
-			(start -0.14058 0.51)
-			(end 0.14058 0.51)
+			(start -0.140581 -0.51)
+			(end 0.140581 -0.51)
 			(stroke
 				(width 0.12)
@@
 		)
 		(fp_line
-			(start -1.48 -0.73)
-			(end 1.48 -0.73)
+			(start -1.48 0.73)
+			(end -1.48 -0.73)
 			(stroke
 				(width 0.05)
@@
 		)
 		(fp_line
-			(start -1.48 0.73)
-			(end -1.48 -0.73)
+			(start -1.48 -0.73)
+			(end 1.48 -0.73)
 			(stroke
 				(width 0.05)
@@
 		)
 		(fp_line
-			(start 1.48 -0.73)
-			(end 1.48 0.73)
+			(start 1.48 0.73)
+			(end -1.48 0.73)
 			(stroke
 				(width 0.05)
@@
 		)
 		(fp_line
-			(start 1.48 0.73)
-			(end -1.48 0.73)
+			(start 1.48 -0.73)
+			(end 1.48 0.73)
 			(stroke
 				(width 0.05)
@@
 		)
 		(fp_line
-			(start -0.8 -0.4)
-			(end 0.8 -0.4)
+			(start -0.8 0.4)
+			(end -0.8 -0.4)
 			(stroke
 				(width 0.1)
@@
 		)
 		(fp_line
-			(start -0.8 0.4)
-			(end -0.8 -0.4)
+			(start -0.8 -0.4)
+			(end 0.8 -0.4)
 			(stroke
 				(width 0.1)
@@
 		)
 		(fp_line
-			(start 0.8 -0.4)
-			(end 0.8 0.4)
+			(start 0.8 0.4)
+			(end -0.8 0.4)
 			(stroke
 				(width 0.1)
@@
 		)
 		(fp_line
-			(start 0.8 0.4)
-			(end -0.8 0.4)
+			(start 0.8 -0.4)
+			(end 0.8 0.4)
 			(stroke
 				(width 0.1)
@@
 		)
 		(fp_text user "${REFERENCE}"
-			(at 0 0 0)
+			(at 0 0 135)
 			(layer "F.Fab")
 			(effects
@@
 		)
 		(pad "1" smd roundrect
-			(at -0.775 0)
+			(at -0.775 0 315)
 			(size 0.9 0.95)
 			(layers "F.Cu" "F.Mask" "F.Paste")
@@
 		)
 		(pad "2" smd roundrect
-			(at 0.775 0)
+			(at 0.775 0 315)
 			(size 0.9 0.95)
 			(layers "F.Cu" "F.Mask" "F.Paste")
@@
 	(footprint "Capacitor_SMD:C_0603_1608Metric"
 		(layer "F.Cu")
-		(at 132.84 68.37)
+		(at 119.183873 20.289684 45)
 		(descr "Capacitor SMD 0603 (1608 Metric), square (rectangular) end terminal, IPC-7351 nominal, (Body size source: IPC-SM-782 page 76, https://www.pcb-3d.com/wordpress/wp-content/uploads/ipc-sm-782a_amendment_1_and_2.pdf), generated with kicad-footprint-generator")
 		(tags "capacitor")
 		(property "Reference" "C18"
-			(at 0 -1.43 0)
+			(at 0 -1.43 45)
 			(layer "F.SilkS")
+			(hide yes)
 			(effects
 				(font
@@
 		)
 		(property "Value" "2u2"
-			(at 0 1.43 0)
+			(at 0 1.43 45)
 			(layer "F.Fab")
 			(effects
@@
 		)
 		(property "Datasheet" "~"
-			(at 0 0 0)
+			(at 0 0 45)
 			(layer "F.Fab")
 			(hide yes)
@@
 		)
 		(property "Description" "Unpolarized capacitor, small symbol"
-			(at 0 0 0)
+			(at 0 0 45)
 			(layer "F.Fab")
 			(hide yes)
@@
 		(attr smd)
 		(fp_line
-			(start -0.14058 -0.51)
-			(end 0.14058 -0.51)
+			(start -0.140581 -0.51)
+			(end 0.140581 -0.51)
 			(stroke
 				(width 0.12)
@@
 		)
 		(fp_line
-			(start -0.14058 0.51)
-			(end 0.14058 0.51)
+			(start -0.140581 0.51)
+			(end 0.140581 0.51)
 			(stroke
 				(width 0.12)
@@
 		)
 		(fp_text user "${REFERENCE}"
-			(at 0 0 0)
+			(at 0 0 45)
 			(layer "F.Fab")
 			(effects
@@
 		)
 		(pad "1" smd roundrect
-			(at -0.775 0)
+			(at -0.775 0 45)
 			(size 0.9 0.95)
 			(layers "F.Cu" "F.Mask" "F.Paste")
@@
 		)
 		(pad "2" smd roundrect
-			(at 0.775 0)
+			(at 0.775 0 45)
 			(size 0.9 0.95)
 			(layers "F.Cu" "F.Mask" "F.Paste")

Commit message: main_unit/hardware: Assign all pins for STM32
Connections:
- U1 pad 10: unconnected-(U1-PF0-Pad10) -> SDRAM_A0
- U1 pad 100: unconnected-(U1-PA8-Pad100) -> LCD_B3
- U1 pad 102: unconnected-(U1-PA10-Pad102) -> LCD_B4
- U1 pad 103: unconnected-(U1-PA11-Pad103) -> CAN_RX
- U1 pad 104: unconnected-(U1-PA12-Pad104) -> CAN_TX
- U1 pad 105: unconnected-(U1-PA13-Pad105) -> DBG_JTMS_SWDIO
- U1 pad 109: unconnected-(U1-PA14-Pad109) -> DBG_JTMS_SWCLK
- U1 pad 11: unconnected-(U1-PF1-Pad11) -> SDRAM_A1
- U1 pad 110: unconnected-(U1-PA15-Pad110) -> DBG_JTMS_JTDI
- U1 pad 111: unconnected-(U1-PC10-Pad111) -> SDMMC_D2
- U1 pad 112: unconnected-(U1-PC11-Pad112) -> SDMMC_D3
- U1 pad 113: unconnected-(U1-PC12-Pad113) -> SDMMC_CLK
- U1 pad 114: unconnected-(U1-PD0-Pad114) -> SDRAM_D2
- U1 pad 115: unconnected-(U1-PD1-Pad115) -> SDRAM_D3
- U1 pad 116: unconnected-(U1-PD2-Pad116) -> SDMMC_CMD
- U1 pad 117: unconnected-(U1-PD3-Pad117) -> LCD_G7
- U1 pad 12: unconnected-(U1-PF2-Pad12) -> SDRAM_A2
- U1 pad 122: unconnected-(U1-PD6-Pad122) -> LCD_B2
- U1 pad 123: unconnected-(U1-PD7-Pad123) -> LCDSPI_MOSI
- U1 pad 124: unconnected-(U1-PG9-Pad124) -> LCDSPI_MISO
- U1 pad 125: unconnected-(U1-PG10-Pad125) -> LCD_G3
- U1 pad 126: unconnected-(U1-PG11-Pad126) -> LCDSPI_SCK
- U1 pad 13: unconnected-(U1-PF3-Pad13) -> SDRAM_A3
- U1 pad 132: unconnected-(U1-PG15-Pad132) -> SDRAM_SDNCAS
- U1 pad 133: unconnected-(U1-PB3-Pad133) -> DBG_JTDO_SWO
- U1 pad 139: unconnected-(U1-PB8-Pad139) -> LCD_B6
- U1 pad 14: unconnected-(U1-PF4-Pad14) -> SDRAM_A4
- U1 pad 140: unconnected-(U1-PB9-Pad140) -> LCD_B7
- U1 pad 15: unconnected-(U1-PF5-Pad15) -> SDRAM_A5
- U1 pad 22: unconnected-(U1-PF10-Pad22) -> LCD_DE
- U1 pad 26: unconnected-(U1-PC0-Pad26) -> LCD_R5
- U1 pad 28: unconnected-(U1-PC2_C-Pad28) -> SDRAM_SDNE0
- U1 pad 29: unconnected-(U1-PC3_C-Pad29) -> SDRAM_SDCKE0
- U1 pad 35: unconnected-(U1-PA1-Pad35) -> LCD_R2
- U1 pad 36: unconnected-(U1-PA2-Pad36) -> LCD_R1
- U1 pad 37: unconnected-(U1-PA3-Pad37) -> LCD_B5
- U1 pad 40: unconnected-(U1-PA4-Pad40) -> LCD_VSYNC
- U1 pad 41: unconnected-(U1-PA5-Pad41) -> LCD_R4
- U1 pad 42: unconnected-(U1-PA6-Pad42) -> LCD_G2
- U1 pad 43: unconnected-(U1-PA7-Pad43) -> SDRAM_SDNWE
- U1 pad 46: unconnected-(U1-PB0-Pad46) -> LCD_R3
- U1 pad 47: unconnected-(U1-PB1-Pad47) -> LCD_R6
- U1 pad 49: unconnected-(U1-PF11-Pad49) -> SDRAM_SDNRAS
- U1 pad 50: unconnected-(U1-PF12-Pad50) -> SDRAM_A6
- U1 pad 53: unconnected-(U1-PF13-Pad53) -> SDRAM_A7
- U1 pad 54: unconnected-(U1-PF14-Pad54) -> SDRAM_A8
- U1 pad 55: unconnected-(U1-PF15-Pad55) -> SDRAM_A9
- U1 pad 56: unconnected-(U1-PG0-Pad56) -> SDRAM_A10
- U1 pad 57: unconnected-(U1-PG1-Pad57) -> SDRAM_A11
- U1 pad 58: unconnected-(U1-PE7-Pad58) -> SDRAM_D4
- U1 pad 59: unconnected-(U1-PE8-Pad59) -> SDRAM_D5
- U1 pad 60: unconnected-(U1-PE9-Pad60) -> SDRAM_D6
- U1 pad 63: unconnected-(U1-PE10-Pad63) -> SDRAM_D7
- U1 pad 64: unconnected-(U1-PE11-Pad64) -> SDRAM_D8
- U1 pad 65: unconnected-(U1-PE12-Pad65) -> SDRAM_D9
- U1 pad 66: unconnected-(U1-PE13-Pad66) -> SDRAM_D10
- U1 pad 67: unconnected-(U1-PE14-Pad67) -> SDRAM_D11
- U1 pad 68: unconnected-(U1-PE15-Pad68) -> SDRAM_D12
- U1 pad 69: unconnected-(U1-PB10-Pad69) -> LCD_G4
- U1 pad 70: unconnected-(U1-PB11-Pad70) -> LCD_G5
- U1 pad 73: unconnected-(U1-PB12-Pad73) -> UART_RX
- U1 pad 74: unconnected-(U1-PB13-Pad74) -> UART_TX
- U1 pad 77: unconnected-(U1-PD8-Pad77) -> SDRAM_D13
- U1 pad 78: unconnected-(U1-PD9-Pad78) -> SDRAM_D14
- U1 pad 79: unconnected-(U1-PD10-Pad79) -> SDRAM_D15
- U1 pad 85: unconnected-(U1-PD14-Pad85) -> SDRAM_D0
- U1 pad 86: unconnected-(U1-PD15-Pad86) -> SDRAM_D1
- U1 pad 89: unconnected-(U1-PG4-Pad89) -> SDRAM_BA0
- U1 pad 90: unconnected-(U1-PG5-Pad90) -> SDRAM_BA1
- U1 pad 91: unconnected-(U1-PG6-Pad91) -> LCD_R7
- U1 pad 92: unconnected-(U1-PG7-Pad92) -> LCD_CLK
- U1 pad 93: unconnected-(U1-PG8-Pad93) -> SDRAM_SDCLK
- U1 pad 96: unconnected-(U1-PC6-Pad96) -> LCD_HSYNC
- U1 pad 97: unconnected-(U1-PC7-Pad97) -> LCD_G6
- U1 pad 98: unconnected-(U1-PC8-Pad98) -> SDMMC_D0
- U1 pad 99: unconnected-(U1-PC9-Pad99) -> SDMMC_D1

Commit message: main_unit/hardware: Add in empty sheets for display, SDRAM, and debug
Parts:
- moved C21 4.98 mm to (103.8, 67.8), turned to 90 degrees
Changed lines of the file:
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@@
 	(footprint "Capacitor_SMD:C_0402_1005Metric"
 		(layer "F.Cu")
-		(at 107.52 71)
+		(at 103.75 67.75 90)
 		(descr "Capacitor SMD 0402 (1005 Metric), square (rectangular) end terminal, IPC-7351 nominal, (Body size source: IPC-SM-782 page 76, https://www.pcb-3d.com/wordpress/wp-content/uploads/ipc-sm-782a_amendment_1_and_2.pdf), generated with kicad-footprint-generator")
 		(tags "capacitor")
 		(property "Reference" "C21"
-			(at 0 -1.16 0)
+			(at 0 -1.16 90)
 			(layer "F.SilkS")
+			(hide yes)
 			(effects
 				(font
@@
 		)
 		(property "Value" "100n"
-			(at 0 1.16 0)
+			(at 0 1.16 90)
 			(layer "F.Fab")
 			(effects
@@
 		)
 		(property "Datasheet" "~"
-			(at 0 0 0)
+			(at 0 0 90)
 			(layer "F.Fab")
 			(hide yes)
@@
 		)
 		(property "Description" "Unpolarized capacitor, small symbol"
-			(at 0 0 0)
+			(at 0 0 90)
 			(layer "F.Fab")
 			(hide yes)
@@
 		)
 		(fp_line
+			(start 0.91 -0.46)
+			(end 0.91 0.46)
+			(stroke
+				(width 0.05)
+				(type solid)
+			)
+			(layer "F.CrtYd")
+		)
+		(fp_line
 			(start -0.91 -0.46)
 			(end 0.91 -0.46)
+			(stroke
+				(width 0.05)
+				(type solid)
+			)
+			(layer "F.CrtYd")
+		)
+		(fp_line
+			(start 0.91 0.46)
+			(end -0.91 0.46)
 			(stroke
 				(width 0.05)
@@
 		)
 		(fp_line
-			(start 0.91 -0.46)
-			(end 0.91 0.46)
+			(start 0.5 -0.25)
+			(end 0.5 0.25)
 			(stroke
-				(width 0.05)
+				(width 0.1)
 				(type solid)
 			)
-			(layer "F.CrtYd")
-		)
-		(fp_line
-			(start 0.91 0.46)
-			(end -0.91 0.46)
-			(stroke
-				(width 0.05)
-				(type solid)
-			)
-			(layer "F.CrtYd")
+			(layer "F.Fab")
 		)
 		(fp_line
 			(start -0.5 -0.25)
 			(end 0.5 -0.25)
+			(stroke
+				(width 0.1)
+				(type solid)
+			)
+			(layer "F.Fab")
+		)
+		(fp_line
+			(start 0.5 0.25)
+			(end -0.5 0.25)
 			(stroke
 				(width 0.1)
@@
 			(layer "F.Fab")
 		)
-		(fp_line
-			(start 0.5 -0.25)
-			(end 0.5 0.25)
-			(stroke
-				(width 0.1)
-				(type solid)
-			)
-			(layer "F.Fab")
-		)
-		(fp_line
-			(start 0.5 0.25)
-			(end -0.5 0.25)
-			(stroke
-				(width 0.1)
-				(type solid)
-			)
-			(layer "F.Fab")
-		)
 		(fp_text user "${REFERENCE}"
-			(at 0 0 0)
+			(at 0 0 90)
 			(layer "F.Fab")
 			(effects
@@
 		)
 		(pad "1" smd roundrect
-			(at -0.48 0)
+			(at -0.48 0 90)
 			(size 0.56 0.62)
 			(layers "F.Cu" "F.Mask" "F.Paste")
@@
 		)
 		(pad "2" smd roundrect
-			(at 0.48 0)
+			(at 0.48 0 90)
 			(size 0.56 0.62)
 			(layers "F.Cu" "F.Mask" "F.Paste")

Commit message: main_unit/hardware: Add in capacitors for SDRAM chip
Parts:
- added C26: 100n, Capacitor_SMD:C_0402_1005Metric, F.Cu at (72.0, 54.2)
- added C27: 1u, Capacitor_SMD:C_0603_1608Metric, F.Cu at (75.5, 54.5)
- added C28: 100n, Capacitor_SMD:C_0402_1005Metric, F.Cu at (72.0, 56.1)
- added C29: 100n, Capacitor_SMD:C_0402_1005Metric, F.Cu at (72.0, 58.1)
- added C30: 100n, Capacitor_SMD:C_0402_1005Metric, F.Cu at (72.0, 60.1)
- added C31: 100n, Capacitor_SMD:C_0402_1005Metric, F.Cu at (72.0, 62.1)
- added C32: 100n, Capacitor_SMD:C_0402_1005Metric, F.Cu at (72.0, 64.0)
- added C33: 100n, Capacitor_SMD:C_0402_1005Metric, F.Cu at (72.0, 66.0)
- added U3: W9864G6KH-6, W9864G6KH-6:SOP80P1176X120-54N, F.Cu at (81.9, 68.3)
Connections:
- U1 pad 141: unconnected-(U1-PE0-Pad141) -> SDRAM_NBL0
- U1 pad 142: unconnected-(U1-PE1-Pad142) -> SDRAM_NBL1

Commit message: main_unit/hardware: Set up rough position for SDRAM chip & capacitors
Parts:
- moved C26 94.5 mm to (162.4, 26.8), turned to 90 degrees
- moved C28 93.4 mm to (160.8, 27.2), turned to 90 degrees
- moved C27 91.2 mm to (164.5, 34.7), turned to -90 degrees
- moved C33 89.5 mm to (158.4, 42.5), turned to -90 degrees
- moved C29 89.4 mm to (156.0, 27.5), turned to 90 degrees
- moved C30 86.4 mm to (152.0, 27.5), turned to 90 degrees
- moved C32 84.4 mm to (153.6, 42.5), turned to -90 degrees
- moved C31 77.7 mm to (141.6, 27.5), turned to 90 degrees
- moved U3 77.6 mm to (152.0, 35.0), turned to -90 degrees

Commit message: main_unit/hardware: Add in display connector, expand LTDC to RGB888 (fixes pin error)
Parts:
- added J1: 62684-402100ALF, 62684-402100ALF:AMPHENOL_62684-402100ALF, F.Cu at (80.5, 35.0)
- moved R1 43.6 mm to (102.0, 30.0), turned to 135 degrees
Connections:
- U1 pad 127: unconnected-(U1-PG12-Pad127) -> LCD_B1
- U1 pad 128: unconnected-(U1-PG13-Pad128) -> LCD_R0
- U1 pad 3: unconnected-(U1-PE4-Pad3) -> LCD_B0
- U1 pad 4: unconnected-(U1-PE5-Pad4) -> LCD_G0
- U1 pad 5: unconnected-(U1-PE6-Pad5) -> LCD_G1
