File: main_unit/hardware/main_unit.kicad_pcb (KiCad board)
At the start: 2 copper layers, 41 parts, among them J1 62684-402100ALF, SW1 SW_SPST, U1 STM32H753ZIT6, U2 LD39200PU33R, U3 W9864G6KH-6, Y1 ABM8G-25.000MHZ-18-D2Y-T, Y2 SC32S-7PF20PPM

Commit message: main_unit/hardware: Add capacitors for display
Parts:
- added C34: 1u, Capacitor_SMD:C_0603_1608Metric, F.Cu at (86.8, 27.2)
- added C35: 100n, Capacitor_SMD:C_0402_1005Metric, F.Cu at (86.8, 28.5)
Connections:
- J1 pad 06: /Display/LCD_RST -> LCD_RST
- J1 pad 09: unconnected-(J1-Pad09) -> LCDSPI_SDA
- J1 pad 10: unconnected-(J1-Pad10) -> LCDSPI_SCK
- J1 pad 11: unconnected-(J1-Pad11) -> LCD_CS
- J1 pad 16: unconnected-(J1-Pad16) -> LCD_B2
- J1 pad 17: unconnected-(J1-Pad17) -> LCD_B3
- J1 pad 18: unconnected-(J1-Pad18) -> LCD_B4
- J1 pad 19: unconnected-(J1-Pad19) -> LCD_B5
- J1 pad 20: unconnected-(J1-Pad20) -> LCD_B6
- J1 pad 21: unconnected-(J1-Pad21) -> LCD_B7
- J1 pad 22: unconnected-(J1-Pad22) -> LCD_G2
- J1 pad 23: unconnected-(J1-Pad23) -> LCD_G3
- J1 pad 24: unconnected-(J1-Pad24) -> LCD_G4
- J1 pad 25: unconnected-(J1-Pad25) -> LCD_G5
- J1 pad 26: unconnected-(J1-Pad26) -> LCD_G6
- J1 pad 27: unconnected-(J1-Pad27) -> LCD_G7
- J1 pad 28: unconnected-(J1-Pad28) -> LCD_R2
- J1 pad 29: unconnected-(J1-Pad29) -> LCD_R3
- J1 pad 30: unconnected-(J1-Pad30) -> LCD_R4
- J1 pad 31: unconnected-(J1-Pad31) -> LCD_R5
- J1 pad 32: unconnected-(J1-Pad32) -> LCD_R6
- J1 pad 33: unconnected-(J1-Pad33) -> LCD_R7
- U1 pad 123: LCDSPI_MOSI -> LCDSPI_SDA
- U1 pad 124: LCDSPI_MISO -> LCD_CS
- U1 pad 129: unconnected-(U1-PG14-Pad129) -> LCD_RST

Commit message: main_unit/hardware: Get general layout of backlight driver components on PCB
Parts:
- added C36: 100n, Capacitor_SMD:C_0402_1005Metric, F.Cu at (155.2, 74.5)
- added C37: 2u2, Capacitor_SMD:C_0603_1608Metric, F.Cu at (156.9, 75.7)
- added C38: 1u, Capacitor_SMD:C_0603_1608Metric, F.Cu at (150.2, 69.9)
- added C39: 100n, Capacitor_SMD:C_0402_1005Metric, F.Cu at (151.9, 70.5)
- added C40: 1u, Capacitor_SMD:C_0805_2012Metric, F.Cu at (155.2, 70.7)
- added C41: 10u, Capacitor_SMD:C_0603_1608Metric, F.Cu at (147.2, 83.5)
- added C42: 47u, 865080342006:WCAP-ASLI_5X5.5_DXL_, F.Cu at (161.5, 77.7)
- added C43: 47u, 865080342006:WCAP-ASLI_5X5.5_DXL_, F.Cu at (143.5, 77.7)
- added C44: 100n, Capacitor_SMD:C_0402_1005Metric, F.Cu at (148.5, 82.9)
- added C45: 2n7, Capacitor_SMD:C_0201_0603Metric, F.Cu at (153.9, 70.7)
- added D1: BAT54T1G, Diode_SMD:D_SOD-123, F.Cu at (147.8, 79.5)
- added D2: BAT54T1G, Diode_SMD:D_SOD-123, F.Cu at (154.8, 79.5)
- added D3: BAT54T1G, Diode_SMD:D_SOD-123, F.Cu at (157.3, 79.5)
- added L1: 22u, Inductor_SMD:L_Taiyo-Yuden_NR-40xx, F.Cu at (151.3, 79.5)
- added Q1: 2N7002BK,215, Package_TO_SOT_SMD:SOT-23-3, F.Cu at (158.4, 72.7)
- added R10: 10k, Resistor_SMD:R_0402_1005Metric, F.Cu at (149.5, 82.9)
- added R11: 1k, Resistor_SMD:R_0402_1005Metric, F.Cu at (150.5, 82.9)
- added R12: 10k, Resistor_SMD:R_0402_1005Metric, F.Cu at (148.0, 76.5)
- added R13: 10k, Resistor_SMD:R_0402_1005Metric, F.Cu at (148.0, 75.5)
- added R14: 10k, Resistor_SMD:R_0402_1005Metric, F.Cu at (148.0, 70.5)
- added R15: 10k, Resistor_SMD:R_0402_1005Metric, F.Cu at (148.0, 69.5)
- added R2: 10k, Resistor_SMD:R_0402_1005Metric, F.Cu at (148.0, 71.5)
- added R3: 10k, Resistor_SMD:R_0402_1005Metric, F.Cu at (148.0, 74.5)
- added R4: 10k, Resistor_SMD:R_0402_1005Metric, F.Cu at (148.0, 73.5)
- added R7: 15k, Resistor_SMD:R_0402_1005Metric, F.Cu at (155.3, 73.0)
- added R8: 10k, Resistor_SMD:R_0402_1005Metric, F.Cu at (153.0, 70.5)
- added R9: 15k, Resistor_SMD:R_0402_1005Metric, F.Cu at (148.0, 72.5)
- added U4: MAX25512ATG/V+T, Package_DFN_QFN:WQFN-24-1EP_4x4mm_P0.5mm_EP2.45x2.45mm_ThermalVias, F.Cu at (151.7, 74.2)
- moved C11 79.4 mm to (163.8, 98.3)
- moved C14 79.4 mm to (145.4, 94.0)
- moved C4 79.4 mm to (142.9, 113.5)
- moved C5 79.4 mm to (147.5, 118.1)
- moved C9 79.4 mm to (164.2, 111.4)
- moved C10 79.4 mm to (167.7, 107.9)
- moved C12 79.4 mm to (159.9, 94.4)
- moved C13 79.4 mm to (155.4, 89.8)
- moved C15 79.4 mm to (141.9, 97.6)
- moved C16 79.4 mm to (137.3, 102.1)
- moved C17 79.4 mm to (167.2, 109.1)
- moved C18 79.4 mm to (156.7, 90.3)
- moved C19 79.4 mm to (149.1, 120.5)
- moved C20 79.4 mm to (152.5, 121.8)
- moved C22 79.4 mm to (141.2, 116.2)
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
Commit message: main_unit/hardware: Change reset button type
Parts:
- SW1: value SW_SPST -> PTS636SM43SMTR LFS; footprint Connector_PinHeader_2.54mm:PinHeader_1x02_P2.54mm_Vertical -> Button_Switch_SMD:SW_Tactile_SPST_NO_Straight_CK_PTS636Sx25SMTRLFS
- moved SW1 58.2 mm to (152.5, 128.2)
- moved C21 43.2 mm to (145.8, 116.3), turned to 45 degrees
- moved C22 0.72 mm to (140.7, 116.8)
- moved Y1 0.72 mm to (142.5, 118.1)
- moved C23 0.72 mm to (144.2, 119.5)
Changed lines of the file:
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@@
 	(footprint "Capacitor_SMD:C_0201_0603Metric"
 		(layer "F.Cu")
-		(at 141.25 116.25 -135)
+		(at 140.743952 116.756048 -135)
 		(descr "Capacitor SMD 0201 (0603 Metric), square (rectangular) end terminal, IPC-7351 nominal, (Body size source: https://www.vishay.com/docs/20052/crcw0201e3.pdf), generated with kicad-footprint-generator")
 		(tags "capacitor")
@@
 	(footprint "Capacitor_SMD:C_0402_1005Metric"
 		(layer "F.Cu")
-		(at 121.25 80.77 90)
+		(at 145.758571 116.337623 45)
 		(descr "Capacitor SMD 0402 (1005 Metric), square (rectangular) end terminal, IPC-7351 nominal, (Body size source: IPC-SM-782 page 76, https://www.pcb-3d.com/wordpress/wp-content/uploads/ipc-sm-782a_amendment_1_and_2.pdf), generated with kicad-footprint-generator")
 		(tags "capacitor")
 		(property "Reference" "C21"
-			(at 0 -1.16 90)
+			(at 0 -1.16 45)
 			(layer "F.SilkS")
 			(hide yes)
@@
 		)
 		(property "Value" "100n"
-			(at 0 1.16 90)
+			(at 0 1.16 45)
 			(layer "F.Fab")
 			(effects
@@
 		)
 		(property "Datasheet" "~"
-			(at 0 0 90)
+			(at 0 0 45)
 			(layer "F.Fab")
 			(hide yes)
@@
 		)
 		(property "Description" "Unpolarized capacitor, small symbol"
-			(at 0 0 90)
+			(at 0 0 45)
 			(layer "F.Fab")
 			(hide yes)
@@
 		)
 		(fp_line
-			(start 0.91 -0.46)
-			(end 0.91 0.46)
+			(start -0.91 -0.46)
+			(end 0.91 -0.46)
 			(stroke
 				(width 0.05)
@@
 		)
 		(fp_line
-			(start -0.91 -0.46)
-			(end 0.91 -0.46)
+			(start -0.91 0.46)
+			(end -0.91 -0.46)
 			(stroke
 				(width 0.05)
@@
 		)
 		(fp_line
-			(start 0.91 0.46)
-			(end -0.91 0.46)
+			(start 0.91 -0.46)
+			(end 0.91 0.46)
 			(stroke
 				(width 0.05)
@@
 		)
 		(fp_line
-			(start -0.91 0.46)
-			(end -0.91 -0.46)
+			(start 0.91 0.46)
+			(end -0.91 0.46)
 			(stroke
 				(width 0.05)
@@
 		)
 		(fp_line
-			(start 0.5 -0.25)
-			(end 0.5 0.25)
+			(start -0.5 -0.25)
+			(end 0.5 -0.25)
 			(stroke
 				(width 0.1)
@@
 		)
 		(fp_line
-			(start -0.5 -0.25)
-			(end 0.5 -0.25)
+			(start -0.5 0.25)
+			(end -0.5 -0.25)
 			(stroke
 				(width 0.1)
@@
 		)
 		(fp_line
-			(start 0.5 0.25)
-			(end -0.5 0.25)
+			(start 0.5 -0.25)
+			(end 0.5 0.25)
 			(stroke
 				(width 0.1)
@@
 		)
 		(fp_line
-			(start -0.5 0.25)
-			(end -0.5 -0.25)
+			(start 0.5 0.25)
+			(end -0.5 0.25)
 			(stroke
 				(width 0.1)
@@
 		)
 		(fp_text user "${REFERENCE}"
-			(at 0 0 90)
+			(at 0 0 45)
 			(layer "F.Fab")
 			(effects
@@
 		)
 		(pad "1" smd roundrect
-			(at -0.48 0 90)
+			(at -0.48 0 45)
 			(size 0.56 0.62)
 			(layers "F.Cu" "F.Mask" "F.Paste")
@@
 		)
 		(pad "2" smd roundrect
-			(at 0.48 0 90)
+			(at 0.48 0 45)
 			(size 0.56 0.62)
 			(layers "F.Cu" "F.Mask" "F.Paste")
@@
 	(footprint "Capacitor_SMD:C_0201_0603Metric"
 		(layer "F.Cu")
-		(at 144.75 119.007716 45)
+		(at 144.243952 119.513764 45)
 		(descr "Capacitor SMD 0201 (0603 Metric), square (rectangular) end terminal, IPC-7351 nominal, (Body size source: https://www.vishay.com/docs/20052/crcw0201e3.pdf), generated with kicad-footprint-generator")
 		(tags "capacitor")
@@
 		)
 	)
-	(footprint "Connector_PinHeader_2.54mm:PinHeader_1x02_P2.54mm_Vertical"
+	(footprint "Button_Switch_SMD:SW_Tactile_SPST_NO_Straight_CK_PTS636Sx25SMTRLFS"
 		(layer "F.Cu")
-		(at 118.84 80.78)
-		(descr "Through hole straight pin header, 1x02, 2.54mm pitch, single row")
-		(tags "Through hole pin header THT 1x02 2.54mm single row")
+		(at 152.5 128.25)
+		(descr "Tactile switch, SPST, 6.0x3.5 mm, H2.5 mm, straight, NO, gull wing leads: https://www.ckswitches.com/media/2779/pts636.pdf")
+		(tags "switch tactile SPST 1P1T straight NO SMTR C&K")
 		(property "Reference" "SW1"
-			(at 0 -2.38 0)
+			(at 0 -3 0)
+			(unlocked yes)
 			(layer "F.SilkS")
 			(effects
@@
 			)
 		)
-		(property "Value" "SW_SPST"
-			(at 0 4.92 0)
+		(property "Value" "PTS636SM43SMTR LFS"
+			(at 0 3 0)
+			(unlocked yes)
 			(layer "F.Fab")
 			(effects
@@
 		(property "Datasheet" "~"
 			(at 0 0 0)
+			(unlocked yes)
 			(layer "F.Fab")
 			(hide yes)
@@
 		(property "Description" "Single Pole Single Throw (SPST) switch"
 			(at 0 0 0)
+			(unlocked yes)
 			(layer "F.Fab")
 			(hide yes)
@@
 		(sheetname "/")
 		(sheetfile "main_unit.kicad_sch")
-		(attr through_hole)
+		(attr smd)
 		(fp_line
-			(start -1.38 -1.38)
-			(end 0 -1.38)
+			(start -3.2 -2)
+			(end -3.2 -0.8)
 			(stroke
 				(width 0.12)
@@
 		)
 		(fp_line
-			(start -1.38 0)
-			(end -1.38 -1.38)
+			(start -3.2 0.8)
+			(end -3.2 2)
 			(stroke
 				(width 0.12)
@@
 		)
 		(fp_line
-			(start -1.38 1.27)
-			(end -1.38 3.92)
+			(start -3.2 2)
+			(end 3.2 2)
 			(stroke
 				(width 0.12)
@@
 		)
 		(fp_line
-			(start -1.38 1.27)
-			(end 1.38 1.27)
+			(start 3.2 -2)
+			(end -3.2 -2)
 			(stroke
 				(width 0.12)
@@
 		)
 		(fp_line
-			(start -1.38 3.92)
-			(end 1.38 3.92)
+			(start 3.2 -0.8)
+			(end 3.2 -2)
 			(stroke
 				(width 0.12)
@@
 		)
 		(fp_line
-			(start 1.38 1.27)
-			(end 1.38 3.92)
+			(start 3.2 2)
+			(end 3.2 0.8)
 			(stroke
 				(width 0.12)
@@
 			(layer "F.SilkS")
 		)
+		(fp_rect
+			(start -1.35 -0.65)
+			(end 1.35 0.65)
+			(stroke
+				(width 0.12)
+				(type solid)
+			)
+			(fill no)
+			(layer "Dwgs.User")
+		)
 		(fp_line
-			(start -1.77 -1.77)
-			(end -1.77 4.32)
+			(start -4.75 -0.75)
+			(end -3.3 -0.75)
 			(stroke
 				(width 0.05)
@@
 		)
 		(fp_line
-			(start -1.77 4.32)
-			(end 1.77 4.32)
+			(start -4.75 0.75)
+			(end -4.75 -0.75)
 			(stroke
 				(width 0.05)
@@
 		)
 		(fp_line
-			(start 1.77 -1.77)
-			(end -1.77 -1.77)
+			(start -3.3 -2.1)
+			(end 3.3 -2.1)
 			(stroke
 				(width 0.05)
@@
 		)
 		(fp_line
-			(start 1.77 4.32)
-			(end 1.77 -1.77)
+			(start -3.3 -0.75)
+			(end -3.3 -2.1)
 			(stroke
 				(width 0.05)
@@
 		)
 		(fp_line
-			(start -1.27 -0.635)
-			(end -0.635 -1.27)
+			(start -3.3 0.75)
+			(end -4.75 0.75)
 			(stroke
-				(width 0.1)
+				(width 0.05)
 				(type solid)
 			)
-			(layer "F.Fab")
+			(layer "F.CrtYd")
 		)
 		(fp_line
-			(start -1.27 3.81)
-			(end -1.27 -0.635)
+			(start -3.3 2.1)
+			(end -3.3 0.75)
 			(stroke
-				(width 0.1)
+				(width 0.05)
 				(type solid)
 			)
-			(layer "F.Fab")
+			(layer "F.CrtYd")
 		)
 		(fp_line
-			(start -0.635 -1.27)
-			(end 1.27 -1.27)
+			(start 3.3 -2.1)
+			(end 3.3 -0.75)
 			(stroke
-				(width 0.1)
+				(width 0.05)
 				(type solid)
 			)
-			(layer "F.Fab")
+			(layer "F.CrtYd")
 		)
 		(fp_line
-			(start 1.27 -1.27)
-			(end 1.27 3.81)
+			(start 3.3 -0.75)
+			(end 4.75 -0.75)
 			(stroke
-				(width 0.1)
+				(width 0.05)
 				(type solid)
 			)
-			(layer "F.Fab")
+			(layer "F.CrtYd")
+		)
+		(fp_line
+			(start 3.3 0.75)
+			(end 3.3 2.1)
+			(stroke
+				(width 0.05)
+				(type solid)
+			)
+			(layer "F.CrtYd")
+		)
+		(fp_line
+			(start 3.3 2.1)
+			(end -3.3 2.1)
+			(stroke
+				(width 0.05)
+				(type solid)
+			)
+			(layer "F.CrtYd")
+		)
+		(fp_line
+			(start 4.75 -0.75)
+			(end 4.75 0.75)
+			(stroke
+				(width 0.05)
+				(type solid)
+			)
+			(layer "F.CrtYd")
 		)
 		(fp_line
-			(start 1.27 3.81)
-			(end -1.27 3.81)
+			(start 4.75 0.75)
+			(end 3.3 0.75)
+			(stroke
+				(width 0.05)
+				(type solid)
+			)
+			(layer "F.CrtYd")
+		)
+		(fp_rect
+			(start -3.05 -1.85)
+			(end 3.05 1.85)
 			(stroke
 				(width 0.1)
 				(type solid)
 			)
+			(fill no)
 			(layer "F.Fab")
 		)
 		(fp_text user "${REFERENCE}"
-			(at 0 1.27 90)
+			(at 0 0 0)
+			(unlocked yes)
 			(layer "F.Fab")
 			(effects
 				(font
-					(size 1 1)
-					(thickness 0.15)
+					(size 0.5 0.5)
+					(thickness 0.1)
 				)
 			)
 		)
-		(pad "1" thru_hole rect
-			(at 0 0)
-			(size 1.7 1.7)
-			(drill 1)
-			(layers "*.Cu" "*.Mask")
-			(remove_unused_layers no)
+		(pad "1" smd rect
+			(at -3.875 0)
+			(size 1.25 1)
+			(layers "F.Cu" "F.Mask" "F.Paste")
 			(net 27 "Net-(SW1-A)")
 			(pinfunction "A")
 			(pintype "passive")
 		)
-		(pad "2" thru_hole circle
-			(at 0 2.54)
-			(size 1.7 1.7)
-			(drill 1)
-			(layers "*.Cu" "*.Mask")
-			(remove_unused_layers no)
+		(pad "2" smd rect
+			(at 3.875 0)
+			(size 1.25 1)
+			(layers "F.Cu" "F.Mask" "F.Paste")
 			(net 1 "GND")
 			(pinfunction "B")
@@
 		)
 		(embedded_fonts no)
-		(model "${KICAD9_3DMODEL_DIR}/Connector_PinHeader_2.54mm.3dshapes/PinHeader_1x02_P2.54mm_Vertical.step"
+		(model "${KICAD9_3DMODEL_DIR}/Button_Switch_SMD.3dshapes/SW_Tactile_SPST_NO_Straight_CK_PTS636Sx25SMTRLFS.step"
 			(offset
 				(xyz 0 0 0)
@@
 	(footprint "Crystal:Crystal_SMD_Abracon_ABM8G-4Pin_3.2x2.5mm"
 		(layer "F.Cu")
-		(at 143 117.628858 -135)
+		(at 142.493952 118.134906 -135)
 		(descr "Abracon ABM8G, Miniature Ceramic Crystal, 3.2x2.5mm package, SMD, generated with kicad-footprint-generator make_crystal.py, http://www.abracon.com/Resonators/ABM8G.pdf")
 		(property "Reference" "Y1"

Commit message: main_unit/hardware: Connect LCD controller FAULT and PWM pin to STM32
Connections:
- U1 pad 136: unconnected-(U1-PB6-Pad136) -> LEDCTRL_DIM_PWM
- U1 pad 137: unconnected-(U1-PB7-Pad137) -> LEDCTRL_FAULT

Commit message: main_unit/hardware: Add in extra capacitor for BOSTMON, move things around slightly for MAX chip according to datasheet recommendations
Parts:
- added C46: 47p, Capacitor_SMD:C_0201_0603Metric, F.Cu at (155.0, 73.6)
- moved R10 12.2 mm to (157.2, 73.5), turned to 180 degrees
- moved R11 10.8 mm to (157.2, 74.5), turned to 0 degrees
- moved Q1 1.52 mm to (158.4, 71.2)
- moved C38 0.50 mm to (150.8, 69.9)
- moved C40 0.22 mm to (155.2, 70.5)
- moved R7 0.22 mm to (155.3, 72.8)

Commit message: main_unit/hardware: Rearrange components in boost converter to minimize loop area
Parts:
- moved D2 11.5 mm to (159.0, 68.8), turned to 180 degrees
- moved D3 8.37 mm to (159.0, 71.2), turned to 0 degrees
- moved C41 5.00 mm to (144.8, 79.1)
- moved C44 4.76 mm to (146.0, 78.8)
- moved C42 4.39 mm to (157.8, 80.0), turned to 180 degrees
- moved C43 4.20 mm to (144.0, 73.5)
- moved Q1 3.89 mm to (160.2, 74.6), turned to -90 degrees
- moved D1 0.55 mm to (147.8, 80.0), turned to -90 degrees
- moved L1 0.53 mm to (151.3, 80.0)

Commit message: main_unit/hardware: Add in input power filtering and ST-Link connector
Parts:
- added C47: 47u, 865080342006:WCAP-ASLI_5X5.5_DXL_, F.Cu at (187.0, 76.8)
- added D4: D5V0H1B2LP-7B, Diode_SMD:D_0402_1005Metric, F.Cu at (193.5, 81.0)
- added J2: Conn_02x07_Odd_Even, FTSH-107-01-L-DV-K-A:SAMTEC_FTSH-107-01-L-DV-K-A, F.Cu at (174.5, 75.2)
- added J3: 691137710002, 691137710002:691137710002, F.Cu at (196.5, 76.0)
- moved C1 63.1 mm to (190.3, 83.0), turned to -90 degrees
- moved C2 56.0 mm to (183.3, 83.0), turned to -90 degrees
- moved U2 54.4 mm to (187.0, 83.0)
Connections:
- net Net-(SW1-A) renamed NRST
