File: main_unit/hardware/main_unit.kicad_pcb (KiCad board)
At the start: 2 copper layers, 76 parts, among them J1 62684-402100ALF, J2 Conn_02x07_Odd_Even, J3 691137710002, Q1 2N7002BK,215, SW1 PTS636SM43SMTR LFS, U1 STM32H753ZIT6, U2 LD39200PU33R, U3 W9864G6KH-6, U4 MAX25512ATG/V+T, Y1 ABM8G-25.000MHZ-18-D2Y-T, Y2 SC32S-7PF20PPM

Commit message: main_unit/hardware: Rearrange components
Parts:
- added REF**: ESD-Logo_6.6x6mm_SilkScreen, Symbol:ESD-Logo_6.6x6mm_SilkScreen, F.Cu at (133.2, 71.8)
- moved C26 24.6 mm to (175.4, 94.6), turned to 180 degrees
- moved J2 23.0 mm to (152.5, 82.0)
- moved C28 22.4 mm to (175.9, 96.2), turned to 180 degrees
- moved C27 22.3 mm to (183.3, 92.5), turned to 0 degrees
- moved C36 19.9 mm to (136.5, 81.1)
- moved C37 19.9 mm to (138.2, 82.3)
- moved C38 19.9 mm to (132.0, 76.5)
- moved C39 19.9 mm to (133.2, 77.1)
- moved C40 19.9 mm to (136.5, 77.1)
- moved C41 19.9 mm to (126.0, 85.8)
- moved C42 19.9 mm to (139.0, 86.6)
- moved C43 19.9 mm to (125.2, 80.2)
- moved C44 19.9 mm to (127.2, 85.5)
- moved C45 19.9 mm to (135.1, 77.3)
- moved C46 19.9 mm to (136.3, 80.2)
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
Commit message: main_unit/hardware: Rearrange more components, add CAN transceiver
Parts:
- added C48: 100n, Capacitor_SMD:C_0402_1005Metric, F.Cu at (128.5, 133.2)
- added D5: D5V0H1B2LP-7B, Diode_SMD:D_0402_1005Metric, F.Cu at (149.5, 127.4)
- added D6: D5V0H1B2LP-7B, Diode_SMD:D_0402_1005Metric, F.Cu at (143.5, 127.4)
- added J4: 691137710002, 691137710002:691137710002, F.Cu at (146.5, 132.9)
- added R5: 120, Resistor_SMD:R_0805_2012Metric_Pad1.20x1.40mm_HandSolder, F.Cu at (138.7, 132.9)
- added U5: ATA6561-GAQW-N, Package_SO:SOIC-8_3.9x4.9mm_P1.27mm, F.Cu at (133.2, 132.6)
- moved J3 59.2 mm to (158.5, 132.9), turned to 0 degrees
- moved C47 52.5 mm to (168.0, 132.2), turned to 90 degrees
- moved D4 47.6 mm to (161.5, 127.9), turned to 180 degrees
- moved SW1 47.3 mm to (162.8, 82.0), turned to 90 degrees
- moved C1 41.6 mm to (164.7, 125.9), turned to 90 degrees
- moved U2 40.1 mm to (168.0, 125.9), turned to 180 degrees
- moved C2 39.7 mm to (171.7, 125.9), turned to 90 degrees
- moved REF** 21.5 mm to (132.0, 93.2)
- moved C35 5.00 mm to (124.2, 97.2)
- moved C34 5.00 mm to (124.7, 98.5)
- moved J1 5.00 mm to (118.7, 105.0)
- moved R4 4.30 mm to (125.0, 79.4)
- moved R9 4.30 mm to (125.0, 78.4)
- moved C36 4.30 mm to (132.2, 80.4)
- moved C37 4.30 mm to (133.9, 81.7)
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Connections:
- U1 pad 101: unconnected-(U1-PA9-Pad101) -> CAN_STANDBY
Other:
- board outline added: 75 x 65 mm

Commit message: main_unit/hardware: Set up board as 4-layer, add ground and power planes
Parts:
- removed REF**: ESD-Logo_6.6x6mm_SilkScreen, Symbol:ESD-Logo_6.6x6mm_SilkScreen
Routing:
- added copper zone on In2.Cu, net +3V3
- added copper zone on B.Cu, net GND
- added copper zone on F.Cu, net GND
- added copper zone on In1.Cu, net GND
Other:
- copper layers 2 -> 4

Commit message: main_unit/hardware: Route out backlight boost converter
Parts:
- moved R2 1.86 mm to (124.0, 79.0)
- moved C43 1.25 mm to (119.8, 79.5)
- moved R12 1.14 mm to (124.0, 83.0)
- moved R13 1.14 mm to (124.0, 82.0)
- moved R14 1.14 mm to (124.0, 77.0)
- moved R15 1.14 mm to (124.0, 76.0)
- moved R3 1.14 mm to (124.0, 81.0)
- moved R4 1.14 mm to (124.0, 80.0)
- moved R9 1.07 mm to (124.0, 78.0)
- moved C40 0.95 mm to (132.2, 75.5)
- moved R7 0.95 mm to (132.3, 77.8)
- moved C46 0.84 mm to (132.8, 79.2), turned to -90 degrees
- moved C37 0.33 mm to (133.9, 82.0)
- moved R10 0.25 mm to (134.5, 79.5)
- moved R11 0.25 mm to (134.5, 80.5)
Routing:
- net /Display/BACKLIGHT_ANODE: track 0.00 -> 34.8 mm, vias 0 -> 2
- net /Display/BACKLIGHT_CATHODE: track 0.00 -> 34.3 mm
- net LEDCTRL_FAULT: track 0.00 -> 22.7 mm, vias 0 -> 1
- net LEDCTRL_SDA: track 0.00 -> 21.5 mm, vias 0 -> 1
- net LEDCTRL_SCL: track 0.00 -> 19.9 mm, vias 0 -> 1
- net LEDCTRL_DIM_PWM: track 0.00 -> 18.5 mm, vias 0 -> 1
- net Net-(D2-K): track 0.00 -> 16.6 mm
- net GND: track 0.00 -> 15.0 mm, vias 0 -> 5
- net +3V3: track 0.00 -> 15.0 mm, vias 0 -> 2
- net Net-(D1-A): track 0.00 -> 11.0 mm
- net /Display/V18: track 0.00 -> 8.63 mm, vias 0 -> 2
- net Net-(D3-K): track 0.00 -> 8.35 mm, vias 0 -> 2
- net +5V: track 0.00 -> 5.28 mm, vias 0 -> 4
- net Net-(U4-BSTMON): track 0.00 -> 4.79 mm
- net Net-(U4-OUT4): track 0.00 -> 4.78 mm
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- added copper zone on F.Cu, net +3V3
- added copper zone on F.Cu, net +5V
- added copper zone on In2.Cu, net +5V

Commit message: main_unit/hardware: More routing, specifically for CAN and decoupling caps
Parts:
- moved D5 10.1 mm to (140.2, 131.4), turned to -90 degrees
- moved D6 7.70 mm to (140.2, 134.3), turned to 90 degrees
- moved D4 4.16 mm to (164.5, 130.8), turned to -90 degrees
- moved C22 2.09 mm to (141.9, 115.0), turned to 135 degrees
- moved U5 1.78 mm to (131.5, 132.9)
- moved C48 1.78 mm to (126.7, 133.6)
- moved J3 1.66 mm to (158.5, 131.2)
- moved J4 1.62 mm to (146.5, 131.2)
- moved C23 1.58 mm to (145.6, 118.8), turned to -45 degrees
- moved R5 0.98 mm to (137.8, 132.9)
- moved R1 0.11 mm to (139.4, 100.0)
Routing:
- net +3V3: track 15.0 -> 62.8 mm, vias 2 -> 4
- net /CANBus/CANH: track 0.00 -> 17.1 mm
- net /CANBus/CANL: track 0.00 -> 11.2 mm
- net Net-(U1-PH1): track 0.00 -> 9.45 mm
- net Net-(U1-PC15): track 0.00 -> 7.04 mm
- net Net-(U1-PC14): track 0.00 -> 7.00 mm
- net Net-(U1-PH0): track 0.00 -> 6.67 mm
- net GND: track 15.0 -> 20.5 mm, vias 5 -> 10
- net Net-(C17-Pad1): track 0.00 -> 2.22 mm
- net Net-(C18-Pad1): track 0.00 -> 2.05 mm
- net +5V: track 5.28 -> 7.08 mm
- net NRST: track 0.00 -> 1.64 mm
- net Net-(U1-BOOT0): track 0.00 -> 1.61 mm
Other:
- board text added: "+5V"
- board text added: "CANH"
- board text added: "CANL"
- board text added: "GND"

Commit message: main_unit/hardware: Route out SDRAM (without length matching)
Routing:
- net SDRAM_NBL1: track 0.00 -> 52.5 mm, vias 0 -> 2
- net SDRAM_SDCKE0: track 0.00 -> 51.4 mm, vias 0 -> 2
- net SDRAM_A5: track 0.00 -> 49.8 mm, vias 0 -> 2
- net SDRAM_A4: track 0.00 -> 48.7 mm, vias 0 -> 2
- net SDRAM_NBL0: track 0.00 -> 46.5 mm, vias 0 -> 2
- net SDRAM_SDNCAS: track 0.00 -> 41.7 mm, vias 0 -> 2
- net SDRAM_A0: track 0.00 -> 40.1 mm, vias 0 -> 2
- net SDRAM_A1: track 0.00 -> 39.4 mm, vias 0 -> 2
- net SDRAM_A2: track 0.00 -> 38.7 mm, vias 0 -> 2
- net SDRAM_A3: track 0.00 -> 37.9 mm, vias 0 -> 2
- net SDRAM_BA1: track 0.00 -> 36.1 mm, vias 0 -> 2
- net SDRAM_BA0: track 0.00 -> 34.2 mm, vias 0 -> 2
- net SDRAM_D12: track 0.00 -> 33.6 mm, vias 0 -> 2
- net SDRAM_D11: track 0.00 -> 33.3 mm, vias 0 -> 2
- net SDRAM_D15: track 0.00 -> 33.0 mm, vias 0 -> 2
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
Commit message: main_unit/hardware: Route out control signals for LCD
Routing:
- net LCD_VSYNC: track 0.00 -> 42.2 mm, vias 0 -> 2
- net LCD_CLK: track 0.00 -> 42.2 mm
- net LCD_HSYNC: track 0.00 -> 42.1 mm, vias 0 -> 2
- net LCD_DE: track 0.00 -> 32.8 mm
- net LCD_CS: track 0.00 -> 26.5 mm, vias 0 -> 2
- net LCDSPI_SDA: track 0.00 -> 26.3 mm
- net LCDSPI_SCK: track 0.00 -> 25.5 mm
- net LCD_G3: track 0.00 -> 19.9 mm, vias 0 -> 2

Commit message: main_unit/hardware: Keep trying to find good way of routing out display
Routing:
- net LCD_B4: track 0.00 -> 51.3 mm, vias 0 -> 4
- net LCD_B3: track 0.00 -> 49.9 mm, vias 0 -> 2
- net LCD_B2: track 0.00 -> 29.4 mm, vias 0 -> 2
- net LCD_G3: track 19.9 -> 0.00 mm, vias 2 -> 0
