File: main_unit/hardware/display.kicad_sch (KiCad schematic)
At the start: 0 parts

Commit message: main_unit/hardware: Add in display connector, expand LTDC to RGB888 (fixes pin error)
Parts:
- added J1: 62684-402100ALF, 62684-402100ALF:AMPHENOL_62684-402100ALF, symbol 62684-402100ALF:62684-402100ALF
Connections:
- new net +3V3: J1.05
- new net BACKLIGHT_ANODE: J1.01
- new net BACKLIGHT_CATHODE: J1.02, J1.03
- new net GND: J1.04, J1.34, J1.40, J1.S1 (SHIELD), J1.S2 (SHIELD__1)
- new net LCDSPI_SCK: J1.10
- new net LCDSPI_SDA: J1.09
- new net LCD_B2: J1.16
- new net LCD_B3: J1.17
- new net LCD_B4: J1.18
- new net LCD_B5: J1.19
- new net LCD_B6: J1.20
- new net LCD_B7: J1.21
- new net LCD_CLK: J1.12
- new net LCD_CS: J1.11
- new net LCD_DE: J1.13
- new net LCD_G2: J1.22
- new net LCD_G3: J1.23
- new net LCD_G4: J1.24
- new net LCD_G5: J1.25
- new net LCD_G6: J1.26
- new net LCD_G7: J1.27
- new net LCD_HSYNC: J1.15
- new net LCD_R2: J1.28
- new net LCD_R3: J1.29
- new net LCD_R4: J1.30
- new net LCD_R5: J1.31
- new net LCD_R6: J1.32
- new net LCD_R7: J1.33
- new net LCD_RST: J1.06
- new net LCD_VSYNC: J1.14
- no-connect marks 0 -> 7
Other:
- note added: "Display: ER-TFT062-1 Datasheet: https://www.buydisplay.com/download/manual/ER-TFT062-1_Datasheet.pdf Purchase: https://www.buydisplay.com/bar-type-6-2-inch-360x960-ips-tft-lcd-display-spi-rgb-interface"

Commit message: main_unit/hardware: Add capacitors for display
Parts:
- added C34: 1u, Capacitor_SMD:C_0603_1608Metric, symbol Device:C_Small
- added C35: 100n, Capacitor_SMD:C_0402_1005Metric, symbol Device:C_Small
Connections:
- net +3V3: now also C34.1, C35.1
- net GND: now also C34.2, C35.2

Commit message: main_unit/hardware: Add in backlight boost converter & LED driver skeleton from MAX chip datasheet
Parts:
- added C36, C39: 100n, Capacitor_SMD:C_0402_1005Metric, symbol Device:C_Small
- added C37: 2u2, Capacitor_SMD:C_0603_1608Metric, symbol Device:C_Small
- added C38: 1u, Capacitor_SMD:C_0603_1608Metric, symbol Device:C_Small
- added C40: COMP, Capacitor_SMD:C_0603_1608Metric, symbol Device:C_Small
- added C41: COUT, Capacitor_SMD:C_0603_1608Metric, symbol Device:C_Small
- added C42: CIN, Capacitor_SMD:C_0603_1608Metric, symbol Device:C_Small
- added D1: D, symbol Device:D
- added D2, D3: D_Small, symbol Device:D_Small
- added L1: L, symbol Device:L
- added Q1: NMOS, symbol Simulation_SPICE:NMOS
- added R10, R11, R12, R13, R14, R2, R3, R4, R5, R6: 10k, Resistor_SMD:R_0402_1005Metric, symbol Device:R_Small
- added R7: RT, Resistor_SMD:R_0402_1005Metric, symbol Device:R_Small
- added R8: COMP, Resistor_SMD:R_0402_1005Metric, symbol Device:R_Small
- added R9: SET, Resistor_SMD:R_0402_1005Metric, symbol Device:R_Small
- added U4: MAX25512ATG/V+T, Package_DFN_QFN:WQFN-24-1EP_4x4mm_P0.5mm_EP2.45x2.45mm_ThermalVias, symbol MAX25512ATG/V+T:MAX25512ATG_V+T
Connections:
- net +3V3: now also R2.1, R3.1, R4.1
- net BACKLIGHT_ANODE: now also C41.1, D1.1 (K), R10.1
- net BACKLIGHT_CATHODE: now also U4.11 (OUT1)
- net GND: now also C36.2, C37.2, C38.2, C39.2, C40.2, C41.2, C42.2, D2.2 (A), R11.2, R12.2, R13.2, R14.2, R6.1, R7.2, R9.2, U4.10 (GND), U4.15 (LEDGND), U4.22 (PGND), U4.23 (PGND), U4.25 (EP)
- new net: R8.1, U4.7 (COMP)
- new net: C40.1, R8.2
- new net: R5.1, R6.2, U4.8 (RSDT)
- new net: D1.2 (A), L1.2, U4.1 (DRAIN), U4.2 (DRAIN)
- new net: R7.1, U4.6 (RT)
- new net: D3.1 (K), Q1.2 (G), U4.4 (NGATE)
- new net: C42.1, D2.1 (K), D3.2 (A), L1.1, Q1.3 (S)
- new net: R12.1, U4.21 (OUT4)
- new net: R10.2, R11.1, U4.5 (BSTMON)
- new net: R13.1, U4.20 (OUT3)
- new net: R14.1, U4.12 (OUT2)
- new net: R9.1, U4.13 (ISET)
- new net +5V: C36.1, C37.1, Q1.1 (D), U4.24 (EN), U4.3 (IN)
- new net LEDCTRL_DIM_PWM: U4.17 (DIM)
- new net LEDCTRL_FAULT: R2.2, U4.16 (FLTB)
- new net LEDCTRL_SCL: R3.2, U4.19 (SCL)
- new net LEDCTRL_SDA: R4.2, U4.18 (SDA)
- new net V18: C38.1, C39.1, R5.2, U4.14 (TEMP), U4.9 (V18)
Other:
- note added: "Backlight Boost Converter & Driver"
- note added: "Display Connector"
- moved on the sheet: C34, C35, J1

Commit message: main_unit/hardware: Fill out LED driver component values except for compensation circuit
Parts:
- removed C42: CIN, Capacitor_SMD:C_0603_1608Metric, symbol Device:C_Small
- removed R5, R6: 10k, Resistor_SMD:R_0402_1005Metric, symbol Device:R_Small
- added C42, C43: 47u, 865080342006:WCAP-ASLI_5X5.5_DXL_, symbol Device:C_Polarized_Small
- added C44: 100n, Capacitor_SMD:C_0402_1005Metric, symbol Device:C_Small
- added R15: 10k, Resistor_SMD:R_0402_1005Metric, symbol Device:R_Small
- C41: value COUT -> 10u
- D1: value D -> BAT54T1G; footprint (none) -> Diode_SMD:D_SOD-123
- D2, D3: value D_Small -> BAT54T1G; footprint (none) -> Diode_SMD:D_SOD-123
- L1: value L -> 22u; footprint (none) -> Inductor_SMD:L_Taiyo-Yuden_NR-40xx
- Q1: value NMOS -> 2N7002BK,215; footprint (none) -> Package_TO_SOT_SMD:SOT-23-3
- R11: value 10k -> 1k
- R7: value RT -> 15k
- R9: value SET -> 15k
Connections:
- net BACKLIGHT_ANODE: now also C43.1, C44.1
- net BACKLIGHT_CATHODE: now also R15.1
- net GND: now also C42.2, C43.2, C44.2, R15.2
- net V18: now also U4.8 (RSDT)
- net at D2.1 (K), D3.2 (A), L1.1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: now also C42.1
Other:
- note added: "15k -> 1.76MHz"
- note added: "Min inductance: ~20uH Min current: 330mA See "Applications Information" in datasheet Part chosen: NRS4018T220MDGJ"
- note added: "P/N: 865080342006"
- note added: "R_{SET} = 1500/0.1A = 15k"
- note added: "V_{OUT_BSTMON} = 0.95*(1+10k/1k) = 10.45V"
- moved on the sheet: C38, C39, C40, D1, D2, D3, L1, Q1, R10, R11, R12, R13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

Commit message: main_unit/hardware: Fill in compensation circuit values
Parts:
- added C45: 2n7, Capacitor_SMD:C_0201_0603Metric, symbol Device:C_Small
- C40: value COMP -> 1u; footprint Capacitor_SMD:C_0603_1608Metric -> Capacitor_SMD:C_0805_2012Metric
- R8: value COMP -> 10k
Connections:
- net GND: now also C45.2
- net at R8.1, U4.7 (COMP): now also C45.1
Other:
- note added: "Min inductance: ~11uH Min current: 330mA See "Applications Information" in datasheet Part chosen: NRS4018T220MDGJ"
- note removed: "Min inductance: ~20uH Min current: 330mA See "Applications Information" in datasheet Part chosen: NRS4018T220MDGJ"
- moved on the sheet: C36, C37, C38, C39, C40, C41, C42, C43, C44, D1, D2, D3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

Commit message: main_unit/hardware: Add in extra capacitor for BOSTMON, move things around slightly for MAX chip according to datasheet recommendations
Parts:
- added C46: 47p, Capacitor_SMD:C_0201_0603Metric, symbol Device:C_Small
Connections:
- net GND: now also C46.2
- net at R10.2, R11.1, U4.5 (BSTMON): now also C46.1
Changed lines of the file:
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@@
 	(text "V_{OUT_BSTMON} = 0.95*(1+10k/1k) = 10.45V"
 		(exclude_from_sim no)
-		(at 267.97 71.628 90)
+		(at 278.638 72.136 90)
 		(effects
 			(font
@@
 	)
 	(junction
+		(at 260.35 78.74)
+		(diameter 0)
+		(color 0 0 0 0)
+	)
+	(junction
 		(at 212.09 55.88)
 		(diameter 0)
@@
 	(wire
 		(pts
+			(xy 260.35 71.12) (xy 267.97 71.12)
+		)
+		(stroke
+			(width 0)
+			(type default)
+		)
+	)
+	(wire
+		(pts
 			(xy 143.51 63.5) (xy 143.51 64.77)
 		)
@@
 	(wire
 		(pts
+			(xy 267.97 72.39) (xy 267.97 71.12)
+		)
+		(stroke
+			(width 0)
+			(type default)
+		)
+	)
+	(wire
+		(pts
+			(xy 260.35 78.74) (xy 260.35 80.01)
+		)
+		(stroke
+			(width 0)
+			(type default)
+		)
+	)
+	(wire
+		(pts
 			(xy 160.02 92.71) (xy 171.45 92.71)
 		)
@@
 	(wire
 		(pts
-			(xy 260.35 77.47) (xy 260.35 80.01)
+			(xy 260.35 77.47) (xy 260.35 78.74)
 		)
 		(stroke
@@
 	(wire
 		(pts
+			(xy 260.35 78.74) (xy 267.97 78.74)
+		)
+		(stroke
+			(width 0)
+			(type default)
+		)
+	)
+	(wire
+		(pts
 			(xy 246.38 104.14) (xy 246.38 105.41)
 		)
@@
 	(wire
 		(pts
+			(xy 267.97 77.47) (xy 267.97 78.74)
+		)
+		(stroke
+			(width 0)
+			(type default)
+		)
+	)
+	(wire
+		(pts
 			(xy 209.55 55.88) (xy 209.55 60.96)
 		)
@@
 					(unit 1)
 				)
+			)
+		)
+	)
+	(symbol
+		(lib_id "Device:C_Small")
+		(at 267.97 74.93 0)
+		(unit 1)
+		(exclude_from_sim no)
+		(in_bom yes)
+		(on_board yes)
+		(dnp no)
+		(fields_autoplaced yes)
+		(property "Reference" "C46"
+			(at 270.51 73.6662 0)
+			(effects
+				(font
+					(size 1.27 1.27)
+				)
+				(justify left)
+			)
+		)
+		(property "Value" "47p"
+			(at 270.51 76.2062 0)
+			(effects
+				(font
+					(size 1.27 1.27)
+				)
+				(justify left)
+			)
+		)
+		(property "Footprint" "Capacitor_SMD:C_0201_0603Metric"
+			(at 267.97 74.93 0)
+			(effects
+				(font
+					(size 1.27 1.27)
+				)
+				(hide yes)
+			)
+		)
+		(property "Datasheet" "~"
+			(at 267.97 74.93 0)
+			(effects
+				(font
+					(size 1.27 1.27)
+				)
+				(hide yes)
+			)
+		)
+		(property "Description" "Unpolarized capacitor, small symbol"
+			(at 267.97 74.93 0)
+			(effects
+				(font
+					(size 1.27 1.27)
+				)
+				(hide yes)
+			)
+		)
+		(pin "2"
+		)
+		(pin "1"
+		)
+		(instances
+			(project ""
+				(path "/c1e2a568-b99f-4357-b0bb-65969671b711/8d15cbf3-f8cd-48ab-b3c4-b2dcdd94b087"
+					(reference "C46")
+					(unit 1)
+				)
