File: main_unit/hardware/untitled.kicad_sch (KiCad schematic)
At the start: 0 parts

Commit message: main_unit/hardware: Add in input power filtering and ST-Link connector
Parts:
- added J2: Conn_02x07_Odd_Even, FTSH-107-01-L-DV-K-A:SAMTEC_FTSH-107-01-L-DV-K-A, symbol Connector_Generic:Conn_02x07_Odd_Even
Connections:
- new net +3V3: J2.3 (Pin_3)
- new net DBG_JTDO_SWO: J2.8 (Pin_8)
- new net DBG_JTMS_JTDI: J2.10 (Pin_10)
- new net DBG_JTMS_SWCLK: J2.6 (Pin_6)
- new net DBG_JTMS_SWDIO: J2.4 (Pin_4)
- new net GND: J2.11 (Pin_11), J2.5 (Pin_5), J2.7 (Pin_7)
- new net NRST: J2.12 (Pin_12)
- new net UART_RX: J2.13 (Pin_13)
- new net UART_TX: J2.14 (Pin_14)
- no-connect marks 0 -> 3
Other:
- note added: "ST-Link"

Commit message: main_unit/hardware: Add more TVS diodes
Parts:
- added D5: DF2S5.6FS,L3M, symbol Device:D_TVS
Changed lines of the file:
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@@
+	)
+	(symbol
+		(lib_id "Device:D_TVS")
+		(at 123.19 92.71 90)
+		(unit 1)
+		(exclude_from_sim no)
+		(in_bom yes)
+		(on_board yes)
+		(dnp no)
+		(fields_autoplaced yes)
+		(property "Reference" "D5"
+			(at 125.73 91.4399 90)
+			(effects
+				(font
+					(size 1.27 1.27)
+				)
+				(justify right)
+			)
+		)
+		(property "Value" "DF2S5.6FS,L3M"
+			(at 125.73 93.9799 90)
+			(effects
+				(font
+					(size 1.27 1.27)
+				)
+				(justify right)
+			)
+		)
+		(property "Footprint" ""
+			(at 123.19 92.71 0)
+			(effects
+				(font
+					(size 1.27 1.27)
+				)
+				(hide yes)
+			)
+		)
+		(property "Datasheet" "~"
+			(at 123.19 92.71 0)
+			(effects
+				(font
+					(size 1.27 1.27)
+				)
+				(hide yes)
+			)
+		)
+		(property "Description" "Bidirectional transient-voltage-suppression diode"
+			(at 123.19 92.71 0)
+			(effects
+				(font
+					(size 1.27 1.27)
+				)
+				(hide yes)
+			)
+		)
+		(pin "1"
+		)
+		(pin "2"
+		)
+		(instances
+			(project ""
+				(path "/c1e2a568-b99f-4357-b0bb-65969671b711/1066afca-0a6b-4ef0-a47e-6cb6f4f4f270"
+					(reference "D5")
+					(unit 1)
+				)
+			)
+		)
 	)
 	(symbol
