File: can-module/can-module.kicad_sch (KiCad schematic)
At the start: 0 parts

Commit message: can-module: Add PIC32 mcu library to project
Parts:
- added IC1: PIC32CM1216JH01048-I_U5B, QFN50P700X700X90-49N-D, symbol PIC32CM1216JH01048-I/U5B:PIC32CM1216JH01048-I_U5B
Changed lines of the file:
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@@
 	(generator_version "9.0")
 	(paper "A4")
+	(symbol
+		(lib_id "PIC32CM1216JH01048-I/U5B:PIC32CM1216JH01048-I_U5B")
+		(at 127 92.71 0)
+		(unit 1)
+		(exclude_from_sim no)
+		(in_bom yes)
+		(on_board yes)
+		(dnp no)
+		(property "Reference" "IC1"
+			(at 183.388 72.136 0)
+			(effects
+				(font
+					(size 1.27 1.27)
+				)
+			)
+		)
+		(property "Value" "PIC32CM1216JH01048-I_U5B"
+			(at 183.388 74.676 0)
+			(effects
+				(font
+					(size 1.27 1.27)
+				)
+			)
+		)
+		(property "Footprint" "QFN50P700X700X90-49N-D"
+			(at 168.91 169.85 0)
+			(effects
+				(font
+					(size 1.27 1.27)
+				)
+				(justify left top)
+				(hide yes)
+			)
+		)
+		(property "Datasheet" "https://ww1.microchip.com/downloads/aemDocuments/documents/MCU32/ProductDocuments/DataSheets/PIC32CM-JH00-JH01-Family-Data-Sheet-DS60001632.pdf"
+			(at 168.91 269.85 0)
+			(effects
+				(font
+					(size 1.27 1.27)
+				)
+				(justify left top)
+				(hide yes)
+			)
+		)
+		(property "Description" "Microchip Technology 5V Cortex M0+, 128KB Flash, 48Pin, VQFN, CAN-FD, 85C Temp"
+			(at 127 92.71 0)
+			(effects
+				(font
+					(size 1.27 1.27)
+				)
+				(hide yes)
+			)
+		)
+		(property "Height" "0.9"
+			(at 168.91 469.85 0)
+			(effects
+				(font
+					(size 1.27 1.27)
+				)
+				(justify left top)
+				(hide yes)
+			)
+		)
+		(property "Manufacturer_Name" "Microchip"
+			(at 168.91 569.85 0)
+			(effects
+				(font
+					(size 1.27 1.27)
+				)
+				(justify left top)
+				(hide yes)
+			)
+		)
+		(property "Manufacturer_Part_Number" "PIC32CM1216JH01048-I/U5B"
+			(at 168.91 669.85 0)
+			(effects
+				(font
+					(size 1.27 1.27)
+				)
+				(justify left top)
+				(hide yes)
+			)
+		)
+		(property "Mouser Part Number" ""
+			(at 168.91 769.85 0)
+			(effects
+				(font
+					(size 1.27 1.27)
+				)
+				(justify left top)
+				(hide yes)
+			)
+		)
+		(property "Mouser Price/Stock" ""
+			(at 168.91 869.85 0)
+			(effects
+				(font
+					(size 1.27 1.27)
+				)
+				(justify left top)
+				(hide yes)
+			)
+		)
+		(property "Arrow Part Number" ""
+			(at 168.91 969.85 0)
+			(effects
+				(font
+					(size 1.27 1.27)
+				)
+				(justify left top)
+				(hide yes)
+			)
+		)
+		(property "Arrow Price/Stock" ""
+			(at 168.91 1069.85 0)
+			(effects
+				(font
+					(size 1.27 1.27)
+				)
+				(justify left top)
+				(hide yes)
+			)
+		)
+		(pin "17"
+		)
+		(pin "35"
+		)
+		(pin "12"
+		)
+		(pin "8"
+		)
+		(pin "42"
+		)
+		(pin "10"
+		)
+		(pin "38"
+		)
+		(pin "40"
+		)
+		(pin "36"
+		)
+		(pin "31"
+		)
+		(pin "49"
+		)
+		(pin "39"
+		)
+		(pin "21"
+		)
+		(pin "20"
+		)
+		(pin "2"
+		)
+		(pin "19"
+		)
+		(pin "7"
+		)
+		(pin "1"
+		)
+		(pin "26"
+		)
+		(pin "25"
+		)
+		(pin "22"
+		)
+		(pin "28"
+		)
+		(pin "6"
+		)
+		(pin "34"
+		)
+		(pin "32"
+		)
+		(pin "24"
+		)
+		(pin "15"
+		)
+		(pin "48"
+		)
+		(pin "4"
+		)
+		(pin "14"
+		)
+		(pin "44"
+		)
+		(pin "13"
+		)
+		(pin "33"
+		)
+		(pin "3"
+		)
+		(pin "27"
+		)
+		(pin "11"
+		)
+		(pin "16"
+		)
+		(pin "23"
+		)
+		(pin "47"
+		)
+		(pin "30"
+		)
+		(pin "18"
+		)
+		(pin "45"
+		)
+		(pin "37"
+		)
+		(pin "46"
+		)
+		(pin "5"
+		)
+		(pin "29"
+		)
+		(pin "43"
+		)
+		(pin "41"
+		)
+		(pin "9"
+		)
+		(instances
+			(project ""
+				(path "/40cb4209-4f7f-4a38-b0f0-dee54a92ee91"
+					(reference "IC1")
+					(unit 1)
+				)
+			)
+		)
+	)
 	(sheet_instances
 		(path "/"

Commit message: can-module: Add decoupling capacitors for mcu
Parts:
- added C1, C2, C3, C4: 10u, Capacitor_SMD:C_0402_1005Metric, symbol Device:C
- added C5, C6, C7, C8, C9: 100n, Capacitor_SMD:C_0201_0603Metric, symbol Device:C_Small
- IC1: footprint QFN50P700X700X90-49N-D -> PIC32CM1216JH01048-I/U5B:QFN50P700X700X90-49N-D
Connections:
- net +5V: now reaches IC1.17 (VDDIO_1)
- net +5V: now also IC1.36 (VDDIO_2), IC1.43 (VDDCORE), IC1.44 (VDDIN), IC1.6 (AVDD), C1.1, C2.1, C3.1, C4.1, C5.1, C6.1, C7.1, C8.1, C9.1
- net GND: now reaches IC1.18 (GND_1)
- net GND: now also IC1.35 (GND_2), IC1.42 (GND_3), IC1.49 (EP), IC1.5 (AVSS), C1.2, C2.2, C3.2, C4.2, C5.2, C6.2, C7.2, C8.2, C9.2
Other:
- note added: "1x bulk cap for each AVDD, VDDIO, VDDIN, VDDCORE"
- note added: "1x decoupling cap for each power pin"

Commit message: can-module: Add reset RC circuit
Parts:
- added C10: 100n, Capacitor_SMD:C_0201_0603Metric, symbol Device:C_Small
- added R1: 100k, Resistor_SMD:R_0201_0603Metric, symbol Device:R_Small
Connections:
- net +5V: now also R1.1
- net GND: now also C10.2
- net at IC1.40 (~{RESET}): now also C10.1, R1.2

Commit message: can-module: Route power, gnd, and swd pins to test points
Parts:
- added R2: 1k, Resistor_SMD:R_0201_0603Metric, symbol Device:R_Small
- added TP1, TP2, TP3, TP4: TestPoint, TestPoint:TestPoint_Pad_D1.0mm, symbol Connector:TestPoint
Connections:
- net +5V: now also R2.2, TP1.1
- net GND: now also TP2.1
- net at IC1.45 (PA30_SWCLK): now also R2.1, TP4.1
- net at IC1.46 (PA31_SWDIO): now also TP3.1

Commit message: can-module: Add ATA6560 CAN transceiver
Parts:
- added C11: 100n, Capacitor_SMD:C_0201_0603Metric, symbol Device:C_Small
- added U1: ATA6560-GBQW-N, VDFN8_3X3_MCH, symbol ATA6560-GBQW-N:ATA6560-GBQW-N
Connections:
- net +5V: now also C11.1, U1.3 (VCC)
- net GND: now also C11.2, U1.2 (GND), U1.9 (EPAD)
- net CAN_NSIL: now reaches IC1.31 (PA22)
- net CAN_NSIL: now also U1.5 (NSIL)
- net CAN_STBY: now reaches IC1.32 (PA23)
- net CAN_STBY: now also U1.8 (STBY)
- net CAN_TX: now reaches IC1.33 (PA24)
- net CAN_TX: now also U1.1 (TXD)
- net CAN_RX: now reaches IC1.34 (PA25)
- net CAN_RX: now also U1.4 (RXD)
- new net CANH: U1.7 (CANH)
- new net CANL: U1.6 (CANL)
Other:
- moved on the sheet: C1, C10, C2, C3, C4, C5, C6, C7, C8, C9, IC1, R1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

Commit message: can-module: Move pins around, select GPIO pins, add test points for GPIOs
Parts:
- added J1, J2: Conn_01x04_Socket, symbol Connector:Conn_01x04_Socket
Connections:
- net CAN_NSIL: now also IC1.32 (PA23); no longer IC1.31 (PA22)
- net CAN_STBY: now also IC1.31 (PA22); no longer IC1.32 (PA23)
- net at IC1.10 (PA05): now also J1.1 (Pin_1)
- net at IC1.13 (PA08): now also J2.4 (Pin_4)
- net at IC1.14 (PA09): now also J2.3 (Pin_3)
- net at IC1.15 (PA10): now also J2.2 (Pin_2)
- net at IC1.16 (PA11): now also J2.1 (Pin_1)
- net at IC1.3 (PA02): now also J1.4 (Pin_4)
- net at IC1.4 (PA03): now also J1.3 (Pin_3)
- net at IC1.9 (PA04): now also J1.2 (Pin_2)
- no-connect marks 0 -> 24

Commit message: can-module: Route out all signals
Parts:
- added C12: 10u, Capacitor_SMD:C_0402_1005Metric, symbol Device:C_Small
- added J3: Conn_01x04_Socket, Connector_PinHeader_1.00mm:PinHeader_1x04_P1.00mm_Vertical, symbol Connector:Conn_01x04_Socket
- added JP2: Jumper_2_Small_Open, Resistor_SMD:R_0201_0603Metric, symbol Jumper:Jumper_2_Small_Open
- added R3: 120, Resistor_SMD:R_0201_0603Metric, symbol Device:R
- J1, J2: footprint (none) -> Connector_PinHeader_1.00mm:PinHeader_1x04_P1.00mm_Vertical
- U1: footprint VDFN8_3X3_MCH -> ATA6560-GBQW-N:VDFN8_3X3_MCH
Connections:
- net +5V: now also C12.1, J3.4 (Pin_4)
- net CANH: now also J3.2 (Pin_2), JP2.1 (A)
- net CANL: now also J3.1 (Pin_1), R3.1
- net GND: now also C12.2, J3.3 (Pin_3)
- net at J2.1 (Pin_1): now also IC1.14 (PA09); no longer IC1.16 (PA11)
- net at J2.2 (Pin_2): now also IC1.13 (PA08); no longer IC1.15 (PA10)
- net at J2.3 (Pin_3): now also IC1.12 (PA07); no longer IC1.14 (PA09)
- net at J2.4 (Pin_4): now also IC1.11 (PA06); no longer IC1.13 (PA08)
- new net: JP2.2 (B), R3.2
- no-connect marks 24 -> 22
Other:
- moved on the sheet: J2

Commit message: can-module: Rearrange components, update constraints for copper to board edge
Parts:
- removed TP1, TP2: TestPoint, TestPoint:TestPoint_Pad_D1.0mm, symbol Connector:TestPoint
- JP2: footprint Resistor_SMD:R_0201_0603Metric -> Jumper:SolderJumper-2_P1.3mm_Open_Pad1.0x1.5mm
