File: can-module/can-module.kicad_sch (KiCad schematic)
At the start: 23 parts, among them IC1 PIC32CM1216JH01048-I_U5B, J1 Conn_01x04_Socket, J2 Conn_01x04_Socket, J3 Conn_01x04_Socket, U1 ATA6560-GBQW-N

Commit message: can-module: Update ATA6560 schematic to have filled background
Parts:
- J1, J2, J3: footprint Connector_PinHeader_1.00mm:PinHeader_1x04_P1.00mm_Vertical -> Conn01x04:01x04_1mm
- U1: footprint ATA6560-GBQW-N:VDFN8_3X3_MCH -> VDFN8_3X3_MCH
Changed lines of the file:
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@@
 			)
 		)
-		(property "Footprint" "Connector_PinHeader_1.00mm:PinHeader_1x04_P1.00mm_Vertical"
+		(property "Footprint" "Conn01x04:01x04_1mm"
 			(at 67.31 147.32 0)
 			(effects
@@
 			)
 		)
-		(property "Footprint" "Connector_PinHeader_1.00mm:PinHeader_1x04_P1.00mm_Vertical"
+		(property "Footprint" "Conn01x04:01x04_1mm"
 			(at 182.88 33.02 0)
 			(effects
@@
 			)
 		)
-		(property "Footprint" "Connector_PinHeader_1.00mm:PinHeader_1x04_P1.00mm_Vertical"
+		(property "Footprint" "Conn01x04:01x04_1mm"
 			(at 67.31 127 0)
 			(effects
@@
 			)
 		)
-		(property "Footprint" "ATA6560-GBQW-N:VDFN8_3X3_MCH"
+		(property "Footprint" "VDFN8_3X3_MCH"
 			(at 212.09 97.79 0)
 			(effects

Commit message: can-module: Add text labels to schematic
Other:
- note added: "CAN Transceiver"
- note added: "Decoupling Capacitors"
- note added: "GPIO Headers"
- note added: "Main connector"
- note added: "PIC32 MCU"
- moved on the sheet: C1, C10, C11, C12, C2, C3, C4, C5, C6, C7, C8, C9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
