File: can-module/can-module.kicad_pcb (KiCad board)
At the start: 2 copper layers, 17 parts, among them IC1 PIC32CM1216JH01048-I_U5B

Commit message: can-module: Add ATA6560 CAN transceiver
Parts:
- added C11: 100n, Capacitor_SMD:C_0201_0603Metric, F.Cu at (137.0, 52.9)
- added U1: ATA6560-GBQW-N, ATA6560-GBQW-N:VDFN8_3X3_MCH, F.Cu at (139.6, 52.3)
- moved R2 23.9 mm to (127.8, 48.0)
- moved R1 16.4 mm to (123.2, 52.2), turned to 90 degrees
- moved C10 15.5 mm to (124.0, 52.2), turned to 90 degrees
- moved C9 15.1 mm to (127.8, 56.2)
- moved C2 12.3 mm to (118.8, 54.2), turned to 180 degrees
- moved C1 11.8 mm to (118.8, 53.2), turned to 180 degrees
- moved C6 9.29 mm to (122.6, 54.0), turned to 90 degrees
- moved C8 8.93 mm to (122.0, 64.0), turned to -90 degrees
- moved C5 7.30 mm to (121.8, 54.0), turned to 90 degrees
- moved C4 5.80 mm to (118.8, 64.8), turned to 180 degrees
- moved C3 4.84 mm to (118.8, 63.8), turned to 180 degrees
- moved TP1 4.25 mm to (119.8, 48.0)
- moved TP2 4.25 mm to (121.8, 48.0)
- moved TP3 4.25 mm to (123.8, 48.0)
- moved TP4 4.25 mm to (125.8, 48.0)
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Connections:
- IC1 pad 31: unconnected-(IC1-PA22-Pad31) -> CAN_NSIL
- IC1 pad 32: unconnected-(IC1-PA23-Pad32) -> CAN_STBY
- IC1 pad 33: unconnected-(IC1-PA24-Pad33) -> CAN_TX
- IC1 pad 34: unconnected-(IC1-PA25-Pad34) -> CAN_RX

Commit message: can-module: Add footprint to ATA6560, arrange so it is close to the MCU
Parts:
- moved U1 12.6 mm to (129.0, 59.2), turned to -90 degrees
- moved R2 9.03 mm to (121.0, 54.0), turned to -90 degrees
- moved C11 8.29 mm to (129.4, 56.2), turned to 0 degrees
- moved TP1 5.13 mm to (116.2, 51.8)
- moved TP2 5.13 mm to (118.2, 51.8)
- moved TP3 5.13 mm to (120.2, 51.8)
- moved TP4 5.13 mm to (122.2, 51.8)
- moved C10 1.77 mm to (124.2, 54.0)
- moved R1 1.77 mm to (123.5, 54.0)

Commit message: can-module: Add power and gnd planes
Parts:
- TP1, TP2, TP3, TP4: moved to B.Cu
- moved TP1 9.76 mm to (125.8, 54.0), turned to 180 degrees
- moved TP2 5.94 mm to (123.8, 54.0), turned to 180 degrees
- moved TP4 3.36 mm to (119.8, 54.0), turned to 180 degrees
- moved TP3 2.70 mm to (121.8, 54.0), turned to 180 degrees
- moved C1 2.37 mm to (117.5, 55.2)
- moved C2 2.37 mm to (117.5, 56.2)
- moved C3 2.37 mm to (117.5, 61.8)
- moved C4 2.37 mm to (117.5, 62.8)
- moved R1 1.25 mm to (124.8, 54.0)
- moved C10 0.25 mm to (124.0, 54.0)
Routing:
- net GND: track 0.00 -> 16.8 mm, vias 0 -> 9
- net CAN_TX: track 0.00 -> 4.71 mm, vias 0 -> 3
- net Net-(IC1-PA30_SWCLK): track 0.00 -> 4.24 mm, vias 0 -> 2
- net +5V: track 0.00 -> 3.08 mm
- net Net-(IC1-PA31_SWDIO): track 0.00 -> 2.86 mm, vias 0 -> 1
- net Net-(IC1-~{RESET}): track 0.00 -> 2.25 mm
- net CAN_RX: track 0.00 -> 2.01 mm
- added copper zone on F.Cu, net +5V
- added copper zone on B.Cu, net GND

Commit message: can-module: Move pins around, select GPIO pins, add test points for GPIOs
Parts:
- added TP10: TestPoint, TestPoint:TestPoint_Pad_D1.0mm, F.Cu at (115.2, 62.2)
- added TP11: TestPoint, TestPoint:TestPoint_Pad_D1.0mm, B.Cu at (115.2, 58.2)
- added TP12: TestPoint, TestPoint:TestPoint_Pad_D1.0mm, B.Cu at (115.2, 56.2)
- added TP5: TestPoint, TestPoint:TestPoint_Pad_D1.0mm, B.Cu at (115.2, 62.2)
- added TP6: TestPoint, TestPoint:TestPoint_Pad_D1.0mm, B.Cu at (115.2, 60.2)
- added TP7: TestPoint, TestPoint:TestPoint_Pad_D1.0mm, F.Cu at (115.2, 56.2)
- added TP8: TestPoint, TestPoint:TestPoint_Pad_D1.0mm, F.Cu at (115.2, 58.2)
- added TP9: TestPoint, TestPoint:TestPoint_Pad_D1.0mm, F.Cu at (115.2, 60.2)
Connections:
- IC1 pad 10: unconnected-(IC1-PA05-Pad10) -> Net-(IC1-PA05)
- IC1 pad 13: unconnected-(IC1-PA08-Pad13) -> Net-(IC1-PA08)
- IC1 pad 14: unconnected-(IC1-PA09-Pad14) -> Net-(IC1-PA09)
- IC1 pad 15: unconnected-(IC1-PA10-Pad15) -> Net-(IC1-PA10)
- IC1 pad 16: unconnected-(IC1-PA11-Pad16) -> Net-(IC1-PA11)
- IC1 pad 3: unconnected-(IC1-PA02-Pad3) -> Net-(IC1-PA02)
- IC1 pad 4: unconnected-(IC1-PA03-Pad4) -> Net-(IC1-PA03)
- IC1 pad 9: unconnected-(IC1-PA04-Pad9) -> Net-(IC1-PA04)
Routing:
- net Net-(IC1-PA11): track 0.00 -> 11.4 mm, vias 0 -> 1
- net Net-(IC1-PA10): track 0.00 -> 9.18 mm, vias 0 -> 1
- net Net-(IC1-PA09): track 0.00 -> 7.85 mm, vias 0 -> 1
- net Net-(IC1-PA08): track 0.00 -> 6.52 mm, vias 0 -> 1
- net Net-(IC1-PA05): track 0.00 -> 4.67 mm
- net Net-(IC1-PA02): track 0.00 -> 4.46 mm
- net Net-(IC1-PA03): track 0.00 -> 4.26 mm
- net Net-(IC1-PA04): track 0.00 -> 4.05 mm

Commit message: can-module: Route out all signals
Parts:
- removed TP10, TP11, TP12, TP5, TP6, TP7, TP8, TP9: TestPoint, TestPoint:TestPoint_Pad_D1.0mm
- added C12: 10u, Capacitor_SMD:C_0402_1005Metric, F.Cu at (128.9, 62.8)
- added J1: Conn_01x04_Socket, Connector_PinHeader_1.00mm:PinHeader_1x04_P1.00mm_Vertical, F.Cu at (115.2, 57.5)
- added J2: Conn_01x04_Socket, Connector_PinHeader_1.00mm:PinHeader_1x04_P1.00mm_Vertical, F.Cu at (115.2, 62.5)
- added J3: Conn_01x04_Socket, Connector_PinHeader_1.00mm:PinHeader_1x04_P1.00mm_Vertical, F.Cu at (126.4, 64.5)
- added JP2: Jumper_2_Small_Open, Resistor_SMD:R_0201_0603Metric, F.Cu at (124.5, 65.2)
- added R3: 120, Resistor_SMD:R_0201_0603Metric, F.Cu at (124.5, 63.8)
- moved C3 0.25 mm to (117.5, 62.0)
- moved C4 0.25 mm to (117.5, 63.0)
Connections:
- IC1 pad 11: unconnected-(IC1-PA06-Pad11) -> Net-(IC1-PA06)
- IC1 pad 12: unconnected-(IC1-PA07-Pad12) -> Net-(IC1-PA07)
- IC1 pad 15: Net-(IC1-PA10) -> unconnected-(IC1-PA10-Pad15)
- IC1 pad 16: Net-(IC1-PA11) -> unconnected-(IC1-PA11-Pad16)
- IC1 pad 31: CAN_NSIL -> CAN_STBY
- IC1 pad 32: CAN_STBY -> CAN_NSIL
Routing:
- net Net-(IC1-PA11): track 11.4 -> 0.00 mm, vias 1 -> 0
- net Net-(IC1-PA10): track 9.18 -> 0.00 mm, vias 1 -> 0
- net CANH: track 0.00 -> 7.96 mm
- net GND: track 16.8 -> 24.5 mm, vias 9 -> 29
- net CAN_STBY: track 0.00 -> 7.19 mm, vias 0 -> 2
- net CANL: track 0.00 -> 6.75 mm
- net Net-(IC1-PA06): track 0.00 -> 4.77 mm
- net Net-(IC1-PA07): track 0.00 -> 4.57 mm
- net CAN_NSIL: track 0.00 -> 3.27 mm
- net Net-(IC1-PA04): track 4.05 -> 6.46 mm
- net Net-(JP2-B): track 0.00 -> 1.50 mm
- net Net-(IC1-PA02): track 4.46 -> 5.88 mm
- net +5V: track 3.08 -> 4.33 mm, vias 0 -> 16
- net Net-(IC1-PA05): track 4.67 -> 5.69 mm
- net Net-(IC1-PA03): track 4.26 -> 5.25 mm
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- added copper zone on B.Cu, net +5V

Commit message: can-module: Add board outline
Other:
- board outline added: 20 x 15 mm
Changed lines of the file:
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@@
 		(embedded_fonts no)
+	)
+	(gr_rect
+		(start 112.75 51.5)
+		(end 132.75 66.5)
+		(stroke
+			(width 0.05)
+			(type solid)
+		)
+		(fill no)
+		(layer "Edge.Cuts")
 	)
 	(segment
@@
 		(polygon
 			(pts
-				(xy 114 51.75) (xy 131.75 51.75) (xy 131.75 66.25) (xy 114 66.25)
+				(xy 112.5 51.35) (xy 133 51.35) (xy 133 66.7) (xy 112.5 66.7)
 			)
 		)
@@
 		(polygon
 			(pts
-				(xy 113.75 51.5) (xy 132 51.5) (xy 132 66.5) (xy 113.75 66.5)
+				(xy 112.1 50.9) (xy 133.35 50.9) (xy 133.35 67.35) (xy 112.1 67.35)
 			)
 		)

Commit message: can-module: Rearrange components, update constraints for copper to board edge
Parts:
- removed TP1, TP2: TestPoint, TestPoint:TestPoint_Pad_D1.0mm
- JP2: footprint Resistor_SMD:R_0201_0603Metric -> Jumper:SolderJumper-2_P1.3mm_Open_Pad1.0x1.5mm
- TP3, TP4: moved to F.Cu
- moved C12 7.62 mm to (131.2, 55.5), turned to 90 degrees
- moved JP2 6.32 mm to (130.5, 63.2)
- moved J3 6.27 mm to (131.2, 60.5), turned to 180 degrees
- moved TP3 5.01 mm to (116.8, 53.7), turned to 0 degrees
- moved R3 4.03 mm to (128.5, 63.2), turned to -90 degrees
- moved TP4 1.06 mm to (118.8, 53.7), turned to 0 degrees
- moved J1 1.00 mm to (114.2, 57.5)
- moved J2 1.00 mm to (114.2, 62.5)
- moved C1 0.75 mm to (116.7, 55.2)
- moved C10 0.75 mm to (123.2, 54.0)
- moved C11 0.75 mm to (128.7, 56.2)
- moved C2 0.75 mm to (116.7, 56.2)
- moved C3 0.75 mm to (116.8, 62.0)
- moved C4 0.75 mm to (116.8, 63.0)
- moved C5 0.75 mm to (121.1, 54.0)
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Routing:
- net CANH: track 7.96 -> 10.4 mm
- net Net-(IC1-PA31_SWDIO): track 2.86 -> 4.61 mm, vias 1 -> 0
- net +5V: track 4.33 -> 3.08 mm, vias 16 -> 15
- net GND: track 24.5 -> 23.3 mm, vias 29 -> 30
- net CANL: track 6.75 -> 6.05 mm
- net Net-(IC1-PA30_SWCLK): track 4.24 -> 3.59 mm, vias 2 -> 0

Commit message: can-module: Change connector footprints, add silkscreen labels
Parts:
- J1, J2, J3: footprint Connector_PinHeader_1.00mm:PinHeader_1x04_P1.00mm_Vertical -> Conn01x04:01x04_1mm
- moved J1 1.12 mm to (114.8, 58.5)
- moved J2 1.12 mm to (114.8, 63.5)
- moved C12 0.75 mm to (131.2, 54.8)
- moved J3 0.71 mm to (131.8, 61.0)
Other:
- board text added: "+"
- board text added: "+5V"
- board text added: "-"
- board text added: "2"
- board text added: "3"
- board text added: "4"
- board text added: "5"
- board text added: "6"
- board text added: "7"
- board text added: "8"
- board text added: "9"
- board text added: "CAN"
- board text added: "CANBus Module"
- board text added: "CK"
- board text added: "H"
- board text added: "IO"
- board text added: "J_{RCAN}"
- board text added: "L"
- board text added: "PA"
- board text added: "SWD"
