File: can-module/can-module.kicad_pcb (KiCad board)
At the start: 2 copper layers, 20 x 15 mm, 23 parts, among them IC1 PIC32CM1216JH01048-I_U5B, J1 Conn_01x04_Socket, J2 Conn_01x04_Socket, J3 Conn_01x04_Socket, U1 ATA6560-GBQW-N

Commit message: can-module: Move around capacitors for PIC32
Parts:
- moved C2 6.52 mm to (122.8, 53.8), turned to 90 degrees
- moved C4 5.62 mm to (122.2, 64.2), turned to -90 degrees
- moved C3 4.26 mm to (116.5, 57.8)
- moved C1 3.82 mm to (120.2, 53.8), turned to 90 degrees
- moved R2 1.90 mm to (121.0, 52.2), turned to 0 degrees
- moved C10 0.43 mm to (123.7, 54.0)
- moved R1 0.43 mm to (124.4, 54.0)
- moved C7 0.09 mm to (117.0, 58.8)
Routing:
- net Net-(IC1-PA30_SWCLK): track 3.59 -> 5.60 mm
- net +5V: track 3.08 -> 4.85 mm, vias 15 -> 10
- net Net-(IC1-PA05): track 5.44 -> 6.02 mm
- net Net-(IC1-PA04): track 6.42 -> 7.00 mm

Commit message: can-module: Extend 5V bar going to AVDD
Routing:
- net +5V: vias 10 -> 15
Changed lines of the file:
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@@
+	)
+	(via
+		(at 117 55.25)
+		(size 0.25)
+		(drill 0.15)
+		(layers "F.Cu" "B.Cu")
+		(free yes)
+		(net 1)
 	)
 	(via
@@
 	)
 	(via
+		(at 117.5 55.25)
+		(size 0.25)
+		(drill 0.15)
+		(layers "F.Cu" "B.Cu")
+		(free yes)
+		(net 1)
+	)
+	(via
 		(at 117 59.5)
 		(size 0.25)
@@
 	)
 	(via
+		(at 117 55.75)
+		(size 0.25)
+		(drill 0.15)
+		(layers "F.Cu" "B.Cu")
+		(free yes)
+		(net 1)
+	)
+	(via
+		(at 117.5 55.75)
+		(size 0.25)
+		(drill 0.15)
+		(layers "F.Cu" "B.Cu")
+		(free yes)
+		(net 1)
+	)
+	(via
 		(at 117.5 64.5)
+		(size 0.25)
+		(drill 0.15)
+		(layers "F.Cu" "B.Cu")
+		(free yes)
+		(net 1)
+	)
+	(via
+		(at 117.25 55.5)
 		(size 0.25)
 		(drill 0.15)
@@
 		(polygon
 			(pts
-				(xy 117.65 65.2) (xy 117.65 59.25) (xy 116.85 59.25) (xy 116.85 65.2)
+				(xy 117.65 65.2) (xy 117.65 55) (xy 116.85 55) (xy 116.85 65.2)
 			)
 		)

Commit message: can-module: Move around traces to maximize power plane area
Routing:
- net Net-(IC1-PA08): track 7.03 -> 5.19 mm
- net Net-(IC1-PA09): track 6.86 -> 6.26 mm
Changed lines of the file:
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@@
 	)
 	(via
-		(at 117 64.5)
+		(at 117 63.5)
 		(size 0.25)
 		(drill 0.15)
@@
 	)
 	(via
-		(at 117.25 64.75)
+		(at 117.25 63.75)
 		(size 0.25)
 		(drill 0.15)
@@
 	)
 	(via
-		(at 117.5 65)
+		(at 117.5 64)
 		(size 0.25)
 		(drill 0.15)
@@
 	)
 	(via
-		(at 117 65)
+		(at 117 64)
 		(size 0.25)
 		(drill 0.15)
@@
 	)
 	(via
-		(at 117.5 64.5)
+		(at 117.5 63.5)
 		(size 0.25)
 		(drill 0.15)
@@
 	)
 	(segment
-		(start 118.725 64)
-		(end 115.25 64)
+		(start 119 63.25)
+		(end 118.75 63)
 		(width 0.1)
 		(layer "F.Cu")
@@
 	)
 	(segment
-		(start 119.75 62.975)
-		(end 118.725 64)
+		(start 119.75 63)
+		(end 119.5 63.25)
 		(width 0.1)
 		(layer "F.Cu")
@@
 	)
 	(segment
-		(start 115.25 64)
+		(start 118.75 63)
 		(end 114.25 63)
 		(width 0.1)
@@
 	(segment
 		(start 119.75 62.45)
-		(end 119.75 62.975)
+		(end 119.75 63)
+		(width 0.1)
+		(layer "F.Cu")
+		(net 7)
+	)
+	(segment
+		(start 119.5 63.25)
+		(end 119 63.25)
 		(width 0.1)
 		(layer "F.Cu")
@@
 	)
 	(segment
-		(start 118.641744 63.799)
-		(end 119.25 63.190744)
+		(start 115.75 62)
+		(end 114.25 62)
 		(width 0.1)
 		(layer "F.Cu")
@@
 	)
 	(segment
-		(start 114.5 62)
-		(end 115.25 62.75)
+		(start 119.25 62.45)
+		(end 116.2 62.45)
 		(width 0.1)
 		(layer "F.Cu")
@@
 	)
 	(segment
-		(start 115.799 63.799)
-		(end 118.641744 63.799)
-		(width 0.1)
-		(layer "F.Cu")
-		(net 11)
-	)
-	(segment
-		(start 114.25 62)
-		(end 114.5 62)
-		(width 0.1)
-		(layer "F.Cu")
-		(net 11)
-	)
-	(segment
-		(start 115.25 63.25)
-		(end 115.799 63.799)
-		(width 0.1)
-		(layer "F.Cu")
-		(net 11)
-	)
-	(segment
-		(start 119.25 63.190744)
-		(end 119.25 62.45)
-		(width 0.1)
-		(layer "F.Cu")
-		(net 11)
-	)
-	(segment
-		(start 115.25 62.75)
-		(end 115.25 63.25)
+		(start 116.2 62.45)
+		(end 115.75 62)
 		(width 0.1)
 		(layer "F.Cu")
@@
 		(polygon
 			(pts
-				(xy 117.65 65.2) (xy 117.65 55) (xy 116.85 55) (xy 116.85 65.2)
+				(xy 117.65 64.2) (xy 117.65 55) (xy 116.85 55) (xy 116.85 64.2)
 			)
 		)

Commit message: can-module: Adjust board size
Parts:
- added D1: PESD5V0S1BAF, Diode_SMD:D_SOD-323, F.Cu at (137.0, 54.5)
- added D2: PESD5V0S1BAF, Diode_SMD:D_SOD-323, F.Cu at (133.0, 57.0)
- added D3: PESD5V0S1BAF, Diode_SMD:D_SOD-323, F.Cu at (133.0, 61.0)
- moved R3 5.57 mm to (134.0, 64.2)
- moved J3 5.40 mm to (137.2, 61.0)
- moved JP2 5.32 mm to (135.8, 64.1), turned to -90 degrees
- moved C12 3.76 mm to (135.0, 55.0)
- moved U1 1.69 mm to (129.9, 59.0), turned to 0 degrees
- moved C11 1.14 mm to (129.7, 56.8)
Routing:
- net GND: track 23.3 -> 28.9 mm, vias 30 -> 41
- net CAN_NSIL: track 3.27 -> 7.67 mm
- net CAN_RX: track 2.01 -> 5.21 mm
- net CANL: track 6.05 -> 9.04 mm, vias 0 -> 1
- net Net-(JP2-B): track 1.48 -> 0.00 mm
- net CAN_TX: track 4.71 -> 3.36 mm, vias 3 -> 2
Other:
- board size 20 x 15 mm -> 25.4 x 15.2 mm

Commit message: can-module: Finalize pcb layout, fix errors and constraints
Routing:
- net Net-(JP2-B): track 0.00 -> 1.86 mm
Other:
- board text added: "Rev A"
Changed lines of the file:
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@@
 	)
 	(gr_text "H"
-		(at 137.15 59.5 0)
+		(at 137.15 59.5 90)
 		(layer "F.SilkS")
 		(effects
@@
 				(thickness 0.09375)
 			)
-			(justify left)
+			(justify top)
 		)
 	)
 	(gr_text "7"
-		(at 113.75 61 0)
+		(at 113.75 61 270)
 		(layer "F.SilkS")
 		(effects
@@
 				(thickness 0.09375)
 			)
-			(justify right)
+			(justify top)
 		)
 	)
@@
 	)
 	(gr_text "+"
-		(at 137.15 57.5 0)
+		(at 137.15 57.5 90)
 		(layer "F.SilkS")
 		(effects
@@
 				(thickness 0.09375)
 			)
-			(justify left)
+			(justify top)
 		)
 	)
 	(gr_text "9"
-		(at 113.75 63 0)
+		(at 113.75 63 270)
 		(layer "F.SilkS")
 		(effects
@@
 				(thickness 0.09375)
 			)
-			(justify right)
+			(justify top)
 		)
 	)
@@
 	)
 	(gr_text "-"
-		(at 137.15 58.5 0)
+		(at 137.15 58.5 90)
 		(layer "F.SilkS")
 		(effects
@@
 				(thickness 0.09375)
 			)
-			(justify left)
+			(justify top)
 		)
 	)
 	(gr_text "6"
-		(at 113.75 60 0)
+		(at 113.75 60 270)
 		(layer "F.SilkS")
 		(effects
@@
 				(thickness 0.09375)
 			)
-			(justify right)
+			(justify top)
 		)
 	)
@@
 	)
 	(gr_text "2"
-		(at 113.75 55 0)
+		(at 113.75 55 270)
 		(layer "F.SilkS")
 		(effects
@@
 				(thickness 0.09375)
 			)
-			(justify right)
+			(justify top)
 		)
 	)
@@
 	)
 	(gr_text "3"
-		(at 113.75 56 0)
+		(at 113.75 56 270)
 		(layer "F.SilkS")
 		(effects
@@
 				(thickness 0.09375)
 			)
-			(justify right)
+			(justify top)
 		)
 	)
 	(gr_text "8"
-		(at 113.75 62 0)
+		(at 113.75 62 270)
 		(layer "F.SilkS")
 		(effects
@@
 				(thickness 0.09375)
 			)
-			(justify right)
+			(justify top)
 		)
 	)
 	(gr_text "L"
-		(at 137.15 60.5 0)
+		(at 137.15 60.5 90)
 		(layer "F.SilkS")
 		(effects
@@
 				(thickness 0.09375)
 			)
-			(justify left)
+			(justify top)
 		)
 	)
@@
 	)
 	(gr_text "5"
-		(at 113.75 58 0)
+		(at 113.75 58 270)
 		(layer "F.SilkS")
 		(effects
@@
 				(thickness 0.09375)
 			)
-			(justify right)
+			(justify top)
+		)
+	)
+	(gr_text "Rev A"
+		(at 112.75 66.5 0)
+		(layer "F.SilkS")
+		(effects
+			(font
+				(size 0.75 0.75)
+				(thickness 0.09375)
+			)
+			(justify left bottom)
 		)
 	)
@@
 	)
 	(gr_text "4"
-		(at 113.75 57 0)
+		(at 113.75 57 270)
 		(layer "F.SilkS")
 		(effects
@@
 				(thickness 0.09375)
 			)
-			(justify right)
+			(justify top)
 		)
 	)
@@
 	)
 	(via
-		(at 117.5 60)
+		(at 117.498615 59.849997)
 		(size 0.25)
 		(drill 0.15)
@@
 	)
 	(via
-		(at 117 59.5)
+		(at 116.998615 59.349997)
 		(size 0.25)
 		(drill 0.15)
@@
 	)
 	(via
-		(at 117.25 59.75)
+		(at 117.248615 59.599997)
 		(size 0.25)
 		(drill 0.15)
@@
 	)
 	(via
-		(at 117.5 59.5)
-		(size 0.25)
-		(drill 0.15)
-		(layers "F.Cu" "B.Cu")
-		(free yes)
-		(net 1)
-	)
-	(via
-		(at 117 60)
+		(at 117.498615 59.349997)
+		(size 0.25)
+		(drill 0.15)
+		(layers "F.Cu" "B.Cu")
+		(free yes)
+		(net 1)
+	)
+	(via
+		(at 116.998615 59.849997)
 		(size 0.25)
 		(drill 0.15)
@@
 	)
 	(segment
+		(start 135.75 64.75)
+		(end 134.275 64.75)
+		(width 0.1)
+		(layer "F.Cu")
+		(net 40)
+	)
+	(segment
+		(start 134.275 64.75)
+		(end 134 64.475)
+		(width 0.1)
+		(layer "F.Cu")
+		(net 40)
+	)
+	(segment
