File: can-module/can-module.kicad_pcb (KiCad board)
At the start: 2 copper layers, 25.4 x 19.1 mm, 44 parts, among them IC1 PIC32CM1216JH01048-I_U5B, J1 Conn_01x04_Socket, J2 Conn_01x04_Socket, J3 Conn_01x04_Socket, U1 ATA6560-GBQW-N

Commit message: can-module: Add SWD pins back in
Parts:
- moved TP3 6.39 mm to (124.5, 51.8)
- moved TP4 6.39 mm to (126.5, 51.8)
Changed lines of the file:
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@@
 	(footprint "TestPoint:TestPoint_Pad_D1.0mm"
 		(layer "B.Cu")
-		(at 125.6 45.45 180)
+		(at 124.549999 51.75 180)
 		(descr "SMD pad as test Point, diameter 1.0mm")
 		(tags "test point SMD pad")
@@
 	(footprint "TestPoint:TestPoint_Pad_D1.0mm"
 		(layer "B.Cu")
-		(at 127.6 45.45 180)
+		(at 126.549999 51.75 180)
 		(descr "SMD pad as test Point, diameter 1.0mm")
 		(tags "test point SMD pad")
@@
 	)
 	(gr_text "IO"
-		(at 125.6 46.45 -180)
+		(at 124.549999 52.75 -180)
 		(layer "B.SilkS")
 		(effects
@@
 	)
 	(gr_text "CLK"
-		(at 127.6 46.45 -180)
+		(at 126.549999 52.75 -180)
 		(layer "B.SilkS")
 		(effects
@@
 	)
 	(gr_text "SWD"
-		(at 126.6 43.45 -180)
+		(at 125.5 49.75 -180)
 		(layer "B.SilkS")
 		(effects

Commit message: can-module: Convert GPIO header from 2x 4pin header to 1x 8pin
Parts:
- removed J2: Conn_01x04_Socket, Conn01x04:01x04_1mm
- J1: value Conn_01x04_Socket -> Conn_01x08_Socket; footprint Conn01x04:01x04_1mm -> Conn_01x08:Untitled
- moved J1 4.51 mm to (115.0, 63.0)
Connections:
- J1 pad 1: PA05 -> PA09
- J1 pad 2: PA04 -> PA08
- J1 pad 3: PA03 -> PA07
- J1 pad 4: PA02 -> PA06
Routing:
- net Net-(IC1-PA30_SWCLK): track 3.81 -> 12.8 mm
- net Net-(IC1-PA31_SWDIO): track 2.90 -> 9.80 mm
- net PA09: track 7.89 -> 8.66 mm
- net PA08: track 9.31 -> 8.76 mm

Commit message: can-module: Add actual Rowan Motorsports logo to PCB
Parts:
- added G***: LOGO, Logos:RowanMotorsports, B.Cu at (125.7, 59.2)
Other:
- board text removed: "ROWAN MOTORSPORTS"

Commit message: can-module: Update PCB to match requirements for JLCPCB economic PCBA
Parts:
- C10, C11, C5, C6, C7, C8, C9: footprint Capacitor_SMD:C_0201_0603Metric -> Capacitor_SMD:C_0402_1005Metric
- R1, R10, R11, R2, R3, R4, R5, R6, R7, R8, R9: footprint Resistor_SMD:R_0201_0603Metric -> Resistor_SMD:R_0402_1005Metric
- moved R2 1.72 mm to (117.8, 53.5), turned to -90 degrees
- moved R11 0.79 mm to (116.5, 64.5)
- moved R5 0.77 mm to (116.5, 53.5)
- moved JP6 0.66 mm to (113.1, 64.9)
- moved JP8 0.66 mm to (115.6, 64.9)
- moved JP7 0.65 mm to (114.4, 64.9)
- moved JP9 0.65 mm to (116.9, 64.9)
- moved R1 0.64 mm to (125.0, 53.7), turned to -90 degrees
- moved JP1 0.61 mm to (116.4, 53.1)
- moved JP3 0.61 mm to (117.7, 53.1)
- moved JP4 0.61 mm to (115.2, 53.1)
- moved JP5 0.61 mm to (113.9, 53.1)
- moved R10 0.56 mm to (115.5, 64.5)
- moved R4 0.53 mm to (115.5, 53.5)
- moved C10 0.41 mm to (124.0, 53.8)
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Routing:
- net +5V: track 13.4 -> 9.75 mm
- net Net-(IC1-PA30_SWCLK): track 12.8 -> 14.1 mm
- net GND: track 28.9 -> 29.9 mm
- net Net-(JP3-C): track 3.08 -> 2.16 mm
- net Net-(JP9-C): track 3.07 -> 2.16 mm
- net Net-(IC1-PA31_SWDIO): track 9.80 -> 10.6 mm
- net Net-(JP1-C): track 2.58 -> 1.91 mm
- net Net-(JP8-C): track 2.57 -> 1.91 mm
- net Net-(JP4-C): track 2.31 -> 1.80 mm
