File: power-can-tap/power-can-tap.kicad_sch (KiCad schematic)
At the start: 0 parts

Commit message: power-can-tap: Add T tap to schematic
Parts:
- added J1: Conn_01x04_Pin, Conn_01x04:01x04_1mm, symbol Connector:Conn_01x04_Pin
- added J2, J3: Conn_01x04_Socket, Connector_PinSocket_2.54mm:PinSocket_1x04_P2.54mm_Vertical, symbol Connector:Conn_01x04_Socket
Connections:
- new net +5V: J1.1 (Pin_1), J2.1 (Pin_1), J3.1 (Pin_1)
- new net CANH: J1.3 (Pin_3), J2.3 (Pin_3), J3.3 (Pin_3)
- new net CANL: J1.4 (Pin_4), J2.4 (Pin_4), J3.4 (Pin_4)
- new net GND: J1.2 (Pin_2), J2.2 (Pin_2), J3.2 (Pin_2)
Other:
- note added: "T-Tap"
