File: can-module/pcb/can-module.kicad_pcb (KiCad board)
At the start: 2 copper layers, 25.4 x 19.1 mm, 44 parts, among them IC1 PIC32CM1216JH01048-I_U5B, J1 Conn_01x08_Socket, J3 Conn_01x04_Socket, U1 ATA6560-GBQW-N

Commit message: can-module: Add 5V output for daughter boards
Parts:
- added J2: Conn_01x02_Socket, Conn_01x02:Untitled, F.Cu at (121.5, 50.2)
Changed lines of the file:
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@@
 		)
 	)
+	(footprint "Conn_01x02:Untitled"
+		(layer "F.Cu")
+		(at 121.5 50.25 -90)
+		(property "Reference" "J2"
+			(at 0 -0.5 270)
+			(unlocked yes)
+			(layer "F.SilkS")
+			(hide yes)
+			(effects
+				(font
+					(size 1 1)
+					(thickness 0.1)
+				)
+			)
+		)
+		(property "Value" "Conn_01x02_Socket"
+			(at 0 1 270)
+			(unlocked yes)
+			(layer "F.Fab")
+			(hide yes)
+			(effects
+				(font
+					(size 1 1)
+					(thickness 0.15)
+				)
+			)
+		)
+		(property "Datasheet" "~"
+			(at 0 0 270)
+			(unlocked yes)
+			(layer "F.Fab")
+			(hide yes)
+			(effects
+				(font
+					(size 1 1)
+					(thickness 0.15)
+				)
+			)
+		)
+		(property "Description" "Generic connector, single row, 01x02, script generated"
+			(at 0 0 270)
+			(unlocked yes)
+			(layer "F.Fab")
+			(hide yes)
+			(effects
+				(font
+					(size 1 1)
+					(thickness 0.15)
+				)
+			)
+		)
+		(property ki_fp_filters "Connector*:*_1x??_*")
+		(sheetname "/")
+		(sheetfile "can-module.kicad_sch")
+		(attr smd)
+		(pad "1" thru_hole circle
+			(at 0.5 0.5 270)
+			(size 0.85 0.85)
+			(drill 0.5)
+			(layers "*.Cu" "*.Mask")
+			(remove_unused_layers no)
+			(net 2 "GND")
+			(pinfunction "Pin_1")
+			(pintype "passive")
+		)
+		(pad "2" thru_hole circle
+			(at 0.5 1.5 270)
+			(size 0.85 0.85)
+			(drill 0.5)
+			(layers "*.Cu" "*.Mask")
+			(remove_unused_layers no)
+			(net 1 "+5V")
+			(pinfunction "Pin_2")
+			(pintype "passive")
+		)
+		(embedded_fonts no)
+	)
 	(footprint "MountingHole:MountingHole_2.2mm_M2"
 		(layer "F.Cu")
@@
 	)
 	(gr_line
+		(start 121.75 51.25)
+		(end 119.25 51.25)
+		(stroke
+			(width 0.1)
+			(type default)
+		)
+		(layer "F.SilkS")
+	)
+	(gr_line
 		(start 135.65 61.5)
 		(end 135.65 56.5)
@@
 	)
 	(gr_line
+		(start 119.25 51.25)
+		(end 119.25 49.75)
+		(stroke
+			(width 0.1)
+			(type default)
+		)
+		(layer "F.SilkS")
+	)
+	(gr_line
 		(start 115.25 54.75)
 		(end 115.25 63.25)
@@
 	)
 	(gr_line
+		(start 121.75 49.75)
+		(end 121.75 51.25)
+		(stroke
+			(width 0.1)
+			(type default)
+		)
+		(layer "F.SilkS")
+	)
+	(gr_line
 		(start 134.5 59)
 		(end 138 59)
@@
 	)
 	(gr_text "+"
+		(at 120 50.5 180)
+		(layer "F.SilkS")
+		(effects
+			(font
+				(size 0.75 0.75)
+				(thickness 0.09375)
+			)
+			(justify top)
+		)
+	)
+	(gr_text "-"
+		(at 121 50.5 180)
+		(layer "F.SilkS")
+		(effects
+			(font
+				(size 0.75 0.75)
+				(thickness 0.09375)
+			)
+			(justify top)
+		)
+	)
+	(gr_text "+"
 		(at 137.15 57.5 90)
 		(layer "F.SilkS")
@@
 		)
 	)
+	(gr_text "+5V"
+		(at 120.5 51.5 180)
+		(layer "F.SilkS")
+		(effects
+			(font
+				(size 0.75 0.75)
+				(thickness 0.15)
+				(bold yes)
+			)
+			(justify bottom)
+		)
+	)
 	(gr_text "9"
 		(at 113.75 62.5 270)
@@
 		(layer "F.Fab")
 		(pts
+			(xy 120 50.75) (xy 114.5 55.5)
+		)
+		(height -3.25)
+		(orientation 0)
+		(format
+			(prefix "")
+			(suffix "")
+			(units 3)
+			(units_format 0)
+			(precision 4)
+			(suppress_zeroes yes)
+		)
+		(style
+			(thickness 0.1)
+			(arrow_length 1.27)
+			(text_position_mode 0)
+			(arrow_direction outward)
+			(extension_height 0.58642)
+			(extension_offset 0.5)
+			(keep_text_aligned yes)
+		)
+		(gr_text "5.5"
+			(at 117.25 46.35 0)
+			(layer "F.Fab")
+			(effects
+				(font
+					(size 1 1)
+					(thickness 0.15)
+				)
+			)
+		)
+	)
+	(dimension
+		(type orthogonal)
+		(layer "F.Fab")
+		(pts
 			(xy 129.65 53.225) (xy 129.65 49.5)
 		)
@@
 			(layer "F.Fab")
 			(effects
+				(font
+					(size 1 1)
+					(thickness 0.15)
+				)
+			)
+		)
+	)
+	(dimension
+		(type orthogonal)
+		(layer "F.Fab")
+		(pts
+			(xy 120 50.75) (xy 114.5 55.5)
+		)
+		(height -9.5)
+		(orientation 1)
+		(format
+			(prefix "")
+			(suffix "")
+			(units 3)
+			(units_format 0)
+			(precision 4)
+			(suppress_zeroes yes)
+		)
+		(style
+			(thickness 0.1)
+			(arrow_length 1.27)
+			(text_position_mode 0)
+			(arrow_direction outward)
+			(extension_height 0.58642)
+			(extension_offset 0.5)
+			(keep_text_aligned yes)
+		)
+		(gr_text "4.75"
+			(at 109.35 53.125 90)
+			(layer "F.Fab")
+			(effects

Commit message: can-module: Adjust positioning for 5V daughterboard connector, add 3D models for daughterboard connector headers
Parts:
- moved J2 0.25 mm to (121.5, 50.5)
Changed lines of the file:
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@@
 		)
 		(embedded_fonts no)
+		(model "${KICAD9_3DMODEL_DIR}/Connector_PinHeader_1.00mm.3dshapes/PinHeader_1x08_P1.00mm_Vertical.step"
+			(offset
+				(xyz 0.5 -0.5 0)
+			)
+			(scale
+				(xyz 1 1 1)
+			)
+			(rotate
+				(xyz -0 -0 -0)
+			)
+		)
 	)
 	(footprint "Diode_SMD:D_SOD-323"
@@
 	(footprint "Conn_01x02:Untitled"
 		(layer "F.Cu")
-		(at 121.5 50.25 -90)
+		(at 121.5 50.5 -90)
 		(property "Reference" "J2"
 			(at 0 -0.5 270)
@@
 		)
 		(embedded_fonts no)
+		(model "${KICAD9_3DMODEL_DIR}/Connector_PinHeader_1.00mm.3dshapes/PinHeader_1x02_P1.00mm_Vertical.step"
+			(offset
+				(xyz 0.5 -0.5 0)
+			)
+			(scale
+				(xyz 1 1 1)
+			)
+			(rotate
+				(xyz -0 -0 -0)
+			)
+		)
 	)
 	(footprint "MountingHole:MountingHole_2.2mm_M2"
@@
 	)
 	(gr_line
-		(start 121.75 51.25)
-		(end 119.25 51.25)
+		(start 121.75 51.5)
+		(end 119.25 51.5)
 		(stroke
 			(width 0.1)
@@
 	)
 	(gr_line
-		(start 119.25 51.25)
+		(start 119.25 51.5)
 		(end 119.25 49.75)
 		(stroke
@@
 	(gr_line
 		(start 121.75 49.75)
-		(end 121.75 51.25)
+		(end 121.75 51.5)
 		(stroke
 			(width 0.1)
@@
 	)
 	(gr_text "+5V"
-		(at 120.5 51.5 180)
+		(at 122 50.25 180)
 		(layer "F.SilkS")
 		(effects
@@
 				(bold yes)
 			)
-			(justify bottom)
+			(justify right)
 		)
 	)

Commit message: can-module: Major changes to routing, placement; remove pull up/down resistors (use PIC32 internal resistors)
Parts:
- removed JP1, JP3, JP4, JP5, JP6, JP7, JP8, JP9: SolderJumper_3_Open, SolderJumperSmall:Jumper3Small
- removed R10, R11, R5, R6, R7, R8, R9: 1k, Resistor_SMD:R_0402_1005Metric
- added C13: 4n7, Capacitor_SMD:C_0402_1005Metric, F.Cu at (133.2, 67.5)
- R3: value 120 -> 60
- R4: value 1k -> 60
- TP3, TP4: moved to F.Cu
- moved R4 22.0 mm to (133.3, 66.5), turned to 0 degrees
- moved TP3 9.05 mm to (115.5, 51.7), turned to 0 degrees
- moved TP4 9.05 mm to (117.5, 51.7), turned to 0 degrees
- moved D2 6.54 mm to (134.8, 63.2), turned to 90 degrees
- moved D3 4.35 mm to (136.8, 63.2)
- moved C11 3.63 mm to (127.2, 59.4), turned to 90 degrees
- moved C12 3.52 mm to (135.0, 51.5)
- moved JP2 2.16 mm to (136.0, 66.2), turned to 0 degrees
- moved R3 1.35 mm to (133.3, 65.5), turned to 180 degrees
- moved R2 1.25 mm to (119.0, 53.6), turned to 90 degrees
- moved C4 0.50 mm to (121.8, 64.2)
- moved C8 0.50 mm to (120.8, 64.2)
- moved C3 0.35 mm to (116.2, 57.5)
- moved C1 0.15 mm to (120.0, 53.6)
- moved C10 0.15 mm to (124.0, 53.6)
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Connections:
- JP2 pad 1: CANH -> Net-(JP2-A)
- JP2 pad 2: Net-(JP2-B) -> CANL
- R3 pad 1: CANL -> CANH
- R3 pad 2: Net-(JP2-B) -> Net-(C13-Pad2)
- R4 pad 1: PA03 -> Net-(C13-Pad2)
- R4 pad 2: Net-(JP1-C) -> Net-(JP2-A)
Routing:
- net CANL: track 9.24 -> 21.1 mm, vias 1 -> 0
- net CANH: track 10.9 -> 21.1 mm
- net +5V: track 9.75 -> 0.50 mm, vias 14 -> 8
- net Net-(IC1-PA30_SWCLK): track 14.1 -> 6.63 mm, vias 1 -> 0
- net CAN_STBY: track 7.28 -> 13.2 mm
- net PA05: track 10.3 -> 4.98 mm
- net PA06: track 9.68 -> 4.77 mm
- net PA04: track 10.1 -> 5.53 mm
- net PA07: track 8.70 -> 4.57 mm
- net Net-(IC1-PA31_SWDIO): track 10.6 -> 6.67 mm, vias 1 -> 0
- net PA08: track 8.72 -> 5.14 mm
- net PA03: track 8.14 -> 4.57 mm
- net PA02: track 7.39 -> 4.77 mm
- net PA09: track 8.83 -> 6.26 mm
- net CAN_RX: track 5.21 -> 7.43 mm, vias 0 -> 2
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Other:
- board text removed: "DOWN"
- board text removed: "UP"

Commit message: can-module: Remove unused GPIO resistors sheet
Parts:
- moved C12 6.20 mm to (133.5, 57.5), turned to 180 degrees
Changed lines of the file:
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@@
 	(footprint "Capacitor_SMD:C_0402_1005Metric"
 		(layer "F.Cu")
-		(at 135 51.48 90)
+		(at 133.5 57.5 180)
 		(descr "Capacitor SMD 0402 (1005 Metric), square (rectangular) end terminal, IPC-7351 nominal, (Body size source: IPC-SM-782 page 76, https://www.pcb-3d.com/wordpress/wp-content/uploads/ipc-sm-782a_amendment_1_and_2.pdf), generated with kicad-footprint-generator")
 		(tags "capacitor")
 		(property "Reference" "C12"
-			(at 0 -1.16 90)
+			(at 0 -1.16 0)
 			(layer "F.SilkS")
 			(hide yes)
@@
 		)
 		(property "Value" "10u"
-			(at 0 1.16 90)
+			(at 0 1.16 0)
 			(layer "F.Fab")
 			(effects
@@
 		)
 		(property "Datasheet" "~"
-			(at 0 0 90)
+			(at 0 0 0)
 			(layer "F.Fab")
 			(hide yes)
@@
 		)
 		(property "Description" "Unpolarized capacitor, small symbol"
-			(at 0 0 90)
+			(at 0 0 0)
 			(layer "F.Fab")
 			(hide yes)
@@
 		(attr smd)
 		(fp_line
-			(start -0.107836 -0.36)
-			(end 0.107836 -0.36)
+			(start -0.107836 0.36)
+			(end 0.107836 0.36)
 			(stroke
 				(width 0.12)
@@
 		)
 		(fp_line
-			(start -0.107836 0.36)
-			(end 0.107836 0.36)
+			(start -0.107836 -0.36)
+			(end 0.107836 -0.36)
 			(stroke
 				(width 0.12)
@@
 		)
 		(fp_line
-			(start 0.91 -0.46)
-			(end 0.91 0.46)
+			(start 0.91 0.46)
+			(end -0.91 0.46)
 			(stroke
 				(width 0.05)
@@
 		)
 		(fp_line
-			(start -0.91 -0.46)
-			(end 0.91 -0.46)
+			(start 0.91 -0.46)
+			(end 0.91 0.46)
 			(stroke
 				(width 0.05)
@@
 		)
 		(fp_line
-			(start 0.91 0.46)
-			(end -0.91 0.46)
+			(start -0.91 0.46)
+			(end -0.91 -0.46)
 			(stroke
 				(width 0.05)
@@
 		)
 		(fp_line
-			(start -0.91 0.46)
-			(end -0.91 -0.46)
+			(start -0.91 -0.46)
+			(end 0.91 -0.46)
 			(stroke
 				(width 0.05)
@@
 		)
 		(fp_line
-			(start 0.5 -0.25)
-			(end 0.5 0.25)
+			(start 0.5 0.25)
+			(end -0.5 0.25)
 			(stroke
 				(width 0.1)
@@
 		)
 		(fp_line
-			(start -0.5 -0.25)
-			(end 0.5 -0.25)
+			(start 0.5 -0.25)
+			(end 0.5 0.25)
 			(stroke
 				(width 0.1)
@@
 		)
 		(fp_line
-			(start 0.5 0.25)
-			(end -0.5 0.25)
+			(start -0.5 0.25)
+			(end -0.5 -0.25)
 			(stroke
 				(width 0.1)
@@
 		)
 		(fp_line
-			(start -0.5 0.25)
-			(end -0.5 -0.25)
+			(start -0.5 -0.25)
+			(end 0.5 -0.25)
 			(stroke
 				(width 0.1)
@@
 		)
 		(fp_text user "${REFERENCE}"
-			(at 0 0 90)
+			(at 0 0 0)
 			(layer "F.Fab")
 			(effects
@@
 		)
 		(pad "1" smd roundrect
-			(at -0.48 0 90)
+			(at -0.48 0 180)
 			(size 0.56 0.62)
 			(layers "F.Cu" "F.Mask" "F.Paste")
@@
 		)
 		(pad "2" smd roundrect
-			(at 0.48 0 90)
+			(at 0.48 0 180)
 			(size 0.56 0.62)
 			(layers "F.Cu" "F.Mask" "F.Paste")
@@
 	)
 	(segment
-		(start 135 51)
-		(end 135.5 51)
+		(start 133.02 57.5)
+		(end 133.02 57)
 		(width 0.2)
 		(layer "F.Cu")
@@
 	)
 	(segment
-		(start 135 51)
-		(end 134.5 51)
+		(start 133.02 57.5)
+		(end 133.02 58)
 		(width 0.2)
 		(layer "F.Cu")
@@
 	)
 	(segment
-		(start 135 51)
-		(end 135 50.48)
+		(start 133.02 57.5)
+		(end 132.5 57.5)
 		(width 0.2)
 		(layer "F.Cu")
@@
 	)
 	(via
-		(at 135.5 51)
+		(at 133.02 57)
 		(size 0.4)
 		(drill 0.3)
@@
 	)
 	(via
-		(at 134.5 51)
+		(at 133.02 58)
 		(size 0.4)
 		(drill 0.3)
@@
 	)
 	(via
-		(at 135 50.48)
+		(at 132.5 57.5)
 		(size 0.4)
 		(drill 0.3)

Commit message: can-module: Change header size from 1mm spacing to 1.27mm spacing
Parts:
- J1: footprint Conn_01x08:Untitled -> Connector_PinHeader_1.27mm:PinHeader_1x08_P1.27mm_Vertical
- J2: footprint Conn_01x02:Untitled -> Connector_PinHeader_1.27mm:PinHeader_1x02_P1.27mm_Vertical
- moved TP3 1.51 mm to (114.0, 51.5)
- moved TP4 1.51 mm to (116.0, 51.5)
- moved J1 0.89 mm to (114.2, 63.5)
- moved J2 0.71 mm to (121.0, 51.0)
- moved C3 0.57 mm to (116.8, 57.8)
Routing:
- net Net-(IC1-PA31_SWDIO): track 6.67 -> 8.25 mm
- net Net-(IC1-PA30_SWCLK): track 6.63 -> 8.20 mm
- net PA05: track 4.98 -> 5.94 mm
- net PA04: track 5.53 -> 6.28 mm
- net PA02: track 4.77 -> 5.42 mm
- net PA03: track 4.57 -> 5.10 mm
Other:
- board size 25.4 x 19.1 mm -> 25.4 x 19 mm
- board text added: "PA2"
- board text added: "PA9"
- board text removed: "2"
- board text removed: "3"
- board text removed: "4"
- board text removed: "5"
- board text removed: "6"
- board text removed: "7"
- board text removed: "8"
- board text removed: "9"
- board text removed: "PA"

Commit message: can-module: Resolve hole clearance issue
Parts:
- moved C12 0.18 mm to (133.7, 57.5)
Changed lines of the file:
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@@
 	(footprint "Capacitor_SMD:C_0402_1005Metric"
 		(layer "F.Cu")
-		(at 133.5 57.525 180)
+		(at 133.68 57.525 180)
 		(descr "Capacitor SMD 0402 (1005 Metric), square (rectangular) end terminal, IPC-7351 nominal, (Body size source: IPC-SM-782 page 76, https://www.pcb-3d.com/wordpress/wp-content/uploads/ipc-sm-782a_amendment_1_and_2.pdf), generated with kicad-footprint-generator")
 		(tags "capacitor")
@@
 	)
 	(segment
-		(start 133.02 57.525)
-		(end 133.02 58.025)
+		(start 133.2 57.525)
+		(end 133.2 58.025)
 		(width 0.2)
 		(layer "F.Cu")
@@
 	)
 	(segment
-		(start 133.02 57.525)
-		(end 132.5 57.525)
+		(start 133.2 57.525)
+		(end 132.68 57.525)
 		(width 0.2)
 		(layer "F.Cu")
@@
 	)
 	(via
-		(at 133.02 57.025)
+		(at 133.2 57.025)
 		(size 0.4)
 		(drill 0.3)
@@
 	)
 	(via
-		(at 133.02 58.025)
+		(at 133.2 58.025)
 		(size 0.4)
 		(drill 0.3)
@@
 	)
 	(via
-		(at 132.5 57.525)
+		(at 132.68 57.525)
 		(size 0.4)
 		(drill 0.3)
@@
 		(single_sided no)
 		(target_length 8.2509)
-		(target_length_max 8.3509)
+		(target_length_max 8.350899)
 		(target_length_min 8.1509)
 		(target_skew 0)
