File: can-module/pcb/can-module.kicad_pcb (KiCad board)
At the start: 2 copper layers, 25.4 x 19 mm, 31 parts, among them IC1 PIC32CM1216JH01048-I_U5B, J1 Conn_01x08_Socket, J2 Conn_01x02_Socket, J3 Conn_01x04_Socket, U1 ATA6560-GBQW-N

Commit message: can-module: Update CAN/PWR header to also be 0.127mm, move some things around to allow for wider min power plane width
Parts:
- J3: footprint Conn01x04:01x04_1mm -> Connector_PinHeader_1.27mm:PinHeader_1x04_P1.27mm_Vertical
- moved TP3 0.80 mm to (114.8, 51.5)
- moved TP4 0.80 mm to (116.8, 51.5)
- moved J3 0.51 mm to (136.7, 60.9)
- moved J2 0.39 mm to (121.4, 51.0)
Routing:
- net Net-(IC1-PA30_SWCLK): track 8.20 -> 6.91 mm
- net Net-(IC1-PA31_SWDIO): track 8.25 -> 7.45 mm
Other:
- board text added: "GND"
- board text added: "ROWAN MOTORSPORTS Rev A"
- board text removed: "Rev A"

Commit message: can-module: Update text
Other:
- board text added: "Rev A"
- board text removed: "ROWAN MOTORSPORTS Rev A"
Changed lines of the file:
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@@
 		)
 	)
-	(gr_text "ROWAN MOTORSPORTS\nRev A"
+	(gr_text "Rev A"
 		(at 112.95 68.275 0)
 		(layer "F.SilkS")

Commit message: can-module: Add indicator arrows for M2 mounting screws
Changed lines of the file:
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@@
+		)
+	)
+	(zone
+		(net 0)
+		(net_name "")
+		(layer "F.SilkS")
+		(hatch none 0.1)
+		(connect_pads
+			(clearance 0.1)
+		)
+		(min_thickness 0)
+		(filled_areas_thickness no)
+		(fill yes
+			(thermal_gap 0.5)
+			(thermal_bridge_width 0.5)
+		)
+		(polygon
+			(pts
+				(xy 126.5 52.5) (xy 127.25 53.25) (xy 126.5 54)
+			)
+		)
+	)
+	(zone
+		(net 0)
+		(net_name "")
+		(layer "F.SilkS")
+		(hatch none 0.1)
+		(connect_pads
+			(clearance 0.1)
+		)
+		(min_thickness 0)
+		(filled_areas_thickness no)
+		(fill yes
+			(thermal_gap 0.5)
+			(thermal_bridge_width 0.5)
+		)
+		(polygon
+			(pts
+				(xy 126.5 64.05) (xy 127.25 64.8) (xy 126.5 65.55)
+			)
 		)
 	)

Commit message: can-module, pmod-adapter: Begin updating PMOD adapter and CAN module
Parts:
- moved C11 17.6 mm to (141.0, 48.5)
- moved C12 13.3 mm to (146.2, 53.0)
- moved C3 11.5 mm to (128.0, 60.0), turned to -45 degrees
- moved C7 10.7 mm to (127.2, 60.8), turned to -45 degrees
- moved C9 9.07 mm to (118.2, 55.2), turned to 135 degrees
- moved R2 8.14 mm to (118.5, 45.5)
- moved TP3 7.77 mm to (114.8, 43.8)
- moved TP4 7.77 mm to (116.8, 43.8)
- moved R1 4.98 mm to (127.8, 57.8), turned to -135 degrees
- moved C10 4.52 mm to (127.0, 57.0), turned to 45 degrees
- moved C8 4.32 mm to (117.2, 61.8), turned to -135 degrees
- moved C2 4.18 mm to (126.2, 56.2), turned to 45 degrees
- moved C4 4.15 mm to (118.0, 62.5), turned to -135 degrees
- moved C1 4.02 mm to (124.0, 54.0), turned to 45 degrees
- moved C6 3.97 mm to (125.5, 55.5), turned to 45 degrees
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Connections:
- IC1 pad 10: PA05 -> Net-(IC1-PA05)
- IC1 pad 11: PA06 -> Net-(IC1-PA06)
- IC1 pad 12: PA07 -> Net-(IC1-PA07)
- IC1 pad 13: PA08 -> Net-(IC1-PA08)
- IC1 pad 14: PA09 -> Net-(IC1-PA09)
- IC1 pad 15: unconnected-(IC1-PA10-Pad15) -> Net-(IC1-PA10)
- IC1 pad 16: unconnected-(IC1-PA11-Pad16) -> Net-(IC1-PA11)
- IC1 pad 3: PA02 -> unconnected-(IC1-PA02-Pad3)
- IC1 pad 4: PA03 -> unconnected-(IC1-PA03-Pad4)
- IC1 pad 9: PA04 -> Net-(IC1-PA04)
- J1 pad 1: PA09 -> Net-(IC1-PA11)
- J1 pad 2: PA08 -> Net-(IC1-PA10)
- J1 pad 3: PA07 -> Net-(IC1-PA09)
- J1 pad 4: PA06 -> Net-(IC1-PA08)
- J1 pad 5: PA05 -> Net-(IC1-PA07)
- J1 pad 6: PA04 -> Net-(IC1-PA06)
- J1 pad 7: PA03 -> Net-(IC1-PA05)
- J1 pad 8: PA02 -> Net-(IC1-PA04)
Routing:
- net GND: track 30.4 -> 11.0 mm, vias 40 -> 17
- net CAN_STBY: track 13.2 -> 0.00 mm, vias 2 -> 0
- net CAN_NSIL: track 9.41 -> 0.00 mm
- net Net-(IC1-PA31_SWDIO): track 7.45 -> 0.00 mm
- net CAN_TX: track 3.16 -> 9.78 mm, vias 0 -> 2
- net PA04: track 6.28 -> 0.00 mm
- net PA09: track 6.24 -> 0.00 mm
- net PA05: track 5.94 -> 0.00 mm
- net PA02: track 5.42 -> 0.00 mm
- net Net-(IC1-PA30_SWCLK): track 6.91 -> 1.64 mm
- net PA08: track 5.11 -> 0.00 mm
- net PA03: track 5.10 -> 0.00 mm
- net PA06: track 4.97 -> 0.00 mm
- net PA07: track 4.65 -> 0.00 mm
- net CAN_RX: track 7.43 -> 6.08 mm, vias 2 -> 0
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- removed copper zone on B.Cu, net +5V
Other:
- board text added: "PA11"
- board text added: "PA4"
- board text removed: "PA2"
- board text removed: "PA9"

Commit message: can-module: Finish updating CAN module
Parts:
- TP3, TP4: moved to B.Cu
- moved TP3 14.0 mm to (126.5, 51.5), turned to 180 degrees
- moved C11 12.8 mm to (131.2, 56.8), turned to 0 degrees
- moved C12 11.1 mm to (135.4, 55.2), turned to 90 degrees
- moved TP4 10.9 mm to (124.5, 51.5), turned to 180 degrees
- moved R2 9.01 mm to (123.5, 53.0), turned to 45 degrees
- moved C4 0.71 mm to (118.5, 63.0)
- moved C8 0.71 mm to (117.8, 62.2)
- moved C1 0.35 mm to (124.2, 53.8)
Routing:
- net GND: track 11.0 -> 29.7 mm, vias 17 -> 36
- net CAN_STBY: track 0.00 -> 13.7 mm, vias 0 -> 2
- net CAN_NSIL: track 0.00 -> 9.35 mm
- net Net-(IC1-PA31_SWDIO): track 0.00 -> 7.57 mm, vias 0 -> 1
- net Net-(IC1-PA04): track 0.00 -> 5.37 mm
- net Net-(IC1-PA11): track 0.00 -> 5.37 mm
- net Net-(IC1-PA10): track 0.00 -> 4.64 mm
- net Net-(IC1-PA05): track 0.00 -> 4.64 mm
- net Net-(IC1-PA09): track 0.00 -> 3.91 mm
- net Net-(IC1-PA06): track 0.00 -> 3.91 mm
- net Net-(IC1-PA30_SWCLK): track 1.64 -> 5.44 mm, vias 0 -> 1
- net Net-(IC1-PA07): track 0.00 -> 3.17 mm
- net Net-(IC1-PA08): track 0.00 -> 3.17 mm

Commit message: can-module: Add power LED and indicator LED
Parts:
- added D4: LTST-C170GKT, LED_SMD:LED_0805_2012Metric, F.Cu at (114.7, 65.9)
- added D5: LTST-C170GKT, LED_SMD:LED_0805_2012Metric, F.Cu at (114.7, 52.2)
- added R5: 30k, Resistor_SMD:R_0402_1005Metric, F.Cu at (119.2, 63.7)
- added R6: 30k, Resistor_SMD:R_0402_1005Metric, F.Cu at (115.1, 50.6)
- moved C4 0.14 mm to (118.4, 62.9)
Connections:
- IC1 pad 21: unconnected-(IC1-PA12-Pad21) -> Net-(IC1-PA12)
Routing:
- net Net-(D4-A): track 0.00 -> 3.96 mm
- net GND: track 29.7 -> 31.4 mm, vias 36 -> 38
- net Net-(D5-A): track 0.00 -> 1.60 mm
- net Net-(IC1-PA12): track 0.00 -> 1.25 mm
Other:
- board text added: "A11"
- board text added: "A12"
- board text added: "A4"
- board text added: "PWR"
- board text removed: "PA11"
- board text removed: "PA4"

Commit message: can-module: Add more dimensions to User-1 layer
Parts:
- moved REF** 0.25 mm to (129.7, 64.5)

Commit message: can-module: Add 10uF bulk capacitor on module power output pin
Parts:
- added C14: 10u, Capacitor_SMD:C_0402_1005Metric, F.Cu at (118.4, 51.5)
Routing:
- net GND: track 31.4 -> 32.0 mm, vias 38 -> 39
Changed lines of the file:
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@@
 	(footprint "Capacitor_SMD:C_0402_1005Metric"
 		(layer "F.Cu")
+		(at 118.4 51.48 -90)
+		(descr "Capacitor SMD 0402 (1005 Metric), square (rectangular) end terminal, IPC-7351 nominal, (Body size source: IPC-SM-782 page 76, https://www.pcb-3d.com/wordpress/wp-content/uploads/ipc-sm-782a_amendment_1_and_2.pdf), generated with kicad-footprint-generator")
+		(tags "capacitor")
+		(property "Reference" "C14"
+			(at 0 -1.16 90)
+			(layer "F.SilkS")
+			(hide yes)
+			(effects
+				(font
+					(size 1 1)
+					(thickness 0.15)
+				)
+			)
+		)
+		(property "Value" "10u"
+			(at 0 1.16 90)
+			(layer "F.Fab")
+			(effects
+				(font
+					(size 1 1)
+					(thickness 0.15)
+				)
+			)
+		)
+		(property "Datasheet" "~"
+			(at 0 0 90)
+			(layer "F.Fab")
+			(hide yes)
+			(effects
+				(font
+					(size 1.27 1.27)
+					(thickness 0.15)
+				)
+			)
+		)
+		(property "Description" "Unpolarized capacitor"
+			(at 0 0 90)
+			(layer "F.Fab")
+			(hide yes)
+			(effects
+				(font
+					(size 1.27 1.27)
+					(thickness 0.15)
+				)
+			)
+		)
+		(property ki_fp_filters "C_*")
+		(sheetname "/")
+		(sheetfile "can-module.kicad_sch")
+		(attr smd)
+		(fp_line
+			(start -0.107836 0.36)
+			(end 0.107836 0.36)
+			(stroke
+				(width 0.12)
+				(type solid)
+			)
+			(layer "F.SilkS")
+		)
+		(fp_line
+			(start -0.107836 -0.36)
+			(end 0.107836 -0.36)
+			(stroke
+				(width 0.12)
+				(type solid)
+			)
+			(layer "F.SilkS")
+		)
+		(fp_rect
+			(start -0.91 -0.46)
+			(end 0.91 0.46)
+			(stroke
+				(width 0.05)
+				(type solid)
+			)
+			(fill no)
+			(layer "F.CrtYd")
+		)
+		(fp_rect
+			(start -0.5 -0.25)
+			(end 0.5 0.25)
+			(stroke
+				(width 0.1)
+				(type solid)
+			)
+			(fill no)
+			(layer "F.Fab")
+		)
+		(fp_text user "${REFERENCE}"
+			(at 0 0 90)
+			(layer "F.Fab")
+			(effects
+				(font
+					(size 0.25 0.25)
+					(thickness 0.04)
+				)
+			)
+		)
+		(pad "1" smd roundrect
+			(at -0.48 0 270)
+			(size 0.56 0.62)
+			(layers "F.Cu" "F.Mask" "F.Paste")
+			(roundrect_rratio 0.25)
+			(net 1 "+5V")
+			(pintype "passive")
+		)
+		(pad "2" smd roundrect
+			(at 0.48 0 270)
+			(size 0.56 0.62)
+			(layers "F.Cu" "F.Mask" "F.Paste")
+			(roundrect_rratio 0.25)
+			(net 2 "GND")
+			(pintype "passive")
+		)
+		(embedded_fonts no)
+		(model "${KICAD9_3DMODEL_DIR}/Capacitor_SMD.3dshapes/C_0402_1005Metric.step"
+			(offset
+				(xyz 0 0 0)
+			)
+			(scale
+				(xyz 1 1 1)
+			)
+			(rotate
+				(xyz 0 0 0)
+			)
+		)
+	)
+	(footprint "Capacitor_SMD:C_0402_1005Metric"
+		(layer "F.Cu")
 		(at 126.25 56.25 45)
 		(descr "Capacitor SMD 0402 (1005 Metric), square (rectangular) end terminal, IPC-7351 nominal, (Body size source: IPC-SM-782 page 76, https://www.pcb-3d.com/wordpress/wp-content/uploads/ipc-sm-782a_amendment_1_and_2.pdf), generated with kicad-footprint-generator")
@@
 	)
 	(segment
+		(start 118.4 52.6)
+		(end 118.4 51.96)
+		(width 0.25)
+		(layer "F.Cu")
+		(net 2)
+	)
+	(segment
 		(start 134.5 67.525)
 		(end 133.72 67.525)
@@
 		(size 0.4)
 		(drill 0.3)
+		(layers "F.Cu" "B.Cu")
+		(free yes)
+		(net 2)
+	)
+	(via
+		(at 118.4 52.6)
+		(size 0.4)
+		(drill 0.3)
