File: can-module/pcb/can-module.kicad_pcb (KiCad board)
At the start: 2 copper layers, 25.4 x 19 mm, 54 parts, among them J1 Conn_01x08_Socket, J2 Conn_01x02_Socket, J3 Conn_01x04_Socket, U1 PIC32CM1216JH01048-I_U5B, U2 ATA6560-GBQW-N, U3 NID5100GWH

Commit message: can-module: Reassign all reference designators by geographical position on schematic
Parts:
- renumbered C15 to C1, C13 to C10, C5 to C11, C6 to C12, C7 to C13, C8 to C14, C9 to C15, C16 to C2, C14 to C3, C10 to C4, C11 to C5, C1 to C6, C2 to C7, C3 to C8, C4 to C9, D3 to D2, D2 to D3, D5 to D4, D4 to D5, J3 to J1, J1 to J2, J2 to J3, JP2 to JP1, R7 to R1, R6 to R2, R2 to R3, R1 to R4, R3 to R5, R4 to R6, R5 to R7, TP14 to TP10, TP13 to TP11, TP11 to TP13, TP8 to TP14, TP9 to TP15, TP10 to TP16, TP3 to TP2, TP4 to TP3, TP2 to TP4, TP16 to TP8, TP15 to TP9, U3 to U1, U1 to U3

Commit message: can-module: Update CAN module to have selectable GPIO voltage (3.3V or 5V)
Parts:
- removed the C10 at (133.2, 67.5)
- removed the C6 at (118.5, 62.9)
- removed JP1: Jumper_2_Small_Open, Jumper:SolderJumper-2_P1.3mm_Open_Pad1.0x1.5mm
- added C4: 10u, Capacitor_SMD:C_0402_1005Metric, F.Cu at (128.5, 50.6)
- added C5: 10u, Capacitor_SMD:C_0402_1005Metric, F.Cu at (123.4, 50.8)
- added C8: 10u, Capacitor_SMD:C_0402_1005Metric, F.Cu at (116.5, 56.0)
- added U2: MIC5365-3.3YC5, Package_TO_SOT_SMD:SOT-353_SC-70-5, F.Cu at (125.8, 50.8)
- R5, R6: value 60 -> 0
- moved R5 24.8 mm to (113.8, 50.1)
- moved R6 24.7 mm to (114.8, 50.1), turned to 180 degrees
- moved R2 2.39 mm to (116.9, 52.2), turned to 90 degrees
- moved C12 0.24 mm to (117.5, 56.0), turned to -90 degrees
- renumbered C8 to C10, C9 to C11, C11 to C12, C12 to C13, C13 to C14, C14 to C15, C15 to C16, C4 to C6, C5 to C7, C7 to C9, D2 to D1, D3 to D2, D1 to D3, U2 to U3, U3 to U4
Connections:
- C10 pad 1: +5V -> VDD_{IO}
- C14 pad 1: +5V -> VDD_{IO}
- C15 pad 1: +5V -> VDD_{IO}
- J3 pad 2: +5V -> VDD_{IO}
- R5 pad 1: CANH -> VDD_{IO}
- R5 pad 2: Net-(C10-Pad2) -> +5V
- R6 pad 1: Net-(C10-Pad2) -> +3V3
- R6 pad 2: Net-(JP1-A) -> VDD_{IO}
- U4 pad 17: +5V -> VDD_{IO}
- U4 pad 36: +5V -> VDD_{IO}
Routing:
- net VDD_{IO}: track 0.00 -> 32.7 mm, vias 0 -> 2
- net CANL: track 20.8 -> 9.34 mm
- net CANH: track 20.7 -> 9.32 mm
- net +3V3: track 0.00 -> 10.1 mm
- net Net-(C10-Pad2): track 2.00 -> 0.00 mm
- net Net-(JP1-A): track 1.67 -> 0.00 mm
- net /PA04: track 5.37 -> 5.99 mm
- net GND: track 34.3 -> 34.4 mm, vias 42 -> 45
- added copper zone on F.Cu, net VDD_{IO}
Other:
- board text removed: "GND"
- board text removed: "J_{RCAN}"
- board text removed: "PWR"

Commit message: can-module: Change programming header to be through hole for easier access
Parts:
- removed TP2, TP3: TestPoint, TestPoints:TestPoint_Pad_D1.0mm_TightSpacing
- added J4: Conn_01x02_Socket, Connector_PinHeader_1.27mm:PinHeader_1x02_P1.27mm_Vertical, F.Cu at (129.4, 50.2)
- moved C4 0.67 mm to (127.8, 50.5), turned to 90 degrees
- moved C5 0.25 mm to (123.2, 50.8)
- moved U2 0.25 mm to (125.5, 50.8)
Connections:
- net Net-(U4-PA30_SWCLK) renamed /SWCLK
- U4 pad 46: Net-(U4-PA31_SWDIO) -> /SWDIO
Routing:
- net /SWDIO: track 0.00 -> 12.1 mm, vias 0 -> 2
- net Net-(U4-PA31_SWDIO): track 7.57 -> 0.00 mm, vias 1 -> 0
- net /SWCLK: track 5.44 -> 12.1 mm, vias 1 -> 2

Commit message: can-module: Label the GPIO voltage selector resistor
Other:
- board text added: "V_{IO}"
Changed lines of the file:
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@@
+		)
+	)
+	(gr_text "V_{IO}"
+		(at 115.75 50.1 180)
+		(layer "F.SilkS")
+		(effects
+			(font
+				(size 0.75 0.75)
+				(thickness 0.15)
+				(bold yes)
+			)
+			(justify right)
 		)
 	)

Commit message: can-module: Flip indicator LED around so that anode is always 5V
Parts:
- turned R2 to -90 degrees
- turned D4 to 180 degrees
- turned D5 to 180 degrees
Connections:
- D5 pad 1: GND -> Net-(D5-K)
- D5 pad 2: Net-(D5-A) -> +5V
- R7 pad 2: Net-(D5-A) -> Net-(D5-K)
Routing:
- net Net-(D5-K): track 0.00 -> 3.96 mm
- net Net-(D5-A): track 3.96 -> 0.00 mm
- net Net-(D4-A): track 1.47 -> 3.71 mm
- net GND: track 34.3 -> 33.1 mm, vias 45 -> 44
Changed lines of the file:
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@@
 	(net 6 "Net-(D4-A)")
 	(net 7 "CAN_NSIL")
-	(net 8 "Net-(D5-A)")
+	(net 8 "Net-(D5-K)")
 	(net 9 "CANL")
 	(net 10 "CANH")
@@
 	(footprint "LED_SMD:LED_0805_2012Metric"
 		(layer "F.Cu")
-		(at 114.7 65.9)
+		(at 114.7 65.9 180)
 		(descr "LED SMD 0805 (2012 Metric), square (rectangular) end terminal, IPC-7351 nominal, (Body size source: https://docs.google.com/spreadsheets/d/1BsfQQcO9C6DZCsRaXUlFlo91Tg2WpOkGARC1WS5S8t0/edit?usp=sharing), generated with kicad-footprint-generator")
 		(tags "LED")
@@
 		)
 		(property "Sim.Pin" "1=K 2=A"
-			(at 0 0 0)
+			(at 0 0 180)
 			(unlocked yes)
 			(layer "F.Fab")
@@
 		(attr smd)
 		(fp_line
-			(start -1.685 -0.96)
-			(end -1.685 0.96)
+			(start 1 -0.96)
+			(end -1.685 -0.96)
 			(stroke
 				(width 0.12)
@@
 		)
 		(fp_line
-			(start 1 -0.96)
-			(end -1.685 -0.96)
+			(start -1.685 -0.96)
+			(end -1.685 0.96)
 			(stroke
 				(width 0.12)
@@
 		)
 		(fp_line
-			(start -1.68 -0.95)
-			(end 1.68 -0.95)
+			(start 1.68 0.95)
+			(end -1.68 0.95)
 			(stroke
 				(width 0.05)
@@
 		)
 		(fp_line
-			(start -1.68 0.95)
-			(end -1.68 -0.95)
+			(start 1.68 -0.95)
+			(end 1.68 0.95)
 			(stroke
 				(width 0.05)
@@
 		)
 		(fp_line
-			(start 1.68 -0.95)
-			(end 1.68 0.95)
+			(start -1.68 0.95)
+			(end -1.68 -0.95)
 			(stroke
 				(width 0.05)
@@
 		)
 		(fp_line
-			(start 1.68 0.95)
-			(end -1.68 0.95)
+			(start -1.68 -0.95)
+			(end 1.68 -0.95)
 			(stroke
 				(width 0.05)
@@
 		)
 		(fp_line
-			(start -1 -0.3)
-			(end -1 0.6)
+			(start 1 0.6)
+			(end 1 -0.6)
 			(stroke
 				(width 0.1)
@@
 		)
 		(fp_line
-			(start -1 0.6)
-			(end 1 0.6)
+			(start 1 -0.6)
+			(end -0.7 -0.6)
 			(stroke
 				(width 0.1)
@@
 		)
 		(fp_line
-			(start 1 -0.6)
-			(end -0.7 -0.6)
+			(start -1 0.6)
+			(end 1 0.6)
 			(stroke
 				(width 0.1)
@@
 		)
 		(fp_line
-			(start 1 0.6)
-			(end 1 -0.6)
+			(start -1 -0.3)
+			(end -1 0.6)
 			(stroke
 				(width 0.1)
@@
 		)
 		(pad "1" smd roundrect
-			(at -0.9375 0)
+			(at -0.9375 0 180)
 			(size 0.975 1.4)
 			(layers "F.Cu" "F.Mask" "F.Paste")
 			(roundrect_rratio 0.25)
-			(net 2 "GND")
+			(net 8 "Net-(D5-K)")
 			(pinfunction "K")
 			(pintype "passive")
 		)
 		(pad "2" smd roundrect
-			(at 0.9375 0)
+			(at 0.9375 0 180)
 			(size 0.975 1.4)
 			(layers "F.Cu" "F.Mask" "F.Paste")
 			(roundrect_rratio 0.25)
-			(net 8 "Net-(D5-A)")
+			(net 1 "+5V")
 			(pinfunction "A")
 			(pintype "passive")
@@
 	(footprint "LED_SMD:LED_0805_2012Metric"
 		(layer "F.Cu")
-		(at 114.7 52.2)
+		(at 114.7 52.2 180)
 		(descr "LED SMD 0805 (2012 Metric), square (rectangular) end terminal, IPC-7351 nominal, (Body size source: https://docs.google.com/spreadsheets/d/1BsfQQcO9C6DZCsRaXUlFlo91Tg2WpOkGARC1WS5S8t0/edit?usp=sharing), generated with kicad-footprint-generator")
 		(tags "LED")
@@
 		)
 		(property "Sim.Pin" "1=K 2=A"
-			(at 0 0 0)
+			(at 0 0 180)
 			(unlocked yes)
 			(layer "F.Fab")
@@
 		(attr smd)
 		(fp_line
-			(start -1.685 -0.96)
-			(end -1.685 0.96)
+			(start 1 -0.96)
+			(end -1.685 -0.96)
 			(stroke
 				(width 0.12)
@@
 		)
 		(fp_line
-			(start 1 -0.96)
-			(end -1.685 -0.96)
+			(start -1.685 -0.96)
+			(end -1.685 0.96)
 			(stroke
 				(width 0.12)
@@
 		)
 		(fp_line
-			(start -1.68 -0.95)
-			(end 1.68 -0.95)
+			(start 1.68 0.95)
+			(end -1.68 0.95)
 			(stroke
 				(width 0.05)
@@
 		)
 		(fp_line
-			(start -1.68 0.95)
-			(end -1.68 -0.95)
+			(start 1.68 -0.95)
+			(end 1.68 0.95)
 			(stroke
 				(width 0.05)
@@
 		)
 		(fp_line
-			(start 1.68 -0.95)
-			(end 1.68 0.95)
+			(start -1.68 0.95)
+			(end -1.68 -0.95)
 			(stroke
 				(width 0.05)
@@
 		)
 		(fp_line
-			(start 1.68 0.95)
-			(end -1.68 0.95)
+			(start -1.68 -0.95)
+			(end 1.68 -0.95)
 			(stroke
 				(width 0.05)
@@
 		)
 		(fp_line
-			(start -1 -0.3)
-			(end -1 0.6)
+			(start 1 0.6)
+			(end 1 -0.6)
 			(stroke
 				(width 0.1)
@@
 		)
 		(fp_line
-			(start -1 0.6)
-			(end 1 0.6)
+			(start 1 -0.6)
+			(end -0.7 -0.6)
 			(stroke
 				(width 0.1)
@@
 		)
 		(fp_line
-			(start 1 -0.6)
-			(end -0.7 -0.6)
+			(start -1 0.6)
+			(end 1 0.6)
 			(stroke
 				(width 0.1)
@@
 		)
 		(fp_line
-			(start 1 0.6)
-			(end 1 -0.6)
+			(start -1 -0.3)
+			(end -1 0.6)
 			(stroke
 				(width 0.1)
@@
 		)
 		(pad "1" smd roundrect
-			(at -0.9375 0)
+			(at -0.9375 0 180)
 			(size 0.975 1.4)
 			(layers "F.Cu" "F.Mask" "F.Paste")
@@
 		)
 		(pad "2" smd roundrect
-			(at 0.9375 0)
+			(at 0.9375 0 180)
 			(size 0.975 1.4)
 			(layers "F.Cu" "F.Mask" "F.Paste")
@@
 			(layers "F.Cu" "F.Mask" "F.Paste")
 			(roundrect_rratio 0.25)
-			(net 8 "Net-(D5-A)")
+			(net 8 "Net-(D5-K)")
 			(pintype "passive")
 		)
@@
 	(footprint "Resistor_SMD:R_0402_1005Metric"
 		(layer "F.Cu")
-		(at 116.9 52.2 90)
+		(at 116.95 52.2 -90)
 		(descr "Resistor SMD 0402 (1005 Metric), square (rectangular) end terminal, IPC-7351 nominal, (Body size source: IPC-SM-782 page 72, https://www.pcb-3d.com/wordpress/wp-content/uploads/ipc-sm-782a_amendment_1_and_2.pdf), generated with kicad-footprint-generator")
 		(tags "resistor")
@@
 		(attr smd)
 		(fp_line
-			(start -0.153641 -0.38)
-			(end 0.153641 -0.38)
+			(start -0.153641 0.38)
+			(end 0.153641 0.38)
 			(stroke
 				(width 0.12)
@@
 		)
 		(fp_line
-			(start -0.153641 0.38)
-			(end 0.153641 0.38)
+			(start -0.153641 -0.38)
+			(end 0.153641 -0.38)
 			(stroke
 				(width 0.12)
@@
 		)
 		(fp_line
-			(start 0.93 -0.47)
-			(end 0.93 0.47)
+			(start -0.93 0.47)
+			(end -0.93 -0.47)
 			(stroke
 				(width 0.05)
@@
 		)
 		(fp_line
-			(start -0.93 -0.47)
-			(end 0.93 -0.47)
+			(start 0.93 0.47)
+			(end -0.93 0.47)
 			(stroke
 				(width 0.05)
@@
 		)
 		(fp_line
-			(start 0.93 0.47)
-			(end -0.93 0.47)
+			(start -0.93 -0.47)
+			(end 0.93 -0.47)
 			(stroke
 				(width 0.05)
@@
 		)
 		(fp_line
-			(start -0.93 0.47)
-			(end -0.93 -0.47)
+			(start 0.93 -0.47)
+			(end 0.93 0.47)
 			(stroke
 				(width 0.05)
@@
 		)
 		(fp_line
-			(start 0.525 -0.27)
-			(end 0.525 0.27)
+			(start -0.525 0.27)
+			(end -0.525 -0.27)
 			(stroke
 				(width 0.1)
@@
 		)
 		(fp_line
-			(start -0.525 -0.27)
-			(end 0.525 -0.27)
+			(start 0.525 0.27)
+			(end -0.525 0.27)
 			(stroke
 				(width 0.1)
@@
 		)
 		(fp_line
-			(start 0.525 0.27)
-			(end -0.525 0.27)
+			(start -0.525 -0.27)
+			(end 0.525 -0.27)
 			(stroke
 				(width 0.1)
@@
 		)
 		(fp_line
-			(start -0.525 0.27)
-			(end -0.525 -0.27)
+			(start 0.525 -0.27)
+			(end 0.525 0.27)
 			(stroke
 				(width 0.1)
@@
 		)
 		(pad "1" smd roundrect
-			(at -0.509999 0 90)
+			(at -0.509999 0 270)
 			(size 0.54 0.64)
 			(layers "F.Cu" "F.Mask" "F.Paste")
@@
 		)
 		(pad "2" smd roundrect
-			(at 0.509999 0 90)
+			(at 0.509999 0 270)
 			(size 0.54 0.64)
 			(layers "F.Cu" "F.Mask" "F.Paste")
@@
 	)
 	(segment
-		(start 113.7625 66.9)
-		(end 113.7625 65.9)
-		(width 0.127)
-		(layer "F.Cu")
-		(net 2)
-	)
-	(segment
 		(start 127.978822 60.7)
 		(end 127.978822 60.678822)
@@
 	)
 	(segment
-		(start 113.7625 51.2)
-		(end 113.7625 52.2)
-		(width 0.127)
-		(layer "F.Cu")
-		(net 2)
-	)
-	(segment
 		(start 127.978822 60.7)
 		(end 127.589411 61.089411)
@@
 	)
 	(segment
+		(start 114.8 52.2)
+		(end 115.6375 52.2)
+		(width 0.127)
+		(layer "F.Cu")
+		(net 2)
+	)
+	(segment
 		(start 129.75 58.6948)
 		(end 129 58.6948)
@@
 	)
 	(via
-		(at 133.25 50.25)
+		(at 114.8 52.2)
 		(size 0.4)
 		(drill 0.3)
@@
 	)
 	(via
-		(at 113.7625 51.2)
+		(at 133.25 50.25)
 		(size 0.4)
 		(drill 0.3)
@@
 	)
 	(via
-		(at 113.7625 66.9)
-		(size 0.4)
-		(drill 0.3)
-		(layers "F.Cu" "B.Cu")
-		(net 2)
-	)
-	(via
 		(at 117 63)
 		(size 0.4)
@@
 	)
 	(segment
-		(start 116.390001 52.2)
-		(end 115.6375 52.2)
+		(start 116.568499 53.0915)
+		(end 114.654 53.0915)
+		(width 0.127)
+		(layer "F.Cu")
+		(net 6)
+	)
+	(segment
+		(start 116.95 52.709999)
+		(end 116.568499 53.0915)
 		(width 0.127)
 		(layer "F.Cu")
@@
 	)
 	(segment
-		(start 116.9 51.690001)
-		(end 116.390001 52.2)
+		(start 114.654 53.0915)
+		(end 113.7625 52.2)
 		(width 0.127)
 		(layer "F.Cu")
@@
 	)
 	(segment
-		(start 118.789376 63.960624)
-		(end 116.85 65.9)
+		(start 116.85 65.9)
+		(end 115.6375 65.9)
 		(width 0.127)
 		(layer "F.Cu")
@@
 	)
 	(segment
-		(start 116.85 65.9)
-		(end 115.6375 65.9)
+		(start 118.789376 63.960624)
+		(end 116.85 65.9)
 		(width 0.127)
 		(layer "F.Cu")

Commit message: can-module: Revert back to only having 5V logic on the board
Parts:
- removed the C4 at (127.8, 50.5)
- removed the C5 at (123.2, 50.8)
- removed the R5 at (113.8, 50.1)
- removed R6: 0, Resistor_SMD:R_0402_1005Metric
- removed the U2 at (125.5, 50.8)
- moved J2 3.48 mm to (126.0, 50.2)
- renumbered C8 to C1, C1 to C10, C6 to C11, C2 to C12, C3 to C13, C7 to C14, C12 to C2, C13 to C3, C9 to C4, C14 to C5, C10 to C6, C15 to C7, C11 to C8, C16 to C9, D5 to D4, D4 to D5, J4 to J2, J2 to J3, J3 to J4, R7 to R1, R4 to R2, R1 to R3, R2 to R4, R3 to R5, TP4 to TP1, TP1 to TP14, TP5 to TP2, TP6 to TP3, TP7 to TP4, TP14 to TP5, TP15 to TP6, TP16 to TP7, U4 to U1, U1 to U2
Connections:
- C5 pad 1: VDD_{IO} -> +5V
- C6 pad 1: VDD_{IO} -> +5V
- C7 pad 1: VDD_{IO} -> +5V
- J4 pad 2: VDD_{IO} -> +5V
- U1 pad 17: VDD_{IO} -> +5V
- U1 pad 36: VDD_{IO} -> +5V
Routing:
- net VDD_{IO}: track 33.2 -> 0.00 mm, vias 2 -> 0
- net +5V: track 0.00 -> 12.1 mm
- net +3V3: track 9.82 -> 0.00 mm
- net /SWCLK: track 12.1 -> 7.88 mm, vias 2 -> 1
- net /SWDIO: track 12.1 -> 8.99 mm, vias 2 -> 1
- net GND: track 33.1 -> 31.1 mm, vias 44 -> 41
- removed copper zone on F.Cu, net VDD_{IO}
Other:
- board text removed: "V_{IO}"

Commit message: can-module: Re-attach microcontroller GND pins to bottom plane
Routing:
- net +5V: track 12.1 -> 0.92 mm
- net GND: track 31.1 -> 32.0 mm, vias 41 -> 40
Changed lines of the file:
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@@
-	)
-	(segment
-		(start 121.829323 62.928811)
-		(end 121.670677 62.928811)
-		(width 0.127)
-		(layer "F.Cu")
-		(net 1)
-	)
-	(segment
-		(start 125.958134 59.25)
-		(end 125.508134 59.25)
-		(width 0.127)
-		(layer "F.Cu")
-		(net 1)
 	)
 	(segment
@@
 	)
 	(segment
-		(start 125.508134 59.25)
-		(end 121.829323 62.928811)
-		(width 0.127)
-		(layer "F.Cu")
-		(net 1)
-	)
-	(segment
 		(start 120.115 51.236)
 		(end 120.115 51)
@@
 	)
 	(segment
-		(start 118.459779 61.240221)
-		(end 118.4 61.3)
-		(width 0.25)
-		(layer "F.Cu")
-		(net 1)
-	)
-	(segment
-		(start 121.670677 62.928811)
-		(end 119.431522 60.689656)
-		(width 0.127)
-		(layer "F.Cu")
-		(net 1)
-	)
-	(segment
-		(start 118.089411 61.624929)
-		(end 118.089411 61.910589)
-		(width 0.25)
-		(layer "F.Cu")
-		(net 1)
-	)
-	(segment
 		(start 119.024684 60.689656)
 		(end 118.780152 60.934188)
@@
 	)
 	(segment
-		(start 119.431522 60.689656)
-		(end 119.024684 60.689656)
-		(width 0.127)
-		(layer "F.Cu")
-		(net 1)
-	)
-	(segment
-		(start 118.780152 60.934188)
-		(end 118.474119 61.240221)
-		(width 0.25)
-		(layer "F.Cu")
-		(net 1)
-	)
-	(segment
-		(start 118.780152 60.934188)
-		(end 118.089411 61.624929)
-		(width 0.25)
-		(layer "F.Cu")
-		(net 1)
-	)
-	(segment
 		(start 126.134062 59.425928)
 		(end 125.958134 59.25)
@@
 	)
 	(segment
-		(start 118.474119 61.240221)
-		(end 118.459779 61.240221)
-		(width 0.25)
-		(layer "F.Cu")
-		(net 1)
-	)
-	(segment
 		(start 127.978822 60.7)
 		(end 127.978822 60.678822)
@@
 	)
 	(segment
-		(start 124.93198 59.025)
-		(end 121.75 59.025)
-		(width 0.127)
-		(layer "F.Cu")
-		(net 2)
-	)
-	(segment
 		(start 136.750118 64.325118)
 		(end 137.249836 64.325118)
@@
 	)
 	(segment
-		(start 127.589411 61.089411)
-		(end 126.793209 61.089411)
-		(width 0.25)
-		(layer "F.Cu")
-		(net 2)
-	)
-	(segment
 		(start 121.75 57.96434)
 		(end 121.75 59.025)
@@
 	)
 	(segment
+		(start 124.93198 59.025)
+		(end 125.780509 59.873529)
+		(width 0.25)
+		(layer "F.Cu")
+		(net 2)
+	)
+	(segment
+		(start 121.75 59.025)
+		(end 124.93198 59.025)
+		(width 0.127)
+		(layer "F.Cu")
+		(net 2)
+	)
+	(segment
 		(start 129.75 58.6948)
 		(end 129 58.6948)
@@
 	)
 	(segment
-		(start 126.25 60.34302)
-		(end 125.780509 59.873529)
-		(width 0.25)
-		(layer "F.Cu")
-		(net 2)
-	)
-	(segment
 		(start 134 51.6)
 		(end 134 51)
@@
 	)
 	(segment
+		(start 121.396447 59.025)
+		(end 121.75 59.025)
+		(width 0.127)
+		(layer "F.Cu")
+		(net 2)
+	)
+	(segment
 		(start 135.25 55.25)
 		(end 135.25 55.75)
@@
 	)
 	(segment
-		(start 126.793209 61.089411)
-		(end 126.25 60.546202)
-		(width 0.25)
-		(layer "F.Cu")
-		(net 2)
-	)
-	(segment
 		(start 122.103553 59.025)
 		(end 121.75 59.025)
@@
 	)
 	(segment
-		(start 118.75 61.671447)
-		(end 119.133705 61.287742)
-		(width 0.25)
-		(layer "F.Cu")
-		(net 2)
-	)
-	(segment
 		(start 126 54.7)
 		(end 125.639411 55.060589)
@@
 	)
 	(segment
-		(start 121.396447 59.025)
-		(end 121.75 59.025)
-		(width 0.127)
-		(layer "F.Cu")
-		(net 2)
-	)
-	(segment
 		(start 117.8 51.98)
 		(end 118.4 51.98)
@@
 	)
 	(segment
+		(start 119.133705 61.287742)
+		(end 121.396447 59.025)
+		(width 0.25)
+		(layer "F.Cu")
+		(net 2)
+	)
+	(segment
 		(start 124.366295 56.762258)
 		(end 122.103553 59.025)
@@
 	)
 	(segment
-		(start 126.25 60.546202)
-		(end 126.25 60.34302)
-		(width 0.25)
-		(layer "F.Cu")
-		(net 2)
-	)
-	(segment
 		(start 136.750114 63.775)
 		(end 136.750114 64.325114)
@@
 		(net 2)
 	)
-	(segment
-		(start 118.75 62.25)
-		(end 118.75 61.671447)
-		(width 0.25)
-		(layer "F.Cu")
-		(net 2)
-	)
 	(via
 		(at 114.8 52.2)
@@
 		(size 0.4)
 		(drill 0.3)
-		(layers "F.Cu" "B.Cu")
-		(free yes)
-		(net 2)
-	)
-	(via
-		(at 118.75 62.25)
-		(size 0.4)
-		(drill 0.3)
