File: can-module/pcb/can-module.kicad_sch (KiCad schematic)
At the start: 25 parts, among them IC1 PIC32CM1216JH01048-I_U5B, J1 Conn_01x08_Socket, J3 Conn_01x04_Socket, U1 ATA6560-GBQW-N

Commit message: can-module: Add 5V output for daughter boards
Parts:
- added J2: Conn_01x02_Socket, Conn_01x02:Untitled, symbol Connector:Conn_01x02_Socket
Connections:
- net +5V: now also J2.2 (Pin_2)
- net GND: now also J2.1 (Pin_1)
Other:
- note added: "GPIO Power Header"
Changed lines of the file:
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@@
 		)
 	)
+	(text "GPIO Power Header"
+		(exclude_from_sim no)
+		(at 83.058 156.21 90)
+		(effects
+			(font
+				(size 1.27 1.27)
+				(thickness 0.1588)
+			)
+		)
+	)
 	(text "Main connector"
 		(exclude_from_sim no)
@@
 	(wire
 		(pts
+			(xy 93.98 157.48) (xy 96.52 157.48)
+		)
+		(stroke
+			(width 0)
+			(type default)
+		)
+	)
+	(wire
+		(pts
 			(xy 30.48 86.36) (xy 41.91 86.36)
 		)
@@
 	(wire
 		(pts
+			(xy 93.98 154.94) (xy 96.52 154.94)
+		)
+		(stroke
+			(width 0)
+			(type default)
+		)
+	)
+	(wire
+		(pts
 			(xy 39.37 127) (xy 49.53 127)
 		)
@@
 	)
 	(symbol
+		(lib_id "power:GND")
+		(at 96.52 157.48 90)
+		(unit 1)
+		(exclude_from_sim no)
+		(in_bom yes)
+		(on_board yes)
+		(dnp no)
+		(fields_autoplaced yes)
+		(property "Reference" "#PWR044"
+			(at 102.87 157.48 0)
+			(effects
+				(font
+					(size 1.27 1.27)
+				)
+				(hide yes)
+			)
+		)
+		(property "Value" "GND"
+			(at 100.33 157.4799 90)
+			(effects
+				(font
+					(size 1.27 1.27)
+				)
+				(justify right)
+			)
+		)
+		(property "Footprint" ""
+			(at 96.52 157.48 0)
+			(effects
+				(font
+					(size 1.27 1.27)
+				)
+				(hide yes)
+			)
+		)
+		(property "Datasheet" ""
+			(at 96.52 157.48 0)
+			(effects
+				(font
+					(size 1.27 1.27)
+				)
+				(hide yes)
+			)
+		)
+		(property "Description" "Power symbol creates a global label with name \"GND\" , ground"
+			(at 96.52 157.48 0)
+			(effects
+				(font
+					(size 1.27 1.27)
+				)
+				(hide yes)
+			)
+		)
+		(pin "1"
+		)
+		(instances
+			(project "can-module"
+				(path "/40cb4209-4f7f-4a38-b0f0-dee54a92ee91"
+					(reference "#PWR044")
+					(unit 1)
+				)
+			)
+		)
+	)
+	(symbol
 		(lib_id "power:+5V")
 		(at 168.91 101.6 270)
@@
 	)
 	(symbol
+		(lib_id "Connector:Conn_01x02_Socket")
+		(at 88.9 157.48 180)
+		(unit 1)
+		(exclude_from_sim no)
+		(in_bom yes)
+		(on_board yes)
+		(dnp no)
+		(property "Reference" "J2"
+			(at 87.63 156.21 0)
+			(effects
+				(font
+					(size 1.27 1.27)
+				)
+				(justify left)
+			)
+		)
+		(property "Value" "Conn_01x02_Socket"
+			(at 87.63 154.9401 0)
+			(effects
+				(font
+					(size 1.27 1.27)
+				)
+				(justify left)
+				(hide yes)
+			)
+		)
+		(property "Footprint" "Conn_01x02:Untitled"
+			(at 88.9 157.48 0)
+			(effects
+				(font
+					(size 1.27 1.27)
+				)
+				(hide yes)
+			)
+		)
+		(property "Datasheet" "~"
+			(at 88.9 157.48 0)
+			(effects
+				(font
+					(size 1.27 1.27)
+				)
+				(hide yes)
+			)
+		)
+		(property "Description" "Generic connector, single row, 01x02, script generated"
+			(at 88.9 157.48 0)
+			(effects
+				(font
+					(size 1.27 1.27)
+				)
+				(hide yes)
+			)
+		)
+		(pin "1"
+		)
+		(pin "2"
+		)
+		(instances
+			(project ""
+				(path "/40cb4209-4f7f-4a38-b0f0-dee54a92ee91"
+					(reference "J2")
+					(unit 1)
+				)
+			)
+		)
+	)
+	(symbol
 		(lib_id "Device:C_Small")
 		(at 170.18 69.85 0)
@@
 					(unit 1)
 				)
+			)
+		)
+	)
+	(symbol
+		(lib_id "power:+5V")
+		(at 96.52 154.94 270)
+		(unit 1)
+		(exclude_from_sim no)
+		(in_bom yes)
+		(on_board yes)
+		(dnp no)
+		(fields_autoplaced yes)
+		(property "Reference" "#PWR043"
+			(at 92.71 154.94 0)
+			(effects
+				(font
+					(size 1.27 1.27)
+				)
+				(hide yes)
+			)
+		)
+		(property "Value" "+5V"
+			(at 100.33 154.9399 90)
+			(effects
+				(font
+					(size 1.27 1.27)
+				)
+				(justify left)
+			)
+		)
+		(property "Footprint" ""
+			(at 96.52 154.94 0)
+			(effects
+				(font
+					(size 1.27 1.27)
+				)
+				(hide yes)
+			)
+		)
+		(property "Datasheet" ""
+			(at 96.52 154.94 0)
+			(effects
+				(font
+					(size 1.27 1.27)
+				)
+				(hide yes)
+			)
+		)
+		(property "Description" "Power symbol creates a global label with name \"+5V\""
+			(at 96.52 154.94 0)
+			(effects
+				(font
+					(size 1.27 1.27)
+				)
+				(hide yes)
+			)
+		)
+		(pin "1"
+		)
+		(instances
+			(project "can-module"
+				(path "/40cb4209-4f7f-4a38-b0f0-dee54a92ee91"
+					(reference "#PWR043")
+					(unit 1)
+				)

Commit message: can-module: Major changes to routing, placement; remove pull up/down resistors (use PIC32 internal resistors)
Parts:
- added C13: 4n7, Capacitor_SMD:C_0402_1005Metric, symbol Device:C_Small
- added R4: 60, Resistor_SMD:R_0402_1005Metric, symbol Device:R
- R3: value 120 -> 60
Connections:
- net CANH: now also R3.1; no longer JP2.1 (A)
- net CANL: now also JP2.2 (B); no longer R3.1
- net GND: now also C13.1
- net at R3.2: now also C13.2, R4.1; no longer JP2.2 (B)
- new net: JP2.1 (A), R4.2
Other:
- removed sheet GPIO Resistors
- note added: "CAN Termination"
- moved on the sheet: C11, JP2, R3, U1

Commit message: can-module: Update ESD diode component
Other:
- note added: "*All TVS diodes are DESD5V0S1BA-7 unless otherwise noted"
- note removed: "*All TVS diodes are PESD5V0S1BAF unless otherwise noted"
Changed lines of the file:
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@@
 		)
 	)
-	(text "*All TVS diodes are PESD5V0S1BAF\nunless otherwise noted"
+	(text "*All TVS diodes are DESD5V0S1BA-7\nunless otherwise noted"
 		(exclude_from_sim no)
 		(at 238.252 28.702 0)

Commit message: can-module: Change header size from 1mm spacing to 1.27mm spacing
Parts:
- J1: footprint Conn_01x08:Untitled -> Connector_PinHeader_1.27mm:PinHeader_1x08_P1.27mm_Vertical
- J2: footprint Conn_01x02:Untitled -> Connector_PinHeader_1.27mm:PinHeader_1x02_P1.27mm_Vertical
Connections:
- no-connect marks 22 -> 24
Changed lines of the file:
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@@
 	)
 	(no_connect
+		(at 135.89 152.4)
+	)
+	(no_connect
 		(at 166.37 121.92)
 	)
@@
 	)
 	(no_connect
+		(at 133.35 152.4)
+	)
+	(no_connect
 		(at 120.65 119.38)
 	)
@@
 	(wire
 		(pts
-			(xy 133.35 152.4) (xy 133.35 160.02)
-		)
-		(stroke
-			(width 0)
-			(type default)
-		)
-	)
-	(wire
-		(pts
 			(xy 39.37 119.38) (xy 49.53 119.38)
 		)
@@
 	(wire
 		(pts
-			(xy 135.89 152.4) (xy 135.89 162.56)
-		)
-		(stroke
-			(width 0)
-			(type default)
-		)
-	)
-	(wire
-		(pts
 			(xy 106.68 104.14) (xy 106.68 111.76)
 		)
@@
 			)
 		)
-		(property "Footprint" "Conn_01x02:Untitled"
+		(property "Footprint" "Connector_PinHeader_1.27mm:PinHeader_1x02_P1.27mm_Vertical"
 			(at 88.9 157.48 0)
 			(effects
@@
 			)
 		)
-		(property "Footprint" "Conn_01x08:Untitled"
+		(property "Footprint" "Connector_PinHeader_1.27mm:PinHeader_1x08_P1.27mm_Vertical"
 			(at 87.63 116.84 0)
 			(effects

Commit message: can-module: Update CAN/PWR header to also be 0.127mm, move some things around to allow for wider min power plane width
Parts:
- J3: footprint Conn01x04:01x04_1mm -> Connector_PinHeader_1.27mm:PinHeader_1x04_P1.27mm_Vertical
Changed lines of the file:
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@@
 			)
 		)
-		(property "Footprint" "Conn01x04:01x04_1mm"
+		(property "Footprint" "Connector_PinHeader_1.27mm:PinHeader_1x04_P1.27mm_Vertical"
 			(at 209.55 41.91 0)
 			(effects

Commit message: can-module, pmod-adapter: Begin updating PMOD adapter and CAN module
Connections:
- net at IC1.15 (PA10): now also J1.2 (Pin_2)
- net at IC1.16 (PA11): now also J1.1 (Pin_1)
- net PA02: no longer names the net of IC1.3 (PA02)
- net PA02: no longer J1.8 (Pin_8)
- net PA03: no longer names the net of J1.7 (Pin_7)
- net PA03: now also IC1.10 (PA05); no longer IC1.4 (PA03)
- net PA04: no longer names the net of J1.6 (Pin_6)
- net PA04: now also IC1.11 (PA06); no longer IC1.9 (PA04)
- net PA05: no longer names the net of J1.5 (Pin_5)
- net PA05: now also IC1.12 (PA07); no longer IC1.10 (PA05)
- net PA06: no longer names the net of J1.4 (Pin_4)
- net PA06: now also IC1.13 (PA08); no longer IC1.11 (PA06)
- net PA07: no longer names the net of J1.3 (Pin_3)
- net PA07: now also IC1.14 (PA09); no longer IC1.12 (PA07)
- removed net PA08: IC1.13 (PA08), J1.2 (Pin_2)
- removed net PA09: IC1.14 (PA09), J1.1 (Pin_1)
- new net: IC1.9 (PA04), J1.8 (Pin_8)
Other:
- moved on the sheet: J1

Commit message: can-module: Add power LED and indicator LED
Parts:
- added D4, D5: LTST-C170GKT, LED_SMD:LED_0805_2012Metric, symbol Device:LED_Small
- added R5, R6: 30k, Resistor_SMD:R_0402_1005Metric, symbol Device:R_Small
Connections:
- net +5V: now also R6.1
- net GND: now also D4.1 (K), D5.1 (K)
- net at IC1.21 (PA12): now also R5.1
- new net: D4.2 (A), R5.2
- new net: D5.2 (A), R6.2
- no-connect marks 24 -> 23

Commit message: can-module: Update sch info
Other:
- company: (none) -> Ryan Hausmann
- title: (none) -> CAN Module
Changed lines of the file:
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@@
 	(generator_version "9.0")
 	(paper "A4")
+	(title_block
+		(title "CAN Module")
+		(date "2026-02-10")
+		(rev "A")
+		(company "Ryan Hausmann")
+		(comment 1 "Rowan Motorsports")
+	)
 	(text "1x decoupling cap for each power pin"
 		(exclude_from_sim no)
