File: can-module/pcb/can-module.kicad_sch (KiCad schematic)
At the start: 33 parts, among them IC1 PIC32CM1216JH01048-I_U5B, J1 Conn_01x08_Socket, J2 Conn_01x02_Socket, J3 Conn_01x04_Socket, U1 ATA6560-GBQW-N

Commit message: can-module: Switch to using DESD5V0U1BA-7 TVS diodes
Parts:
- D1, D2, D3: value PESD5V0S1BAF -> DESD5V0U1BA-7
Other:
- note added: "*All TVS diodes are DESD5V0U1BA-7 unless otherwise noted"
- note removed: "*All TVS diodes are DESD5V0S1BA-7 unless otherwise noted"
Changed lines of the file:
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@@
 		)
 	)
-	(text "*All TVS diodes are DESD5V0S1BA-7\nunless otherwise noted"
+	(text "*All TVS diodes are DESD5V0U1BA-7\nunless otherwise noted"
 		(exclude_from_sim no)
 		(at 238.252 25.146 0)
@@
 			)
 		)
-		(property "Value" "PESD5V0S1BAF"
+		(property "Value" "DESD5V0U1BA-7"
 			(at 224.79 52.0699 90)
 			(effects
@@
 			)
 		)
-		(property "Value" "PESD5V0S1BAF"
+		(property "Value" "DESD5V0U1BA-7"
 			(at 229.87 52.0699 90)
 			(effects
@@
 			)
 		)
-		(property "Value" "PESD5V0S1BAF"
+		(property "Value" "DESD5V0U1BA-7"
 			(at 219.71 52.0699 90)
 			(effects

Commit message: can-module: Update CAN Module schematic to include power filtering & reverse polarity protection
Parts:
- removed C12: 10u, Capacitor_SMD:C_0402_1005Metric, symbol Device:C_Small
- added C15, C16: 10u, Capacitor_SMD:C_0402_1005Metric, symbol Device:C_Small
- added F1: 1206L050YR, Fuse:Fuse_1206_3216Metric, symbol Device:Polyfuse_Small
- added IC2: NID5100GWH, NID5100GWH:NID5100GWH, symbol NID5100GWH:NID5100GWH
- added R7: 30k, Resistor_SMD:R_0402_1005Metric, symbol Device:R_Small
Connections:
- net +5V: now also C16.1, IC2.6 (OUT), R7.1; no longer D1.2 (A2), J3.4 (Pin_4)
- net GND: now also C15.2, C16.2, IC2.2 (GND), IC2.3 (~{EN})
- net PA05: now reaches IC1.10 (PA05)
- net PA05: now also J1.2 (Pin_2); no longer J1.7 (Pin_7)
- net PA06: now reaches IC1.11 (PA06)
- net PA06: now also J1.3 (Pin_3); no longer J1.6 (Pin_6)
- net PA07: now reaches IC1.12 (PA07)
- net PA07: now also J1.4 (Pin_4); no longer J1.5 (Pin_5)
- net PA08: now reaches IC1.13 (PA08)
- net PA08: now also J1.5 (Pin_5); no longer J1.4 (Pin_4)
- net PA09: now reaches IC1.14 (PA09)
- net PA09: now also J1.6 (Pin_6); no longer J1.3 (Pin_3)
- net PA10: now reaches IC1.15 (PA10)
- net PA10: now also J1.7 (Pin_7); no longer J1.2 (Pin_2)
- net PA04: now reaches J1.1 (Pin_1)
- net PA04: now also IC1.9 (PA04); no longer IC1.16 (PA11)
- net PA11: now reaches J1.8 (Pin_8)
- net PA11: now also IC1.16 (PA11); no longer IC1.9 (PA04)
- new net: C15.1, F1.2, IC2.1 (IN)
- new net: IC2.5 (ST), R7.2
- new net VIN: D1.2 (A2), F1.1, J3.4 (Pin_4)
Other:
- note added: "MCU Decoupling Capacitors"
- note added: "Power Filtering & Protection"
- note added: "Power Header"
- note added: "Sensor Interface Connectors"
- note added: "Vehicle Interface Connector"
- note removed: "*All TVS diodes are DESD5V0U1BA-7 unless otherwise noted"
- note removed: "Decoupling Capacitors"
- note removed: "GPIO Power Header & Cap"
- note removed: "Main connector"
- moved on the sheet: C1, C10, C11, C13, C14, C2, C3, C4, C5, C6, C7, C8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

Commit message: can-module: Update schematic and PCB to fully add in power filtering components
Parts:
- added TP1: TestPoint, TestPoint:TestPoint_Pad_D1.0mm, symbol Connector:TestPoint
- renumbered IC1 to U1, U1 to U2, IC2 to U3
Connections:
- net +5V: now also TP1.1
- net PA04: now also J1.8 (Pin_8); no longer J1.1 (Pin_1)
- net PA05: now also J1.7 (Pin_7); no longer J1.2 (Pin_2)
- net PA06: now also J1.6 (Pin_6); no longer J1.3 (Pin_3)
- net PA07: now also J1.5 (Pin_5); no longer J1.4 (Pin_4)
- net PA08: now also J1.4 (Pin_4); no longer J1.5 (Pin_5)
- net PA09: now also J1.3 (Pin_3); no longer J1.6 (Pin_6)
- net PA10: now also J1.2 (Pin_2); no longer J1.7 (Pin_7)
- net PA11: now also J1.1 (Pin_1); no longer J1.8 (Pin_8)
Changed lines of the file:
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@@
 	)
 	(junction
+		(at 203.2 33.02)
+		(diameter 0)
+		(color 0 0 0 0)
+	)
+	(junction
 		(at 46.99 115.57)
 		(diameter 0)
@@
 	(wire
 		(pts
+			(xy 203.2 30.48) (xy 203.2 33.02)
+		)
+		(stroke
+			(width 0)
+			(type default)
+		)
+	)
+	(wire
+		(pts
 			(xy 46.99 114.3) (xy 46.99 115.57)
 		)
@@
 		(on_board yes)
 		(dnp no)
-		(property "Reference" "IC1"
+		(property "Reference" "U1"
 			(at 157.226 160.528 0)
 			(effects
@@
 			(project ""
 				(path "/40cb4209-4f7f-4a38-b0f0-dee54a92ee91"
-					(reference "IC1")
+					(reference "U1")
 					(unit 1)
 				)
@@
 	)
 	(symbol
+		(lib_id "Connector:TestPoint")
+		(at 203.2 30.48 0)
+		(unit 1)
+		(exclude_from_sim no)
+		(in_bom yes)
+		(on_board yes)
+		(dnp no)
+		(property "Reference" "TP1"
+			(at 204.978 27.686 0)
+			(effects
+				(font
+					(size 1.27 1.27)
+				)
+				(justify left)
+			)
+		)
+		(property "Value" "TestPoint"
+			(at 205.74 28.4479 0)
+			(effects
+				(font
+					(size 1.27 1.27)
+				)
+				(justify left)
+				(hide yes)
+			)
+		)
+		(property "Footprint" "TestPoint:TestPoint_Pad_D1.0mm"
+			(at 208.28 30.48 0)
+			(effects
+				(font
+					(size 1.27 1.27)
+				)
+				(hide yes)
+			)
+		)
+		(property "Datasheet" "~"
+			(at 208.28 30.48 0)
+			(effects
+				(font
+					(size 1.27 1.27)
+				)
+				(hide yes)
+			)
+		)
+		(property "Description" "test point"
+			(at 203.2 30.48 0)
+			(effects
+				(font
+					(size 1.27 1.27)
+				)
+				(hide yes)
+			)
+		)
+		(pin "1"
+		)
+		(instances
+			(project ""
+				(path "/40cb4209-4f7f-4a38-b0f0-dee54a92ee91"
+					(reference "TP1")
+					(unit 1)
+				)
+			)
+		)
+	)
+	(symbol
 		(lib_id "power:+5V")
 		(at 270.51 111.76 0)
@@
 	(symbol
 		(lib_id "Connector:Conn_01x08_Socket")
-		(at 251.46 31.75 0)
+		(at 251.46 34.29 0)
+		(mirror x)
 		(unit 1)
 		(exclude_from_sim no)
@@
 		(dnp no)
 		(property "Reference" "J1"
-			(at 249.428 43.942 0)
+			(at 249.174 43.942 0)
 			(effects
 				(font
@@
 		)
 		(property "Value" "Conn_01x08_Socket"
-			(at 250.825 44.45 0)
+			(at 250.825 21.59 0)
 			(effects
 				(font
@@
 		)
 		(property "Footprint" "Connector_PinHeader_1.27mm:PinHeader_1x08_P1.27mm_Vertical"
-			(at 251.46 31.75 0)
+			(at 251.46 34.29 0)
 			(effects
 				(font
@@
 		)
 		(property "Datasheet" "~"
-			(at 251.46 31.75 0)
+			(at 251.46 34.29 0)
 			(effects
 				(font
@@
 		)
 		(property "Description" "Generic connector, single row, 01x08, script generated"
-			(at 251.46 31.75 0)
+			(at 251.46 34.29 0)
 			(effects
 				(font
@@
 		(dnp no)
 		(fields_autoplaced yes)
-		(property "Reference" "IC2"
+		(property "Reference" "U3"
 			(at 167.64 25.4 0)
 			(effects
@@
 			(project ""
 				(path "/40cb4209-4f7f-4a38-b0f0-dee54a92ee91"
-					(reference "IC2")
+					(reference "U3")
 					(unit 1)
 				)
@@
 		(dnp no)
 		(fields_autoplaced yes)
-		(property "Reference" "U1"
+		(property "Reference" "U2"
 			(at 231.14 101.6 0)
 			(effects
@@
 			(project ""
 				(path "/40cb4209-4f7f-4a38-b0f0-dee54a92ee91"
-					(reference "U1")
+					(reference "U2")
 					(unit 1)
 				)

Commit message: can-module: Add in test points on exposed and unused GPIOs
Parts:
- added TP10, TP11, TP12, TP13, TP14, TP15, TP16, TP2, TP5, TP6, TP7, TP8, TP9: TestPoint, TestPoint:TestPoint_Pad_D1.0mm, symbol Connector:TestPoint
Connections:
- net at U1.1 (PA00_XIN32): now also TP2.1
- net at U1.2 (PA01_XOUT32): now also TP5.1
- net at U1.22 (PA13): now also TP8.1
- net at U1.23 (PA14_XIN): now also TP9.1
- net at U1.24 (PA15_XOUT): now also TP10.1
- net at U1.25 (PA16): now also TP11.1
- net at U1.26 (PA17): now also TP12.1
- net at U1.27 (PA18): now also TP13.1
- net at U1.28 (PA19): now also TP14.1
- net at U1.29 (PA20): now also TP15.1
- net at U1.3 (PA02): now also TP6.1
- net at U1.30 (PA21): now also TP16.1
- net at U1.4 (PA03): now also TP7.1
- no-connect marks 23 -> 10
Other:
- moved on the sheet: D4

Commit message: can-module: Use tight spacing test points on GPIO test points
Parts:
- TP10, TP11, TP12, TP13, TP14, TP15, TP16, TP2, TP5, TP6, TP7, TP8, TP9: footprint TestPoint:TestPoint_Pad_D1.0mm -> TestPoints:TestPoint_Pad_D1.0mm_TightSpacing
Changed lines of the file:
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@@
 			)
 		)
-		(property "Footprint" "TestPoint:TestPoint_Pad_D1.0mm"
+		(property "Footprint" "TestPoints:TestPoint_Pad_D1.0mm_TightSpacing"
 			(at 144.78 171.45 0)
 			(effects
@@
 			)
 		)
-		(property "Footprint" "TestPoint:TestPoint_Pad_D1.0mm"
+		(property "Footprint" "TestPoints:TestPoint_Pad_D1.0mm_TightSpacing"
 			(at 139.7 171.45 0)
 			(effects
@@
 			)
 		)
-		(property "Footprint" "TestPoint:TestPoint_Pad_D1.0mm"
+		(property "Footprint" "TestPoints:TestPoint_Pad_D1.0mm_TightSpacing"
 			(at 162.56 148.59 0)
 			(effects
@@
 			)
 		)
-		(property "Footprint" "TestPoint:TestPoint_Pad_D1.0mm"
+		(property "Footprint" "TestPoints:TestPoint_Pad_D1.0mm_TightSpacing"
 			(at 162.56 140.97 0)
 			(effects
@@
 			)
 		)
-		(property "Footprint" "TestPoint:TestPoint_Pad_D1.0mm"
+		(property "Footprint" "TestPoints:TestPoint_Pad_D1.0mm_TightSpacing"
 			(at 111.76 118.11 0)
 			(effects
@@
 			)
 		)
-		(property "Footprint" "TestPoint:TestPoint_Pad_D1.0mm"
+		(property "Footprint" "TestPoints:TestPoint_Pad_D1.0mm_TightSpacing"
 			(at 162.56 138.43 0)
 			(effects
@@
 			)
 		)
-		(property "Footprint" "TestPoint:TestPoint_Pad_D1.0mm"
+		(property "Footprint" "TestPoints:TestPoint_Pad_D1.0mm_TightSpacing"
 			(at 162.56 151.13 0)
 			(effects
@@
 			)
 		)
-		(property "Footprint" "TestPoint:TestPoint_Pad_D1.0mm"
+		(property "Footprint" "TestPoints:TestPoint_Pad_D1.0mm_TightSpacing"
 			(at 162.56 146.05 0)
 			(effects
@@
 			)
 		)
-		(property "Footprint" "TestPoint:TestPoint_Pad_D1.0mm"
+		(property "Footprint" "TestPoints:TestPoint_Pad_D1.0mm_TightSpacing"
 			(at 111.76 120.65 0)
 			(effects
@@
 			)
 		)
-		(property "Footprint" "TestPoint:TestPoint_Pad_D1.0mm"
+		(property "Footprint" "TestPoints:TestPoint_Pad_D1.0mm_TightSpacing"
 			(at 162.56 143.51 0)
 			(effects
@@
 			)
 		)
-		(property "Footprint" "TestPoint:TestPoint_Pad_D1.0mm"
+		(property "Footprint" "TestPoints:TestPoint_Pad_D1.0mm_TightSpacing"
 			(at 111.76 115.57 0)
 			(effects
@@
 			)
 		)
-		(property "Footprint" "TestPoint:TestPoint_Pad_D1.0mm"
+		(property "Footprint" "TestPoints:TestPoint_Pad_D1.0mm_TightSpacing"
 			(at 142.24 171.45 0)
 			(effects
@@
 			)
 		)
-		(property "Footprint" "TestPoint:TestPoint_Pad_D1.0mm"
+		(property "Footprint" "TestPoints:TestPoint_Pad_D1.0mm_TightSpacing"
 			(at 111.76 113.03 0)
 			(effects

Commit message: can-module: Update to have 13x GPIO test points exposed
Parts:
- TP1, TP3, TP4: footprint TestPoint:TestPoint_Pad_D1.0mm -> TestPoints:TestPoint_Pad_D1.0mm_TightSpacing
Changed lines of the file:
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@@
 			)
 		)
-		(property "Footprint" "TestPoint:TestPoint_Pad_D1.0mm"
+		(property "Footprint" "TestPoints:TestPoint_Pad_D1.0mm_TightSpacing"
 			(at 134.62 76.2 0)
 			(effects
@@
 			)
 		)
-		(property "Footprint" "TestPoint:TestPoint_Pad_D1.0mm"
+		(property "Footprint" "TestPoints:TestPoint_Pad_D1.0mm_TightSpacing"
 			(at 208.28 30.48 0)
 			(effects
@@
 			)
 		)
-		(property "Footprint" "TestPoint:TestPoint_Pad_D1.0mm"
+		(property "Footprint" "TestPoints:TestPoint_Pad_D1.0mm_TightSpacing"
 			(at 137.16 76.2 0)
 			(effects

Commit message: can-module: Fix critical error bridging 5V to VDDCORE
Connections:
- net +5V: no longer C4.1, C9.1, U1.43 (VDDCORE)
- new net VDD_{CORE}: C4.1, C9.1, U1.43 (VDDCORE)
Other:
- moved on the sheet: R2, TP3, TP4
