File: can-module/pcb/can-module.kicad_sch (KiCad schematic)
At the start: 51 parts, among them J1 Conn_01x08_Socket, J2 Conn_01x02_Socket, J3 Conn_01x04_Socket, U1 PIC32CM1216JH01048-I_U5B, U2 ATA6560-GBQW-N, U3 NID5100GWH

Commit message: can-module: Reassign all reference designators by geographical position on schematic
Parts:
- renumbered C15 to C1, C13 to C10, C5 to C11, C6 to C12, C7 to C13, C8 to C14, C9 to C15, C16 to C2, C14 to C3, C10 to C4, C11 to C5, C1 to C6, C2 to C7, C3 to C8, C4 to C9, D3 to D2, D2 to D3, D5 to D4, D4 to D5, J3 to J1, J1 to J2, J2 to J3, JP2 to JP1, R7 to R1, R6 to R2, R2 to R3, R1 to R4, R3 to R5, R4 to R6, R5 to R7, TP14 to TP10, TP13 to TP11, TP11 to TP13, TP8 to TP14, TP9 to TP15, TP10 to TP16, TP3 to TP2, TP4 to TP3, TP2 to TP4, TP16 to TP8, TP15 to TP9, U3 to U1, U1 to U3

Commit message: can-module: Update CAN module to have selectable GPIO voltage (3.3V or 5V)
Parts:
- removed C10: 4n7, Capacitor_SMD:C_0402_1005Metric, symbol Device:C_Small
- removed JP1: Jumper_2_Small_Open, Jumper:SolderJumper-2_P1.3mm_Open_Pad1.0x1.5mm, symbol Jumper:Jumper_2_Small_Open
- removed R5, R6: 60, Resistor_SMD:R_0402_1005Metric, symbol Device:R
- added C4, C5: 10u, Capacitor_SMD:C_0402_1005Metric, symbol Device:C_Small
- added R5, R6: 0, Resistor_SMD:R_0402_1005Metric, symbol Device:R_Small
- added U2: MIC5365-3.3YC5, Package_TO_SOT_SMD:SOT-353_SC-70-5, symbol Regulator_Linear:MIC5365-3.3YC5
- renumbered C8 to C10, C9 to C11, C11 to C12, C12 to C13, C13 to C14, C14 to C15, C15 to C16, C4 to C6, C5 to C7, C6 to C8, C7 to C9, D2 to D1, D3 to D2, D1 to D3, U2 to U3, U3 to U4
Connections:
- net +5V: now also C4.1, R5.2, U2.1 (VIN), U2.3 (EN); no longer C10.1, C14.1, C15.1, J3.2 (Pin_2), U4.17 (VDDIO_1), U4.36 (VDDIO_2)
- net GND: now also C4.2, C5.2, U2.2 (GND)
- new net +3V3: C5.1, R6.1, U2.5 (VOUT)
- new net VDD_{IO}: C10.1, C14.1, C15.1, J3.2 (Pin_2), R5.1, R6.2, U4.17 (VDDIO_1), U4.36 (VDDIO_2)
Other:
- note added: "GPIO Voltage Regulator & Selector"
- note added: "GPIO voltage is 5V by default, but can be changed to 3.3V"
- note removed: "CAN Termination"
- moved on the sheet: C1, C10, C11, C12, C13, C14, C15, C16, C2, C3, C7, C8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

Commit message: can-module: Change programming header to be through hole for easier access
Parts:
- removed TP2, TP3: TestPoint, TestPoints:TestPoint_Pad_D1.0mm_TightSpacing, symbol Connector:TestPoint
- added J4: Conn_01x02_Socket, Connector_PinHeader_1.27mm:PinHeader_1x02_P1.27mm_Vertical, symbol Connector:Conn_01x02_Socket
Connections:
- net SWCLK: now reaches R3.1, U4.45 (PA30_SWCLK)
- net SWCLK: now also J4.1 (Pin_1)
- net SWDIO: now reaches U4.46 (PA31_SWDIO)
- net SWDIO: now also J4.2 (Pin_2)
Other:
- note added: "Programming/Debug Header"
- moved on the sheet: C6, C7, R3, R4, U3

Commit message: can-module: Flip indicator LED around so that anode is always 5V
Connections:
- net +5V: now also D5.2 (A)
- net GND: no longer D5.1 (K)
- net at R7.2: now also D5.1 (K); no longer D5.2 (A)
Other:
- moved on the sheet: D5
Changed lines of the file:
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@@
 	(wire
 		(pts
-			(xy 142.24 176.53) (xy 142.24 179.07)
+			(xy 142.24 176.53) (xy 142.24 181.61)
 		)
 		(stroke
@@
 	(wire
 		(pts
+			(xy 144.78 189.23) (xy 142.24 189.23)
+		)
+		(stroke
+			(width 0)
+			(type default)
+		)
+	)
+	(wire
+		(pts
 			(xy 252.73 99.06) (xy 255.27 99.06)
 		)
@@
 	(wire
 		(pts
-			(xy 142.24 184.15) (xy 142.24 186.69)
+			(xy 132.08 36.83) (xy 134.62 36.83)
 		)
 		(stroke
@@
 	(wire
 		(pts
-			(xy 132.08 36.83) (xy 134.62 36.83)
+			(xy 46.99 130.81) (xy 46.99 132.08)
 		)
 		(stroke
@@
 	(wire
 		(pts
-			(xy 46.99 130.81) (xy 46.99 132.08)
+			(xy 46.99 25.4) (xy 58.42 25.4)
 		)
 		(stroke
@@
 	(wire
 		(pts
-			(xy 46.99 25.4) (xy 58.42 25.4)
+			(xy 142.24 189.23) (xy 142.24 186.69)
 		)
 		(stroke
@@
 	(symbol
 		(lib_id "Device:LED_Small")
-		(at 142.24 181.61 90)
+		(at 142.24 184.15 90)
+		(mirror x)
 		(unit 1)
 		(exclude_from_sim no)
@@
 		(dnp no)
 		(property "Reference" "D5"
-			(at 139.7 180.2764 90)
+			(at 139.7 185.4836 90)
 			(effects
 				(font
@@
 		)
 		(property "Value" "LTST-C170GKT"
-			(at 139.7 182.8164 90)
+			(at 139.7 182.9436 90)
 			(effects
 				(font
@@
 		)
 		(property "Footprint" "LED_SMD:LED_0805_2012Metric"
-			(at 142.24 181.61 90)
+			(at 142.24 184.15 90)
 			(effects
 				(font
@@
 		)
 		(property "Datasheet" "~"
-			(at 142.24 181.61 90)
+			(at 142.24 184.15 90)
 			(effects
 				(font
@@
 		)
 		(property "Description" "Light emitting diode, small symbol"
-			(at 142.24 181.61 0)
+			(at 142.24 184.15 0)
 			(effects
 				(font
@@
 		)
 		(property "Sim.Pin" "1=K 2=A"
-			(at 142.24 181.61 0)
+			(at 142.24 184.15 0)
 			(effects
 				(font
@@
 		)
 		(instances
-			(project ""
+			(project "can-module"
 				(path "/40cb4209-4f7f-4a38-b0f0-dee54a92ee91"
 					(reference "D5")
@@
 	)
 	(symbol
-		(lib_id "power:GND")
-		(at 142.24 186.69 0)
-		(mirror y)
-		(unit 1)
-		(exclude_from_sim no)
-		(in_bom yes)
-		(on_board yes)
-		(dnp no)
-		(property "Reference" "#PWR046"
-			(at 142.24 193.04 0)
-			(effects
-				(font
-					(size 1.27 1.27)
-				)
-				(hide yes)
-			)
-		)
-		(property "Value" "GND"
-			(at 142.24 191.262 0)
-			(effects
-				(font
-					(size 1.27 1.27)
-				)
-			)
-		)
-		(property "Footprint" ""
-			(at 142.24 186.69 0)
-			(effects
-				(font
-					(size 1.27 1.27)
-				)
-				(hide yes)
-			)
-		)
-		(property "Datasheet" ""
-			(at 142.24 186.69 0)
-			(effects
-				(font
-					(size 1.27 1.27)
-				)
-				(hide yes)
-			)
-		)
-		(property "Description" "Power symbol creates a global label with name \"GND\" , ground"
-			(at 142.24 186.69 0)
-			(effects
-				(font
-					(size 1.27 1.27)
-				)
-				(hide yes)
-			)
-		)
-		(pin "1"
-		)
-		(instances
-			(project "can-module"
-				(path "/40cb4209-4f7f-4a38-b0f0-dee54a92ee91"
-					(reference "#PWR046")
-					(unit 1)
-				)
-			)
-		)
-	)
-	(symbol
 		(lib_id "Device:C")
 		(at 58.42 135.89 0)
@@
 					(unit 1)
 				)
+			)
+		)
+	)
+	(symbol
+		(lib_id "power:+5V")
+		(at 144.78 189.23 270)
+		(unit 1)
+		(exclude_from_sim no)
+		(in_bom yes)
+		(on_board yes)
+		(dnp no)
+		(fields_autoplaced yes)
+		(property "Reference" "#PWR013"
+			(at 140.97 189.23 0)
+			(effects
+				(font
+					(size 1.27 1.27)
+				)
+				(hide yes)
+			)
+		)
+		(property "Value" "+5V"
+			(at 148.59 189.2299 90)
+			(effects
+				(font
+					(size 1.27 1.27)
+				)
+				(justify left)
+			)
+		)
+		(property "Footprint" ""
+			(at 144.78 189.23 0)
+			(effects
+				(font
+					(size 1.27 1.27)
+				)
+				(hide yes)
+			)
+		)
+		(property "Datasheet" ""
+			(at 144.78 189.23 0)
+			(effects
+				(font
+					(size 1.27 1.27)
+				)
+				(hide yes)
+			)
+		)
+		(property "Description" "Power symbol creates a global label with name \"+5V\""
+			(at 144.78 189.23 0)
+			(effects
+				(font
+					(size 1.27 1.27)
+				)
+				(hide yes)
+			)
+		)
+		(pin "1"
+		)
+		(instances
+			(project "can-module"
+				(path "/40cb4209-4f7f-4a38-b0f0-dee54a92ee91"
+					(reference "#PWR013")
+					(unit 1)
+				)
