File: sd-card-board/sd-card-board.kicad_pcb (KiCad board)
At the start: 2 copper layers, 22.9 x 19.1 mm, 9 parts, among them J1 Conn_01x08, J2 Conn_01x02, J3 1051620001, U1 MIC5365-3.3YC5-TR, U2 FXMAR2104UMX

Commit message: sd-card-board: Route out PCB, add microSD card model
Connections:
- U2 pad 10: /SD_CLK -> /SD_DI
- U2 pad 11: /SD_DI -> /SD_CLK
- U2 pad 12: /~{SD_CS} -> /SD_DO
- U2 pad 3: /~{MCU_CS} -> /MCU_DO
- U2 pad 4: /MCU_DI -> /MCU_CLK
- U2 pad 5: /MCU_CLK -> /MCU_DI
- U2 pad 6: /MCU_DO -> /~{MCU_CS}
- U2 pad 9: /SD_DO -> /~{SD_CS}
Routing:
- net GND: track 0.00 -> 12.0 mm, vias 0 -> 11
- net /SD_DO: track 0.00 -> 11.0 mm
- net /~{MCU_CS}: track 0.00 -> 10.4 mm
- net /SD_CLK: track 0.00 -> 9.36 mm
- net /MCU_DI: track 0.00 -> 8.86 mm
- net /SD_DI: track 0.00 -> 7.41 mm
- net /MCU_CLK: track 0.00 -> 7.22 mm
- net /~{SD_CS}: track 0.00 -> 6.85 mm
- net /MCU_DO: track 0.00 -> 5.34 mm
- net +5V: track 0.00 -> 1.82 mm
- added copper zone on F.Cu, net +3V3
- added copper zone on F.Cu, net +5V
- added copper zone on B.Cu, net GND
Other:
- board text added: "ROWAN MOTORSPORTS"

Commit message: sd-card-board: Fix connector spacing
Parts:
- moved J2 0.38 mm to (112.0, 73.2)
- moved REF** 0.29 mm to (120.6, 87.1)
- moved REF** 0.29 mm to (120.6, 75.6)
Changed lines of the file:
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@@
 	(footprint "MountingHole:MountingHole_2.2mm_M2"
 		(layer "F.Cu")
-		(at 120.9 87.105)
+		(at 120.61 87.105)
 		(descr "Mounting Hole 2.2mm, M2, no annular, generated by kicad-footprint-generator mountinghole.py")
 		(tags "mountinghole M2")
@@
 	(footprint "MountingHole:MountingHole_2.2mm_M2"
 		(layer "F.Cu")
-		(at 120.9 75.555)
+		(at 120.61 75.555)
 		(descr "Mounting Hole 2.2mm, M2, no annular, generated by kicad-footprint-generator mountinghole.py")
 		(tags "mountinghole M2")
@@
 			)
 		)
+		(model "${KIPRJMOD}/lib/1051620001/Micro SD Card.STEP"
+			(hide yes)
+			(offset
+				(xyz -24 -21 0)
+			)
+			(scale
+				(xyz 1 1 1)
+			)
+			(rotate
+				(xyz -0 -0 -0)
+			)
+		)
 	)
 	(footprint "Connector_PinSocket_1.00mm:PinSocket_1x02_P1.00mm_Vertical"
 		(layer "B.Cu")
-		(at 112.25 73 90)
+		(at 111.96 73.25 90)
 		(descr "Through hole straight socket strip, 1x02, 1.00mm pitch, single row (https://gct.co/files/drawings/bc065.pdf), script generated")
 		(tags "Through hole socket strip THT 1x02 1.00mm single row")
@@
 		(layer "F.Fab")
 		(pts
-			(xy 105.75 77.75) (xy 110.25 73)
+			(xy 105.75 77.75) (xy 111.25 73.25)
 		)
 		(height -2.25)
@@
 			(keep_text_aligned yes)
 		)
-		(gr_text "4.75"
-			(at 102.35 75.375 90)
+		(gr_text "4.5"
+			(at 102.35 75.5 90)
 			(layer "F.Fab")
 			(effects
@@
 		(layer "F.Fab")
 		(pts
-			(xy 105.75 77.75) (xy 111.25 73)
+			(xy 105.46 76.5) (xy 111.96 73.25)
 		)
 		(height -9.5)
@@
 			(keep_text_aligned yes)
 		)
-		(gr_text "5.5"
-			(at 108.5 67.1 0)
+		(gr_text "6.5"
+			(at 108.71 65.85 0)
 			(layer "F.Fab")
 			(effects
@@
 		(layer "F.Fab")
 		(pts
-			(xy 111.25 73) (xy 120.9 75.555)
+			(xy 111.96 73.25) (xy 120.61 75.555)
 		)
 		(height -4.25)
@@
 			(keep_text_aligned yes)
 		)
-		(gr_text "9.65"
-			(at 116.075 67.6 0)
+		(gr_text "8.65"
+			(at 116.285 67.85 0)
 			(layer "F.Fab")
 			(effects

Commit message: sd-card-board: Fully fix positioning issues
Parts:
- moved J2 0.29 mm to (112.0, 73.0)
- moved REF** 0.08 mm to (120.6, 75.5)
- moved REF** 0.08 mm to (120.6, 87.0)
Changed lines of the file:
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@@
 	(footprint "MountingHole:MountingHole_2.2mm_M2"
 		(layer "F.Cu")
-		(at 120.61 87.105)
+		(at 120.61 87.025)
 		(descr "Mounting Hole 2.2mm, M2, no annular, generated by kicad-footprint-generator mountinghole.py")
 		(tags "mountinghole M2")
@@
 	(footprint "MountingHole:MountingHole_2.2mm_M2"
 		(layer "F.Cu")
-		(at 120.61 75.555)
+		(at 120.61 75.475)
 		(descr "Mounting Hole 2.2mm, M2, no annular, generated by kicad-footprint-generator mountinghole.py")
 		(tags "mountinghole M2")
@@
 	(footprint "Connector_PinSocket_1.00mm:PinSocket_1x02_P1.00mm_Vertical"
 		(layer "B.Cu")
-		(at 111.96 73.25 90)
+		(at 111.96 72.96 90)
 		(descr "Through hole straight socket strip, 1x02, 1.00mm pitch, single row (https://gct.co/files/drawings/bc065.pdf), script generated")
 		(tags "Through hole socket strip THT 1x02 1.00mm single row")
@@
 		(layer "F.Fab")
 		(pts
-			(xy 105.75 77.75) (xy 111.25 73.25)
+			(xy 105.75 77.75) (xy 109.71 73.25)
 		)
 		(height -2.25)
@@
 			(thickness 0.1)
 			(arrow_length 1.27)
-			(text_position_mode 0)
+			(text_position_mode 2)
 			(arrow_direction outward)
 			(extension_height 0.58642)
@@
 		)
 		(gr_text "4.5"
-			(at 102.35 75.5 90)
+			(at 100.5 75.249998 90)
 			(layer "F.Fab")
 			(effects
@@
 		(layer "F.Fab")
 		(pts
-			(xy 120.9 75.555) (xy 120.9 87.105)
+			(xy 120.61 75.475) (xy 120.61 87.025)
 		)
 		(height -20.9)
@@
 		)
 		(gr_text "11.55"
-			(at 98.85 81.33 90)
+			(at 98.56 81.25 90)
 			(layer "F.Fab")
 			(effects
@@
 			(layer "F.Fab")
 			(effects
+				(font
+					(size 1 1)
+					(thickness 0.15)
+				)
+			)
+		)
+	)
+	(dimension
+		(type orthogonal)
+		(layer "F.Fab")
+		(pts
+			(xy 113.21 73.25) (xy 120.61 75.475)
+		)
+		(height -17.46)
+		(orientation 1)
+		(format
+			(prefix "")
+			(suffix "")
+			(units 3)
+			(units_format 0)
+			(precision 4)
+			(suppress_zeroes yes)
+		)
+		(style
+			(thickness 0.1)
+			(arrow_length 1.27)
+			(text_position_mode 0)
+			(arrow_direction outward)
+			(extension_height 0.58642)
+			(extension_offset 0.5)
+			(keep_text_aligned yes)
+		)
+		(gr_text "2.225"
+			(at 94.6 74.3625 90)
+			(layer "F.Fab")
+			(effects

Commit message: sd-card-board: Switch from 1mm to 1.27mm spacing for pin headers
Parts:
- J1: footprint Connector_PinSocket_1.00mm:PinSocket_1x08_P1.00mm_Vertical -> Connector_PinSocket_1.27mm:PinSocket_1x08_P1.27mm_Vertical
- J2: footprint Connector_PinSocket_1.00mm:PinSocket_1x02_P1.00mm_Vertical -> Connector_PinSocket_1.27mm:PinSocket_1x02_P1.27mm_Vertical
- moved J1 1.06 mm to (105.3, 85.7)
- moved J2 0.48 mm to (112.4, 73.2)
Routing:
- net /~{MCU_CS}: track 10.4 -> 11.9 mm, vias 0 -> 1
