File: sd-card-board/sd-card-board.kicad_sch (KiCad schematic)
At the start: 0 parts

Commit message: sd-card-board: Set up schematic
Parts:
- added C1, C2: 1u, Capacitor_SMD:C_0402_1005Metric, symbol Device:C_Small
- added J1: Conn_01x08, Connector_PinSocket_1.00mm:PinSocket_1x08_P1.00mm_Vertical, symbol Connector_Generic:Conn_01x08
- added J2: Conn_01x02, Connector_PinSocket_1.00mm:PinSocket_1x02_P1.00mm_Vertical, symbol Connector_Generic:Conn_01x02
- added J3: MEM2067-02-180-00-A, MEM2067-02-180-00-A:GCT_MEM2067-02-180-00-A_REVB, symbol Connector:Micro_SD_Card
- added U1: MIC5365-3.3YC5-TR, Package_TO_SOT_SMD:SOT-353_SC-70-5, symbol Regulator_Linear:MIC5365-3.3YC5
- added U2: CD4504BM96, Package_SO:SOIC-16_3.9x9.9mm_P1.27mm, symbol 4xxx:4504
Connections:
- new net +3V3: C2.1, J3.4 (VDD), U1.5 (VOUT), U2.16 (VDD)
- new net +5V: C1.1, J2.2 (Pin_2), U1.1 (VIN), U1.3 (EN), U2.1 (VCC), U2.13 (Select)
- new net GND: C1.2, C2.2, J2.1 (Pin_1), J3.6 (VSS), J3.9 (SHIELD), U1.2 (GND), U2.8 (VSS)
- new net MCU_CLK: J1.4 (Pin_4), U2.7 (Cin)
- new net MCU_DI: J1.5 (Pin_5), U2.5 (Bin)
- new net MCU_DO: J1.3 (Pin_3), U2.9 (Din)
- new net SD_CLK: J3.5 (CLK), U2.6 (Cout)
- new net SD_DI: J3.3 (CMD), U2.4 (Bout)
- new net SD_DO: J3.7 (DAT0), U2.10 (Dout)
- new net ~{MCU_CS}: J1.6 (Pin_6), U2.3 (Ain)
- new net ~{SD_CS}: J3.2 (DAT3/CD), U2.2 (Aout)
- no-connect marks 0 -> 10
Other:
- note added: "5V <=> 3.3V Level Shifter"
- note added: "5V to 3.3V Conversion"
- note added: "Card is used in SPI Mode"
- note added: "GPIO"
- note added: "MicroSD Card Slot"
- note added: "Power Input"

Commit message: sd-card-board: Swap components, get general placement of components on PCB done
Parts:
- removed U2: CD4504BM96, Package_SO:SOIC-16_3.9x9.9mm_P1.27mm, symbol 4xxx:4504
- added U2: FXMAR2104UMX, ULTRATHIN_MLP_12L_ONS, symbol FXMAR2104UMX:FXMAR2104UMX
- J3: value MEM2067-02-180-00-A -> 1051620001; footprint MEM2067-02-180-00-A:GCT_MEM2067-02-180-00-A_REVB -> 1051620001:105162-0001_MOL
Connections:
- net +3V3: now also U2.1 (VCCB)
- net +5V: now also U2.2 (VCCA), U2.8 (OE)
- net GND: now also U2.7 (GND)
- net MCU_CLK: now also U2.5 (A2)
- net MCU_DI: now also U2.4 (A1)
- net MCU_DO: now also U2.6 (A3)
- net SD_CLK: now also U2.10 (B2)
- net SD_DI: now also U2.11 (B1)
- net SD_DO: now also U2.9 (B3)
- net ~{MCU_CS}: now also U2.3 (A0)
- net ~{SD_CS}: now also U2.12 (B0)
- no-connect marks 10 -> 6

Commit message: sd-card-board: Route out PCB, add microSD card model
Parts:
- U2: footprint ULTRATHIN_MLP_12L_ONS -> FXMAR2104UMX:ULTRATHIN_MLP_12L_ONS
Connections:
- net MCU_CLK: now also U2.4 (A1); no longer U2.5 (A2)
- net MCU_DI: now also U2.5 (A2); no longer U2.4 (A1)
- net MCU_DO: now also U2.3 (A0); no longer U2.6 (A3)
- net SD_CLK: now also U2.11 (B1); no longer U2.10 (B2)
- net SD_DI: now also U2.10 (B2); no longer U2.11 (B1)
- net SD_DO: now also U2.12 (B0); no longer U2.9 (B3)
- net ~{MCU_CS}: now also U2.6 (A3); no longer U2.3 (A0)
- net ~{SD_CS}: now also U2.9 (B3); no longer U2.12 (B0)
Changed lines of the file:
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@@
 		)
 	)
-	(label "SD_DO"
-		(at 171.45 115.57 180)
+	(label "MCU_DI"
+		(at 85.09 114.3 180)
 		(effects
 			(font
@@
 	)
 	(label "MCU_CLK"
+		(at 113.03 115.57 0)
+		(effects
+			(font
+				(size 1.27 1.27)
+				(thickness 0.1588)
+			)
+			(justify left bottom)
+		)
+	)
+	(label "MCU_DI"
 		(at 113.03 118.11 0)
 		(effects
@@
 			)
 			(justify left bottom)
-		)
-	)
-	(label "~{MCU_CS}"
-		(at 113.03 113.03 0)
-		(effects
-			(font
-				(size 1.27 1.27)
-				(thickness 0.1588)
-			)
-			(justify left bottom)
-		)
-	)
-	(label "SD_DI"
-		(at 171.45 110.49 180)
-		(effects
-			(font
-				(size 1.27 1.27)
-				(thickness 0.1588)
-			)
-			(justify right bottom)
 		)
 	)
@@
 		)
 	)
+	(label "SD_DO"
+		(at 171.45 107.95 180)
+		(effects
+			(font
+				(size 1.27 1.27)
+				(thickness 0.1588)
+			)
+			(justify right bottom)
+		)
+	)
 	(label "SD_CLK"
 		(at 194.31 118.11 0)
@@
 		)
 	)
+	(label "~{MCU_CS}"
+		(at 113.03 120.65 0)
+		(effects
+			(font
+				(size 1.27 1.27)
+				(thickness 0.1588)
+			)
+			(justify left bottom)
+		)
+	)
+	(label "MCU_DO"
+		(at 113.03 113.03 0)
+		(effects
+			(font
+				(size 1.27 1.27)
+				(thickness 0.1588)
+			)
+			(justify left bottom)
+		)
+	)
 	(label "~{SD_CS}"
-		(at 171.45 107.95 180)
-		(effects
-			(font
-				(size 1.27 1.27)
-				(thickness 0.1588)
-			)
-			(justify right bottom)
-		)
-	)
-	(label "SD_CLK"
-		(at 171.45 113.03 180)
-		(effects
-			(font
-				(size 1.27 1.27)
-				(thickness 0.1588)
-			)
-			(justify right bottom)
-		)
-	)
-	(label "MCU_DI"
-		(at 113.03 115.57 0)
-		(effects
-			(font
-				(size 1.27 1.27)
-				(thickness 0.1588)
-			)
-			(justify left bottom)
+		(at 194.31 110.49 0)
+		(effects
+			(font
+				(size 1.27 1.27)
+				(thickness 0.1588)
+			)
+			(justify left bottom)
+		)
+	)
+	(label "~{SD_CS}"
+		(at 171.45 115.57 180)
+		(effects
+			(font
+				(size 1.27 1.27)
+				(thickness 0.1588)
+			)
+			(justify right bottom)
 		)
 	)
@@
 		)
 	)
-	(label "~{SD_CS}"
-		(at 194.31 110.49 0)
-		(effects
-			(font
-				(size 1.27 1.27)
-				(thickness 0.1588)
-			)
-			(justify left bottom)
+	(label "SD_CLK"
+		(at 171.45 110.49 180)
+		(effects
+			(font
+				(size 1.27 1.27)
+				(thickness 0.1588)
+			)
+			(justify right bottom)
+		)
+	)
+	(label "SD_DI"
+		(at 194.31 113.03 0)
+		(effects
+			(font
+				(size 1.27 1.27)
+				(thickness 0.1588)
+			)
+			(justify left bottom)
+		)
+	)
+	(label "MCU_CLK"
+		(at 85.09 116.84 180)
+		(effects
+			(font
+				(size 1.27 1.27)
+				(thickness 0.1588)
+			)
+			(justify right bottom)
 		)
 	)
@@
 		)
 	)
-	(label "MCU_CLK"
-		(at 85.09 116.84 180)
-		(effects
-			(font
-				(size 1.27 1.27)
-				(thickness 0.1588)
-			)
-			(justify right bottom)
-		)
-	)
-	(label "MCU_DO"
-		(at 113.03 120.65 0)
-		(effects
-			(font
-				(size 1.27 1.27)
-				(thickness 0.1588)
-			)
-			(justify left bottom)
-		)
-	)
 	(label "SD_DI"
-		(at 194.31 113.03 0)
-		(effects
-			(font
-				(size 1.27 1.27)
-				(thickness 0.1588)
-			)
-			(justify left bottom)
-		)
-	)
-	(label "MCU_DI"
-		(at 85.09 114.3 180)
+		(at 171.45 113.03 180)
 		(effects
 			(font
@@
 			)
 		)
-		(property "Footprint" "ULTRATHIN_MLP_12L_ONS"
+		(property "Footprint" "FXMAR2104UMX:ULTRATHIN_MLP_12L_ONS"
 			(at 121.92 107.95 0)
 			(effects

Commit message: sd-card-board: Switch from 1mm to 1.27mm spacing for pin headers
Parts:
- J1: footprint Connector_PinSocket_1.00mm:PinSocket_1x08_P1.00mm_Vertical -> Connector_PinSocket_1.27mm:PinSocket_1x08_P1.27mm_Vertical
- J2: footprint Connector_PinSocket_1.00mm:PinSocket_1x02_P1.00mm_Vertical -> Connector_PinSocket_1.27mm:PinSocket_1x02_P1.27mm_Vertical
Changed lines of the file:
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@@
 			)
 		)
-		(property "Footprint" "Connector_PinSocket_1.00mm:PinSocket_1x02_P1.00mm_Vertical"
+		(property "Footprint" "Connector_PinSocket_1.27mm:PinSocket_1x02_P1.27mm_Vertical"
 			(at 99.06 67.31 0)
 			(effects
@@
 			)
 		)
-		(property "Footprint" "Connector_PinSocket_1.00mm:PinSocket_1x08_P1.00mm_Vertical"
+		(property "Footprint" "Connector_PinSocket_1.27mm:PinSocket_1x08_P1.27mm_Vertical"
 			(at 71.12 116.84 0)
 			(effects
