File: accelerometer-board/accelerometer-board.kicad_sch (KiCad schematic)
At the start: 20 parts, among them J1 Conn_01x08, J2 Conn_01x02, U1 LIS2HH12, U2 LIS2HH12, U3 FXMA2102L8X, U4 MCP1700T-2502E/TT

Commit message: accelerometer-board: Update to contain a single IMU chip
Parts:
- removed C3, C5, C6: 100n, Capacitor_SMD:C_0402_1005Metric, symbol Device:C_Small
- removed C4: 10u, Capacitor_SMD:C_0402_1005Metric, symbol Device:C_Small
- removed U1, U2: LIS2HH12, Package_LGA:LGA-12_2x2mm_P0.5mm, symbol Sensor_Motion:LIS2HH12
- removed U4: MCP1700T-2502E/TT, Package_TO_SOT_SMD:SOT-23, symbol Regulator_Linear:MCP1700x-250xxTT
- added U1: BMI323, BMI323_BOS, symbol BMI323:BMI323
- added U6: MIC5365-3.3YC5-TR, Package_TO_SOT_SMD:SOT-353_SC-70-5, symbol Regulator_Linear:MIC5365-3.3YC5
- C1: value 10u -> 100n
Connections:
- net +5V: now also U6.1 (VIN), U6.3 (EN)
- net GND: now also U1.1 (SDO), U1.6 (GNDIO), U1.7 (GND), U6.2 (GND)
- net SCL_5V: now also J1.6 (Pin_6), R3.2, U3.2 (A0); no longer J1.5 (Pin_5), R4.2, U3.3 (A1)
- net SDA_5V: now also J1.5 (Pin_5), R4.2, U3.3 (A1); no longer J1.6 (Pin_6), R3.2, U3.2 (A0)
- net +2V5 renamed +3V3
- net +3V3: now also U1.12 (CSB), U1.5 (VDDIO), U1.8 (VDD), U6.5 (VOUT)
- net SCL_2V5 renamed SDA_3V3
- net SDA_3V3: now also U1.14 (SDX)
- net SDA_2V5 renamed SCL_3V3
- net SCL_3V3: now also U1.13 (SCX)
- no-connect marks 10 -> 8
Other:
- note added: "5V -> 3.3V Regulator"
- note added: "5V <=> 3.3V Level Shifter"
- note added: "Inertial Measurement Unit (IMU)"
- note removed: "5V -> 2.5V Regulator"
- note removed: "5V <=> 2.5V Level Shifter"
- note removed: "Accelerometers"
- note removed: "I2C Addr: rd 0x3B, wr 0x3A"
- note removed: "I2C Addr: rd 0x3D, wr 0x3C"
- moved on the sheet: C10, C7, C8, C9, J1, J2, R1, R2, R3, R4, U3

Commit message: accelerometer-board: Expose x2 interrupt lines from IMU
Parts:
- removed R1, R2, R3, R4: 4k7, Resistor_SMD:R_0402_1005Metric, symbol Device:R_Small
- removed U3: FXMA2102L8X, FXMA2102L8X:MICROPAK8_1P6X1P6_ONS, symbol FXMA2102L8X:FXMA2102L8X
- added R5, R6, R7, R8: 4k7, Resistor_SMD:R_0402_1005Metric, symbol Device:R_Small
- added U2: FXMAR2104UMX, ULTRATHIN_MLP_12L_ONS, symbol FXMA2104L8X:FXMAR2104UMX
Connections:
- net +3V3: now also R7.1, R8.1, U2.1 (VCCB)
- net +5V: now also R5.1, R6.1, U2.2 (VCCA), U2.8 (OE)
- net GND: now also U2.7 (GND)
- net SCL_3V3: now also R7.2, U2.12 (B0)
- net SCL_5V: now also R6.2, U2.3 (A0)
- net SDA_3V3: now also R8.2, U2.11 (B1)
- net SDA_5V: now also R5.2, U2.4 (A1)
- net IMU_INT2_5V: now reaches J1.3 (Pin_3)
- net IMU_INT2_5V: now also U2.6 (A3)
- net IMU_INT1_5V: now reaches J1.4 (Pin_4)
- net IMU_INT1_5V: now also U2.5 (A2)
- net IMU_INT1_3V3: now reaches U1.4 (INT1)
- net IMU_INT1_3V3: now also U2.10 (B2)
- net IMU_INT2_3V3: now reaches U1.9 (INT2)
- net IMU_INT2_3V3: now also U2.9 (B3)
- no-connect marks 8 -> 4
Other:
- moved on the sheet: C7, C8

Commit message: accelerometer-board: Update footprints
Parts:
- J1: footprint Connector_PinSocket_1.00mm:PinSocket_1x08_P1.00mm_Vertical -> Connector_PinSocket_1.27mm:PinSocket_1x08_P1.27mm_Vertical
- J2: footprint Connector_PinSocket_1.00mm:PinSocket_1x02_P1.00mm_Vertical -> Connector_PinSocket_1.27mm:PinSocket_1x02_P1.27mm_Vertical
- U1: footprint BMI323_BOS -> BMI323:BMI323_BOS
- U2: footprint ULTRATHIN_MLP_12L_ONS -> FXMA2104L8X:ULTRATHIN_MLP_12L_ONS
Changed lines of the file:
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@@
 			)
 		)
-		(property "Footprint" "Connector_PinSocket_1.00mm:PinSocket_1x02_P1.00mm_Vertical"
+		(property "Footprint" "Connector_PinSocket_1.27mm:PinSocket_1x02_P1.27mm_Vertical"
 			(at 52.07 86.36 0)
 			(effects
@@
 			)
 		)
-		(property "Footprint" "Connector_PinSocket_1.00mm:PinSocket_1x08_P1.00mm_Vertical"
+		(property "Footprint" "Connector_PinSocket_1.27mm:PinSocket_1x08_P1.27mm_Vertical"
 			(at 55.88 119.38 0)
 			(effects
@@
 			)
 		)
-		(property "Footprint" "BMI323_BOS"
+		(property "Footprint" "BMI323:BMI323_BOS"
 			(at 213.36 90.17 0)
 			(effects
@@
 			)
 		)
-		(property "Footprint" "ULTRATHIN_MLP_12L_ONS"
+		(property "Footprint" "FXMA2104L8X:ULTRATHIN_MLP_12L_ONS"
 			(at 120.65 119.38 0)
 			(effects
