File: comm-unit/comm-unit.kicad_pcb (KiCad board)
At the start: 2 copper layers, 25.4 x 19.1 mm, 12 parts, among them J1 Conn_01x02, J2 Conn_01x08, U1 TXS0108ERGYR, U2 MIC5365-3.3YC5-TR, U3 Wio-SX1262

Commit message: comm-module: Rearrange components and redo traces
Parts:
- removed the REF** at (161.9, 121.0)
- moved C3 20.2 mm to (148.8, 119.0), turned to -90 degrees
- moved U3 19.4 mm to (166.8, 123.8), turned to 90 degrees
- moved U1 14.5 mm to (150.5, 115.2), turned to 180 degrees
- moved C5 13.5 mm to (168.5, 114.1)
- moved C4 10.6 mm to (152.2, 119.0), turned to -90 degrees
- moved C1 0.51 mm to (168.2, 108.3)
- moved C2 0.51 mm to (166.3, 110.5)
- moved U2 0.51 mm to (166.2, 108.3)
Connections:
- J2 pad 1: unconnected-(J2-Pin_1-Pad1) -> /MCU_DIO1
- J2 pad 2: /MCU_RST -> /MCU_BUSY
- J2 pad 3: /MCU_SCK -> /MCU_RFSW
- J2 pad 4: /MCU_MISO -> /MCU_MOSI
- J2 pad 5: /MCU_MOSI -> /MCU_MISO
- J2 pad 6: /MCU_RFSW -> /MCU_SCK
- J2 pad 7: /MCU_DIO1 -> /MCU_RST
- J2 pad 8: /MCU_BUSY -> unconnected-(J2-Pin_8-Pad8)
- U1 pad 17: /MCU_DIO1 -> /MCU_BUSY
- U1 pad 18: /MCU_BUSY -> /MCU_DIO1
- U1 pad 3: /MOD_BUSY -> /MOD_DIO1
- U1 pad 4: /MOD_DIO1 -> /MOD_BUSY
Routing:
- net /MCU_BUSY: track 26.9 -> 3.30 mm, vias 1 -> 0
- net /MCU_MOSI: track 25.7 -> 2.16 mm, vias 1 -> 0
- net /MCU_MISO: track 25.3 -> 1.95 mm, vias 1 -> 0
- net /MCU_RFSW: track 26.1 -> 2.81 mm, vias 1 -> 0
- net /MCU_SCK: track 24.9 -> 1.95 mm, vias 1 -> 0
- net /MCU_DIO1: track 26.6 -> 3.81 mm, vias 1 -> 0
- net /MCU_RST: track 24.5 -> 2.16 mm, vias 1 -> 0
- net /MOD_DIO1: track 16.2 -> 7.67 mm
- net /MOD_BUSY: track 15.2 -> 6.77 mm
- net /MOD_RST: track 12.3 -> 16.0 mm
- net /MOD_SCK: track 13.3 -> 16.3 mm
- net /MOD_MOSI: track 14.2 -> 16.6 mm
- net GND: track 11.5 -> 9.65 mm, vias 9 -> 10
- net /MOD_MISO: track 15.4 -> 16.9 mm
Other:
- board text added: "LoRaWAN US915"
- board text added: "ROWAN MOTORSPORTS"
- board text added: "Wireless Comm."

Commit message: comm-unit: Update headers to 1.27mm spacing
Parts:
- J1: footprint Connector_PinSocket_1.00mm:PinSocket_1x02_P1.00mm_Vertical -> Connector_PinSocket_1.27mm:PinSocket_1x02_P1.27mm_Vertical
- J2: footprint Connector_PinSocket_1.00mm:PinSocket_1x08_P1.00mm_Vertical -> Connector_PinSocket_1.27mm:PinSocket_1x08_P1.27mm_Vertical
- moved J2 1.06 mm to (146.5, 119.7)
- moved J1 0.48 mm to (153.6, 107.2)
Connections:
- U1 pad 22: GND -> (no net)
- U1 pad 23: GND -> (no net)
- U1 pad 24: GND -> (no net)
- U1 pad 25: GND -> (no net)
Routing:
- net /MCU_BUSY: track 3.30 -> 4.21 mm
- net /MCU_RST: track 2.16 -> 2.91 mm
- net /MCU_DIO1: track 3.81 -> 4.49 mm
- net /MCU_SCK: track 1.95 -> 2.59 mm
- net /MCU_MOSI: track 2.16 -> 2.69 mm
