File: comm-unit/comm-unit.kicad_sch (KiCad schematic)
At the start: 10 parts, among them J1 Conn_01x02, J2 Conn_01x08, U1 TXS0108ERGYR, U2 MIC5365-3.3YC5-TR, U3 Wio-SX1262

Commit message: comm-unit: Update headers to 1.27mm spacing
Parts:
- J1: footprint Connector_PinSocket_1.00mm:PinSocket_1x02_P1.00mm_Vertical -> Connector_PinSocket_1.27mm:PinSocket_1x02_P1.27mm_Vertical
- J2: footprint Connector_PinSocket_1.00mm:PinSocket_1x08_P1.00mm_Vertical -> Connector_PinSocket_1.27mm:PinSocket_1x08_P1.27mm_Vertical
Changed lines of the file:
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@@
 			)
 		)
-		(property "Footprint" "Connector_PinSocket_1.00mm:PinSocket_1x02_P1.00mm_Vertical"
+		(property "Footprint" "Connector_PinSocket_1.27mm:PinSocket_1x02_P1.27mm_Vertical"
 			(at 33.02 81.28 0)
 			(effects
@@
 			)
 		)
-		(property "Footprint" "Connector_PinSocket_1.00mm:PinSocket_1x08_P1.00mm_Vertical"
+		(property "Footprint" "Connector_PinSocket_1.27mm:PinSocket_1x08_P1.27mm_Vertical"
 			(at 36.83 114.3 0)
 			(effects
