File: head-unit/pcb/head-unit.kicad_sch (KiCad schematic)
At the start: 0 parts

Commit message: Sync files
Parts:
- added J1: Conn_01x08_Socket, symbol Connector:Conn_01x08_Socket
- added J2: Conn_01x02_Pin, symbol Connector:Conn_01x02_Pin
- added J3, J4: Conn_01x03_Pin, symbol Connector:Conn_01x03_Pin
Connections:
- new net: J1.4 (Pin_4), J4.1 (Pin_1)
- new net: J1.6 (Pin_6), J3.1 (Pin_1)
- new net +5V: J2.1 (Pin_1), J3.2 (Pin_2), J4.2 (Pin_2)
- new net GND: J2.2 (Pin_2), J3.3 (Pin_3), J4.3 (Pin_3)
Other:
- note added: "GPIO Header"
- note added: "Power Header"
- note added: "Servo Headers"
