File: pmod-adapter/pmod-adapter.kicad_sch (KiCad schematic)
At the start: 0 parts

Commit message: can-module, pmod-adapter: Begin updating PMOD adapter and CAN module
Parts:
- added C1, C2: 1u, Capacitor_SMD:C_0402_1005Metric, symbol Device:C_Small
- added J1: Conn_01x08, Connector_PinSocket_1.27mm:PinSocket_1x08_P1.27mm_Vertical, symbol Connector_Generic:Conn_01x08
- added J2: Conn_01x02, Connector_PinSocket_1.27mm:PinSocket_1x02_P1.27mm_Vertical, symbol Connector_Generic:Conn_01x02
- added J3: Conn_02x06_Top_Bottom, symbol Connector_Generic:Conn_02x06_Top_Bottom
- added R1, R2, R3, R4, R5, R6, R7, R8: 200, symbol Device:R_Small
- added U1: FXMA108BQX, Package_DFN_QFN:WQFN-20-1EP_2.5x4.5mm_P0.5mm_EP1x2.9mm, symbol Logic_LevelTranslator:FXMA108
- added U2: MIC5365-3.3YC5-TR, Package_TO_SOT_SMD:SOT-353_SC-70-5, symbol Regulator_Linear:MIC5365-3.3YC5
Connections:
- new net: J1.1 (Pin_1), U1.9 (A7)
- new net: J1.2 (Pin_2), U1.8 (A6)
- new net: J1.3 (Pin_3), U1.7 (A5)
- new net: J1.4 (Pin_4), U1.6 (A4)
- new net: J1.5 (Pin_5), U1.5 (A3)
- new net: J1.6 (Pin_6), U1.4 (A2)
- new net: J1.7 (Pin_7), U1.3 (A1)
- new net: J1.8 (Pin_8), U1.2 (A0)
- new net: R5.1, U1.15 (B4)
- new net: R4.1, U1.16 (B3)
- new net: R8.1, U1.12 (B7)
- new net: R3.1, U1.17 (B2)
- new net: R6.1, U1.14 (B5)
- new net: R2.1, U1.18 (B1)
- new net: R7.1, U1.13 (B6)
- new net: R1.1, U1.19 (B0)
- new net +3V3: C2.1, J3.12 (Pin_12), J3.6 (Pin_6), U1.20 (VCCB), U2.5 (VOUT)
- new net +5V: C1.1, J2.2 (Pin_2), U1.1 (VCCA), U2.1 (VIN), U2.3 (EN)
- new net GND: C1.2, C2.2, J2.1 (Pin_1), J3.11 (Pin_11), J3.5 (Pin_5), U1.10 (GND), U2.2 (GND)
- new net PMOD0: J3.1 (Pin_1), R1.2
- new net PMOD1: J3.2 (Pin_2), R2.2
- new net PMOD2: J3.3 (Pin_3), R3.2
- new net PMOD3: J3.4 (Pin_4), R4.2
- new net PMOD4: J3.7 (Pin_7), R5.2
- new net PMOD5: J3.8 (Pin_8), R6.2
- new net PMOD6: J3.9 (Pin_9), R7.2
- new net PMOD7: J3.10 (Pin_10), R8.2
Other:
- note added: "5V to 3.3V Conversion"
- note added: "All resistors below are 200Ω"
- note added: "Connects to CAN Module"
- note added: "Level Shifter & Connectors"
- note added: "PMOD Connector"
- note added: "Power Input"

Commit message: pmod-adapter: Begin working on PMOD adapter PCB
Parts:
- J3: footprint (none) -> Connector_PinSocket_2.54mm:PinSocket_2x06_P2.54mm_Horizontal
- R1, R2, R3, R4, R5, R6, R7, R8: footprint (none) -> Resistor_SMD:R_0402_1005Metric
Other:
- note added: "Note: pins are in reverse order for routing purposes"
Changed lines of the file:
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@@
+		)
+	)
+	(text "Note: pins are in reverse\norder for routing purposes"
+		(exclude_from_sim no)
+		(at 132.842 142.494 0)
+		(effects
+			(font
+				(size 1.27 1.27)
+			)
 		)
 	)
@@
 					(size 1.27 1.27)
 				)
+				(hide yes)
 			)
 		)
@@
 			)
 		)
-		(property "Footprint" ""
+		(property "Footprint" "Resistor_SMD:R_0402_1005Metric"
 			(at 171.45 130.81 0)
 			(effects
@@
 			)
 		)
-		(property "Footprint" ""
+		(property "Footprint" "Resistor_SMD:R_0402_1005Metric"
 			(at 171.45 128.27 0)
 			(effects
@@
 			)
 		)
-		(property "Footprint" ""
+		(property "Footprint" "Resistor_SMD:R_0402_1005Metric"
 			(at 171.45 138.43 0)
 			(effects
@@
 			)
 		)
-		(property "Footprint" ""
+		(property "Footprint" "Connector_PinSocket_2.54mm:PinSocket_2x06_P2.54mm_Horizontal"
 			(at 229.87 125.73 0)
 			(effects
@@
 			)
 		)
-		(property "Footprint" ""
+		(property "Footprint" "Resistor_SMD:R_0402_1005Metric"
 			(at 171.45 125.73 0)
 			(effects
@@
 			)
 		)
-		(property "Footprint" ""
+		(property "Footprint" "Resistor_SMD:R_0402_1005Metric"
 			(at 171.45 133.35 0)
 			(effects
@@
 			)
 		)
-		(property "Footprint" ""
+		(property "Footprint" "Resistor_SMD:R_0402_1005Metric"
 			(at 171.45 123.19 0)
 			(effects
@@
 			)
 		)
-		(property "Footprint" ""
+		(property "Footprint" "Resistor_SMD:R_0402_1005Metric"
 			(at 171.45 135.89 0)
 			(effects
@@
 			)
 		)
-		(property "Footprint" ""
+		(property "Footprint" "Resistor_SMD:R_0402_1005Metric"
 			(at 171.45 120.65 0)
 			(effects

Commit message: pmod-adapter: Finish board design
Parts:
- added C3: 1u, Capacitor_SMD:C_0402_1005Metric, symbol Device:C_Small
- added C4, C5: 100n, Capacitor_SMD:C_0402_1005Metric, symbol Device:C_Small
- added JP1: SolderJumper_3_Bridged12, Jumper:SolderJumper-3_P1.3mm_Bridged12_RoundedPad1.0x1.5mm, symbol Jumper:SolderJumper_3_Bridged12
Connections:
- net +3V3: now also JP1.1 (A); no longer J3.12 (Pin_12), J3.6 (Pin_6), U1.20 (VCCB)
- net +5V: now also C4.1, JP1.3 (B)
- net GND: now also U1.11 (~{OE}), U1.21 (NC), C3.2, C4.2, C5.2
- new net V_{PMOD}: C3.1, C5.1, J3.12 (Pin_12), J3.6 (Pin_6), JP1.2 (C), U1.20 (VCCB)
Other:
- note added: "Note: pins are out of order for routing purposes"
- note added: "PMOD Voltage Selection"
- note added: "~{OE} low -> Normal Operation"
- note removed: "Note: pins are in reverse order for routing purposes"
- moved on the sheet: C1, C2, J2, J3, R1, R2, R3, R4, R5, R6, R7, R8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
