File: pmod-adapter/pcb/pmod-adapter.kicad_sch (KiCad schematic)
At the start: 19 parts, among them J1 Conn_01x08, J2 Conn_01x02, J3 Conn_02x06_Top_Bottom, U1 FXMA108BQX, U2 MIC5365-3.3YC5-TR

Commit message: pmod-adapter: Fill out info on sch
Other:
- company: (none) -> Ryan Hausmann
- title: (none) -> PMOD Adapter
Changed lines of the file:
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@@
 	(generator_version "9.0")
 	(paper "A4")
+	(title_block
+		(title "PMOD Adapter")
+		(date "2026-02-12")
+		(rev "A")
+		(company "Ryan Hausmann")
+		(comment 1 "Rowan Motorsports")
+	)
 	(text "Power Input"
 		(exclude_from_sim no)
