File: accelerometer-board/pcb/accelerometer-board.kicad_sch (KiCad schematic)
At the start: 15 parts, among them J1 Conn_01x08, J2 Conn_01x02, U1 BMI323, U2 FXMAR2104UMX, U6 MIC5365-3.3YC5-TR

Commit message: accelerometer-board: Fill out info on sch
Other:
- company: (none) -> Ryan Hausmann
- title: (none) -> Accelerometer Board
Changed lines of the file:
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@@
 	(generator_version "9.0")
 	(paper "A4")
+	(title_block
+		(title "Accelerometer Board")
+		(date "2026-02-12")
+		(rev "A")
+		(company "Ryan Hausmann")
+		(comment 1 "Rowan Motorsports")
+	)
 	(text "Inertial Measurement Unit (IMU)"
 		(exclude_from_sim no)
