File: comm-unit/pcb/comm-unit.kicad_sch (KiCad schematic)
At the start: 10 parts, among them J1 Conn_01x02, J2 Conn_01x08, U1 TXS0108ERGYR, U2 MIC5365-3.3YC5-TR, U3 Wio-SX1262

Commit message: comm-unit: Fill out info in sch
Other:
- company: (none) -> Ryan Hausmann
- title: (none) -> Wireless Communication Unit
Changed lines of the file:
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@@
 	(generator_version "9.0")
 	(paper "A4")
+	(title_block
+		(title "Wireless Communication Unit")
+		(date "2026-02-12")
+		(rev "A")
+		(company "Ryan Hausmann")
+		(comment 1 "Rowan Motorsports")
+	)
 	(text "5V -> 3.3V Regulator"
 		(exclude_from_sim no)
