File: sd-card-board/pcb/sd-card-board.kicad_pcb (KiCad board)
At the start: 2 copper layers, 22.9 x 19.1 mm, 9 parts, among them J1 Conn_01x08, J2 Conn_01x02, J3 1051620001, U1 MIC5365-3.3YC5-TR, U2 FXMAR2104UMX

Commit message: sd-card-board: Fix PCB, switch from using SERCOM0 to SERCOM2
Connections:
- J1 pad 1: unconnected-(J1-Pin_1-Pad1) -> /MCU_DO
- J1 pad 2: unconnected-(J1-Pin_2-Pad2) -> /MCU_CLK
- J1 pad 3: /MCU_DO -> /MCU_DI
- J1 pad 4: /MCU_CLK -> /~{MCU_CS}
- J1 pad 5: /MCU_DI -> unconnected-(J1-Pin_5-Pad5)
- J1 pad 6: /~{MCU_CS} -> unconnected-(J1-Pin_6-Pad6)
Routing:
- net /~{MCU_CS}: track 11.9 -> 8.38 mm, vias 1 -> 0
- net /MCU_DO: track 5.37 -> 1.96 mm
- net /MCU_DI: track 9.13 -> 6.38 mm
- net /MCU_CLK: track 7.23 -> 4.50 mm
