File: sd-card-board/pcb/sd-card-board.kicad_sch (KiCad schematic)
At the start: 7 parts, among them J1 Conn_01x08, J2 Conn_01x02, J3 1051620001, U1 MIC5365-3.3YC5-TR, U2 FXMAR2104UMX

Commit message: sd-card-board: Fill out info on sch
Other:
- company: (none) -> Ryan Hausmann
- title: (none) -> SD Card Board
Changed lines of the file:
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@@
 	(generator_version "9.0")
 	(paper "A4")
+	(title_block
+		(title "SD Card Board")
+		(date "2026-02-12")
+		(rev "A")
+		(company "Ryan Hausmann")
+		(comment 1 "Rowan Motorsports")
+	)
 	(text "MicroSD Card Slot"
 		(exclude_from_sim no)

Commit message: sd-card-board: Switch pins around to ensure that all SPI pins are connected to the same peripheral
Connections:
- net MCU_CLK: now also J1.6 (Pin_6); no longer J1.4 (Pin_4)
- net MCU_DI: now also J1.7 (Pin_7); no longer J1.5 (Pin_5)
- net MCU_DO: now also J1.5 (Pin_5); no longer J1.3 (Pin_3)
- net ~{MCU_CS}: now also J1.8 (Pin_8); no longer J1.6 (Pin_6)
Changed lines of the file:
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@@
-	)
-	(no_connect
-		(at 76.2 106.68)
 	)
 	(no_connect
@@
 	)
 	(no_connect
+		(at 76.2 119.38)
+	)
+	(no_connect
 		(at 76.2 124.46)
 	)
 	(no_connect
-		(at 76.2 109.22)
+		(at 76.2 116.84)
 	)
 	(wire
@@
 	(wire
 		(pts
+			(xy 76.2 109.22) (xy 85.09 109.22)
+		)
+		(stroke
+			(width 0)
+			(type default)
+		)
+	)
+	(wire
+		(pts
 			(xy 179.07 63.5) (xy 176.53 63.5)
 		)
@@
 	(wire
 		(pts
+			(xy 76.2 114.3) (xy 85.09 114.3)
+		)
+		(stroke
+			(width 0)
+			(type default)
+		)
+	)
+	(wire
+		(pts
+			(xy 76.2 111.76) (xy 85.09 111.76)
+		)
+		(stroke
+			(width 0)
+			(type default)
+		)
+	)
+	(wire
+		(pts
 			(xy 171.45 60.96) (xy 171.45 63.5)
 		)
@@
 	(wire
 		(pts
-			(xy 76.2 114.3) (xy 85.09 114.3)
-		)
-		(stroke
-			(width 0)
-			(type default)
-		)
-	)
-	(wire
-		(pts
 			(xy 176.53 63.5) (xy 171.45 63.5)
 		)
@@
 	(wire
 		(pts
+			(xy 76.2 106.68) (xy 85.09 106.68)
+		)
+		(stroke
+			(width 0)
+			(type default)
+		)
+	)
+	(wire
+		(pts
 			(xy 194.31 110.49) (xy 201.93 110.49)
 		)
@@
 	(wire
 		(pts
-			(xy 76.2 111.76) (xy 85.09 111.76)
-		)
-		(stroke
-			(width 0)
-			(type default)
-		)
-	)
-	(wire
-		(pts
 			(xy 171.45 74.93) (xy 189.23 74.93)
 		)
@@
 	(wire
 		(pts
-			(xy 76.2 116.84) (xy 85.09 116.84)
-		)
-		(stroke
-			(width 0)
-			(type default)
-		)
-	)
-	(wire
-		(pts
 			(xy 201.93 66.04) (xy 201.93 63.5)
 		)
@@
 	(wire
 		(pts
-			(xy 76.2 119.38) (xy 85.09 119.38)
-		)
-		(stroke
-			(width 0)
-			(type default)
-		)
-	)
-	(wire
-		(pts
 			(xy 113.03 118.11) (xy 121.92 118.11)
 		)
@@
 		)
 	)
-	(label "MCU_DI"
-		(at 85.09 114.3 180)
+	(label "~{MCU_CS}"
+		(at 85.09 106.68 180)
 		(effects
 			(font
@@
 		)
 	)
+	(label "MCU_CLK"
+		(at 85.09 111.76 180)
+		(effects
+			(font
+				(size 1.27 1.27)
+				(thickness 0.1588)
+			)
+			(justify right bottom)
+		)
+	)
 	(label "~{SD_CS}"
 		(at 194.31 110.49 0)
@@
 		)
 	)
-	(label "~{MCU_CS}"
-		(at 85.09 111.76 180)
+	(label "MCU_DI"
+		(at 85.09 109.22 180)
 		(effects
 			(font
@@
 		)
 	)
+	(label "MCU_DO"
+		(at 85.09 114.3 180)
+		(effects
+			(font
+				(size 1.27 1.27)
+				(thickness 0.1588)
+			)
+			(justify right bottom)
+		)
+	)
 	(label "SD_DI"
 		(at 194.31 113.03 0)
@@
 		)
 	)
-	(label "MCU_CLK"
-		(at 85.09 116.84 180)
-		(effects
-			(font
-				(size 1.27 1.27)
-				(thickness 0.1588)
-			)
-			(justify right bottom)
-		)
-	)
-	(label "MCU_DO"
-		(at 85.09 119.38 180)
-		(effects
-			(font
-				(size 1.27 1.27)
-				(thickness 0.1588)
-			)
-			(justify right bottom)
-		)
-	)

Commit message: sd-card-board: Fix PCB, switch from using SERCOM0 to SERCOM2
Connections:
- net MCU_CLK: now also J1.2 (Pin_2); no longer J1.6 (Pin_6)
- net MCU_DI: now also J1.3 (Pin_3); no longer J1.7 (Pin_7)
- net MCU_DO: now also J1.1 (Pin_1); no longer J1.5 (Pin_5)
- net ~{MCU_CS}: now also J1.4 (Pin_4); no longer J1.8 (Pin_8)
Changed lines of the file:
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@@
 	)
 	(no_connect
-		(at 76.2 121.92)
+		(at 76.2 114.3)
+	)
+	(no_connect
+		(at 76.2 111.76)
 	)
 	(no_connect
@@
 	)
 	(no_connect
-		(at 76.2 119.38)
+		(at 76.2 106.68)
 	)
 	(no_connect
-		(at 76.2 124.46)
-	)
-	(no_connect
-		(at 76.2 116.84)
+		(at 76.2 109.22)
 	)
 	(wire
@@
 	(wire
 		(pts
-			(xy 76.2 109.22) (xy 85.09 109.22)
-		)
-		(stroke
-			(width 0)
-			(type default)
-		)
-	)
-	(wire
-		(pts
 			(xy 179.07 63.5) (xy 176.53 63.5)
 		)
@@
 	(wire
 		(pts
-			(xy 76.2 114.3) (xy 85.09 114.3)
-		)
-		(stroke
-			(width 0)
-			(type default)
-		)
-	)
-	(wire
-		(pts
-			(xy 76.2 111.76) (xy 85.09 111.76)
-		)
-		(stroke
-			(width 0)
-			(type default)
-		)
-	)
-	(wire
-		(pts
 			(xy 171.45 60.96) (xy 171.45 63.5)
 		)
@@
 	(wire
 		(pts
+			(xy 76.2 116.84) (xy 85.09 116.84)
+		)
+		(stroke
+			(width 0)
+			(type default)
+		)
+	)
+	(wire
+		(pts
+			(xy 76.2 124.46) (xy 85.09 124.46)
+		)
+		(stroke
+			(width 0)
+			(type default)
+		)
+	)
+	(wire
+		(pts
 			(xy 176.53 63.5) (xy 171.45 63.5)
 		)
@@
 	(wire
 		(pts
-			(xy 76.2 106.68) (xy 85.09 106.68)
-		)
-		(stroke
-			(width 0)
-			(type default)
-		)
-	)
-	(wire
-		(pts
 			(xy 194.31 110.49) (xy 201.93 110.49)
 		)
@@
 	(wire
 		(pts
+			(xy 76.2 121.92) (xy 85.09 121.92)
+		)
+		(stroke
+			(width 0)
+			(type default)
+		)
+	)
+	(wire
+		(pts
 			(xy 246.38 132.08) (xy 246.38 130.81)
 		)
@@
 	(wire
 		(pts
+			(xy 76.2 119.38) (xy 85.09 119.38)
+		)
+		(stroke
+			(width 0)
+			(type default)
+		)
+	)
+	(wire
+		(pts
 			(xy 189.23 74.93) (xy 189.23 76.2)
 		)
@@
 		)
 	)
-	(label "~{MCU_CS}"
-		(at 85.09 106.68 180)
+	(label "MCU_CLK"
+		(at 85.09 121.92 180)
 		(effects
 			(font
@@
 		)
 	)
+	(label "MCU_DI"
+		(at 85.09 119.38 180)
+		(effects
+			(font
+				(size 1.27 1.27)
+				(thickness 0.1588)
+			)
+			(justify right bottom)
+		)
+	)
 	(label "SD_CLK"
 		(at 194.31 118.11 0)
@@
 		)
 	)
-	(label "MCU_CLK"
-		(at 85.09 111.76 180)
+	(label "~{MCU_CS}"
+		(at 85.09 116.84 180)
 		(effects
 			(font
@@
 		)
 	)
-	(label "MCU_DI"
-		(at 85.09 109.22 180)
+	(label "MCU_DO"
+		(at 85.09 124.46 180)
 		(effects
 			(font
@@
 		(effects
 			(font
-				(size 1.27 1.27)
-				(thickness 0.1588)
-			)
-			(justify right bottom)
-		)
-	)
-	(label "MCU_DO"
-		(at 85.09 114.3 180)
-		(effects
-			(font
